File: pcb/slice/slice.kicad_pcb (KiCad board)
At the start: 2 copper layers, 163 parts, among them J1 Bottom, J2 Top, Q1 2N7002, Q10 2N7002, Q100 2N7002, Q101 2N7002, Q102 2N7002, Q103 2N7002, Q104 2N7002, Q105 2N7002, Q106 2N7002, Q107 2N7002, Q108 2N7002, Q109 2N7002, Q11 2N7002, Q110 2N7002, Q111 2N7002, Q112 2N7002, Q113 2N7002, Q114 2N7002, Q115 2N7002, Q116 2N7002, Q117 2N7002, Q118 2N7002, Q119 2N7002, Q12 2N7002, Q120 2N7002, Q121 2N7002, Q13 2N7002, Q14 2N7002, Q15 2N7002, Q16 2N7002, Q17 2N7002, Q18 2N7002, Q19 2N7002, Q2 2N7002, Q20 2N7002, Q21 2N7002, Q22 2N7002, Q23 2N7002, Q24 2N7002, Q25 2N7002, Q26 2N7002, Q27 2N7002, Q28 2N7002, Q29 2N7002, Q3 2N7002, Q30 2N7002, Q31 2N7002, Q32 2N7002, Q33 2N7002, Q34 2N7002, Q35 2N7002, Q36 2N7002, Q37 2N7002, Q38 2N7002, Q39 2N7002, Q4 2N7002, Q40 2N7002, Q41 2N7002, Q42 2N7002, Q43 2N7002, Q44 2N7002, Q45 2N7002, Q46 2N7002, Q47 2N7002, Q48 2N7002, Q49 2N7002, Q5 2N7002, Q50 2N7002, Q51 2N7002, Q52 2N7002, Q53 2N7002, Q54 2N7002, Q55 2N7002, Q56 2N7002, Q57 2N7002, Q58 2N7002, Q59 2N7002, Q6 2N7002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

Commit message: New design
Parts:
- removed J2: Top, Connector_Harwin:Harwin_M20-89020xx_1x20_P2.54mm_Horizontal
- removed the Q1 at (233.3, 91.2)
- removed Q100, Q101, Q102, Q103, Q104, Q105, Q106, Q107, Q108, Q109, Q110, Q111, Q112, Q114, Q116, Q117, Q118, Q119, Q120, Q121, Q83, Q84, Q85, Q86, Q87, Q88, Q89, Q90, Q94, Q95, Q96, Q99: 2N7002, Package_TO_SOT_SMD:SOT-23
- removed the Q22 at (130.2, 138.2)
- removed the Q23 at (134.7, 138.2)
- removed the Q25 at (192.6, 69.5)
- removed the Q30 at (253.1, 78.1)
- removed the Q31 at (255.4, 52.8)
- removed the Q52 at (266.8, 52.8)
- removed the Q54 at (279.8, 78.1)
- removed the Q6 at (183.7, 74.0)
- removed the Q7 at (196.7, 78.6)
- removed the R19 at (209.3, 74.6)
- added D4: S, LED_THT:LED_D3.0mm_Horizontal_O1.27mm_Z2.0mm, F.Cu at (91.0, 7.00)
- added Q4: 2N7002, Package_TO_SOT_SMD:SOT-23_Handsoldering, F.Cu at (169.5, 50.0)
- added Q68: 2N7002, Package_TO_SOT_SMD:SOT-23_Handsoldering, F.Cu at (151.5, 61.0)
- added Q69: 2N7002, Package_TO_SOT_SMD:SOT-23_Handsoldering, F.Cu at (99.0, 9.50)
- D1, D2, D3: footprint LED_THT:LED_D3.0mm -> LED_THT:LED_D3.0mm_Horizontal_O1.27mm_Z2.0mm
- J1: value Bottom -> Conn_02x16_Odd_Even; footprint Connector_Harwin:Harwin_M20-89020xx_1x20_P2.54mm_Horizontal -> Connector_PinHeader_2.54mm:PinHeader_2x16_P2.54mm_Horizontal; moved to F.Cu
- Q1: renamed from Q2; footprint Package_TO_SOT_SMD:SOT-23 -> Package_TO_SOT_SMD:SOT-23_Handsoldering
- Q10, Q11, Q12, Q13, Q14, Q15, Q16, Q17, Q18, Q19, Q20, Q21, Q24, Q26, Q27, Q28, Q29, Q32, Q33, Q34, Q35, Q36, Q37, Q38, Q39, Q40, Q41, Q42, Q43, Q44, Q45, Q46, Q47, Q48, Q49, Q5, Q50, Q51, Q53, Q55, Q56, Q57, Q58, Q59, Q60, Q61, Q62, Q63, Q64, Q65, Q66, Q67, Q70, Q71, Q72, Q73, Q74, Q75, Q76, Q77, Q78, Q79, Q8, Q80, Q81, Q82, Q9: footprint Package_TO_SOT_SMD:SOT-23 -> Package_TO_SOT_SMD:SOT-23_Handsoldering
- Q2: renamed from Q3; footprint Package_TO_SOT_SMD:SOT-23 -> Package_TO_SOT_SMD:SOT-23_Handsoldering
- Q22: renamed from Q91; footprint Package_TO_SOT_SMD:SOT-23 -> Package_TO_SOT_SMD:SOT-23_Handsoldering
- Q23: renamed from Q97; footprint Package_TO_SOT_SMD:SOT-23 -> Package_TO_SOT_SMD:SOT-23_Handsoldering
- Q25: renamed from Q98; footprint Package_TO_SOT_SMD:SOT-23 -> Package_TO_SOT_SMD:SOT-23_Handsoldering
- Q3: renamed from Q4; footprint Package_TO_SOT_SMD:SOT-23 -> Package_TO_SOT_SMD:SOT-23_Handsoldering
- Q30: renamed from Q93; footprint Package_TO_SOT_SMD:SOT-23 -> Package_TO_SOT_SMD:SOT-23_Handsoldering
- Q31: renamed from Q92; footprint Package_TO_SOT_SMD:SOT-23 -> Package_TO_SOT_SMD:SOT-23_Handsoldering
- Q52: renamed from Q113; footprint Package_TO_SOT_SMD:SOT-23 -> Package_TO_SOT_SMD:SOT-23_Handsoldering
- Q54: renamed from Q115; footprint Package_TO_SOT_SMD:SOT-23 -> Package_TO_SOT_SMD:SOT-23_Handsoldering
- Q6: renamed from Q68; footprint Package_TO_SOT_SMD:SOT-23 -> Package_TO_SOT_SMD:SOT-23_Handsoldering
- Q7: renamed from Q69; footprint Package_TO_SOT_SMD:SOT-23 -> Package_TO_SOT_SMD:SOT-23_Handsoldering
- moved R33 160.9 mm to (95.0, 20.5), turned to 90 degrees
- moved Q22 160.4 mm to (145.5, 9.50), turned to 180 degrees
- moved R32 156.8 mm to (110.5, 26.0), turned to 90 degrees
- moved Q23 155.7 mm to (151.5, 9.50), turned to 180 degrees
- moved Q6 155.2 mm to (114.5, 50.0), turned to 180 degrees
- moved Q34 152.8 mm to (136.0, 9.50), turned to 180 degrees
- moved Q7 152.5 mm to (120.5, 50.0), turned to 180 degrees
- moved Q42 152.1 mm to (136.0, 15.0), turned to 180 degrees
- moved Q53 151.8 mm to (130.0, 50.0), turned to 180 degrees
- moved R34 150.7 mm to (110.5, 20.5), turned to 90 degrees
- moved R31 150.6 mm to (110.5, 15.0), turned to 90 degrees
- moved Q33 149.0 mm to (130.0, 26.0), turned to 180 degrees
- moved Q78 148.6 mm to (99.0, 20.5), turned to 180 degrees
- moved Q70 148.3 mm to (99.0, 15.0), turned to 180 degrees
- moved Q72 147.5 mm to (105.0, 9.50), turned to 180 degrees
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- renumbered R36 to R19
Connections:
- D1 pad 1: ~A -> Net-(D1-Pad1)
- D2 pad 1: ~P -> Net-(D2-Pad1)
- D3 pad 1: GND -> Net-(D3-Pad1)
- J1 pad 1: GND -> VCC
- J1 pad 10: RDX_ABUS -> (no net)
- J1 pad 11: XIN_DBUS -> ~RST
- J1 pad 12: XIN_ABUS -> ~WRP
- J1 pad 13: RDP_ABUS -> DEP
- J1 pad 14: WRP -> RDP_ABUS
- J1 pad 15: PIN_NEXT -> RDA_DBUS
- J1 pad 16: PIN_X -> RDX_ABUS
- J1 pad 17: PCOUT -> WRA
- J1 pad 18: FOUT -> XIN_DBUS
- J1 pad 19: Xn -> WRS
- J1 pad 2: DBUS -> VCC
- J1 pad 20: VCC -> XIN_SHIFT
- J1 pad 3: ABUS -> INCP_CLK
- J1 pad 4: CLK2 -> ~P
- J1 pad 5: (no net) -> AOUT
- J1 pad 6: DEP -> AIN
- J1 pad 7: ~SW -> ~XOUT
- J1 pad 8: WRX -> ~XIN
- J1 pad 9: RDX_DBUS -> XOUT
- Q10 pad 1: Net-(Q10-Pad1) -> /A Register/A DFF/~Q
- Q10 pad 2: Net-(Q10-Pad2) -> GND
- Q12 pad 1: Net-(Q12-Pad1) -> AOUT
- Q12 pad 2: GND -> Net-(Q12-Pad2)
- Q12 pad 3: Net-(Q12-Pad3) -> /A Register/A DFF/~Q
- Q13 pad 1: A -> Net-(Q13-Pad1)
- Q14 pad 2: Net-(Q14-Pad2) -> GND
- Q14 pad 3: Net-(Q12-Pad1) -> Net-(Q12-Pad2)
- Q15 pad 1: Net-(Q11-Pad1) -> WRA
- Q15 pad 2: Net-(Q13-Pad2) -> GND
- Q15 pad 3: Net-(Q15-Pad3) -> Net-(Q13-Pad2)
- Q16 pad 1: Net-(Q12-Pad1) -> Net-(Q11-Pad1)
- Q16 pad 2: Net-(Q14-Pad2) -> Net-(Q16-Pad2)
- Q16 pad 3: Net-(Q10-Pad1) -> Net-(Q14-Pad1)
- Q17 pad 1: FIN -> Net-(Q17-Pad1)
- Q17 pad 2: GND -> Net-(Q17-Pad2)
- Q17 pad 3: Net-(Q14-Pad2) -> Net-(Q16-Pad2)
- Q18 pad 1: Net-(Q12-Pad1) -> WRA
- Q18 pad 2: Net-(Q18-Pad2) -> GND
- Q18 pad 3: FOUT -> Net-(Q17-Pad2)
- Q19 pad 1: Net-(Q11-Pad1) -> Net-(Q14-Pad1)
- Q19 pad 3: Net-(Q18-Pad2) -> Net-(Q17-Pad1)
- Q20 pad 1: ADD -> AIN
- Q21 pad 1: SUB -> P
- Q21 pad 3: Net-(Q19-Pad2) -> Net-(D2-Pad1)
- Q24 pad 1: SUB -> ~WRP
- Q24 pad 3: Net-(Q13-Pad2) -> SETP
- Q25 pad 1: RST -> ~XOUT
- Q25 pad 2: GND -> Net-(Q24-Pad2)
- Q25 pad 3: Net-(Q92-Pad2) -> SETP
- Q26 pad 1: ~X -> ~WRP
- Q26 pad 2: GND -> Net-(Q26-Pad2)
- Q26 pad 3: Net-(Q24-Pad2) -> CLRP
- Q27 pad 1: X -> XOUT
- Q27 pad 2: GND -> Net-(Q26-Pad2)
- Q27 pad 3: Net-(Q25-Pad2) -> CLRP
- Q28 pad 1: ~X -> ~RST
- Q28 pad 2: Net-(Q28-Pad2) -> GND
- Q28 pad 3: ALU_OUT -> Net-(Q24-Pad2)
- Q29 pad 1: Net-(Q29-Pad1) -> ~SW
- Q29 pad 2: Net-(Q29-Pad2) -> GND
- Q29 pad 3: FOUT -> Net-(Q24-Pad2)
- Q30 pad 1: SW -> ~RST
- Q30 pad 2: Net-(Q92-Pad2) -> GND
- Q30 pad 3: ~NP -> Net-(Q26-Pad2)
- Q31 pad 1: ~SW -> SW
- Q31 pad 2: Net-(Q92-Pad2) -> GND
- Q31 pad 3: NP -> Net-(Q26-Pad2)
- Q32 pad 1: FIN -> Net-(Q32-Pad1)
- Q32 pad 2: GND -> Net-(Q32-Pad2)
- Q32 pad 3: Net-(Q29-Pad1) -> P
- Q33 pad 1: X -> Net-(Q33-Pad1)
- Q33 pad 3: ALU_OUT -> Net-(Q33-Pad3)
- Q34 pad 1: ~X -> ~P
- Q34 pad 2: Net-(Q34-Pad2) -> SETP
- Q34 pad 3: ALU_OUT -> Net-(Q32-Pad2)
- Q35 pad 1: LD -> Net-(Q32-Pad1)
- Q35 pad 2: GND -> SETP
- Q35 pad 3: Net-(Q29-Pad2) -> Net-(Q33-Pad2)
- Q36 pad 1: NOT -> P
- Q36 pad 2: GND -> Net-(Q36-Pad2)
- Q36 pad 3: Net-(Q29-Pad2) -> ~P
- Q37 pad 1: AND -> Net-(Q33-Pad3)
- Q37 pad 2: GND -> Net-(Q37-Pad2)
- Q37 pad 3: Net-(Q29-Pad2) -> Net-(Q32-Pad1)
- Q38 pad 1: OR -> Net-(Q38-Pad1)
- Q38 pad 2: GND -> CLRP
- Q38 pad 3: Net-(Q29-Pad2) -> Net-(Q36-Pad2)
- Q39 pad 1: XOR -> INCP_CLK
- Q39 pad 2: GND -> CLRP
- Q39 pad 3: Net-(Q29-Pad2) -> Net-(Q37-Pad2)
- Q40 pad 1: X -> Net-(Q32-Pad1)
- Q40 pad 3: ALU_OUT -> Net-(Q38-Pad1)
- Q41 pad 1: A -> Net-(Q33-Pad1)
- Q41 pad 3: Net-(Q33-Pad2) -> Net-(Q40-Pad2)
- Q42 pad 1: ~A -> INCP_CLK
- Q42 pad 2: Net-(Q41-Pad2) -> GND
- Q42 pad 3: Net-(Q34-Pad2) -> Net-(Q41-Pad2)
- Q43 pad 1: NOT -> Net-(Q38-Pad1)
- Q43 pad 2: GND -> Net-(Q43-Pad2)
- Q43 pad 3: Net-(Q40-Pad2) -> Net-(Q33-Pad1)
- Q44 pad 1: XOR -> ~P
- Q44 pad 2: GND -> CLRP
- Q44 pad 3: Net-(Q41-Pad2) -> Net-(Q43-Pad2)
- Q45 pad 1: ~X -> XIN_ZERO
- Q45 pad 2: Net-(Q45-Pad2) -> GND
- Q45 pad 3: ALU_OUT -> /X Register/X DFF/D
- Q46 pad 1: ~A -> ~DBUS
- Q46 pad 3: ALU_OUT -> /X Register/X DFF/D
- Q47 pad 1: ~X -> ~P
- Q47 pad 2: Net-(Q46-Pad2) -> Net-(Q47-Pad2)
- Q47 pad 3: ALU_OUT -> /X Register/X DFF/D
- Q48 pad 1: ~A -> ~XIN
- Q48 pad 3: Net-(Q45-Pad2) -> /X Register/X DFF/D
- Q49 pad 1: AND -> XIN_DBUS
- Q5 pad 1: Net-(Q5-Pad1) -> AOUT
- Q5 pad 2: Net-(Q5-Pad2) -> GND
- Q5 pad 3: Net-(Q14-Pad1) -> Net-(D1-Pad1)
- Q50 pad 1: OR -> XIN_P
- Q50 pad 3: Net-(Q48-Pad2) -> Net-(Q47-Pad2)
- Q51 pad 1: Net-(Q51-Pad1) -> XIN_SHIFT
- Q51 pad 2: Net-(Q51-Pad2) -> GND
- Q51 pad 3: ALU_OUT -> Net-(Q48-Pad2)
- Q52 pad 1: ~X -> ~XOUT
- Q53 pad 1: Xn -> XOUT
- Q53 pad 3: Net-(Q51-Pad1) -> Net-(D3-Pad1)
- Q55 pad 1: ROR -> DBUS
- Q55 pad 3: Net-(Q52-Pad2) (its old number) -> ~DBUS
- Q56 pad 1: ALU_OUT -> Net-(Q56-Pad1)
- Q56 pad 3: Net-(Q56-Pad3) -> XOUT
- Q57 pad 1: ~ALU_OUT -> Net-(Q57-Pad1)
- Q58 pad 1: Net-(Q57-Pad3) -> ~XOUT
- Q58 pad 2: Net-(Q58-Pad2) -> GND
- Q58 pad 3: ~A -> Net-(Q56-Pad2)
- Q59 pad 1: Net-(Q56-Pad3) -> Net-(Q56-Pad1)
- Q59 pad 2: Net-(Q59-Pad2) -> GND
- Q59 pad 3: A -> Net-(Q57-Pad2)
- Q6 pad 1: ~A -> /A Register/A DFF/~Q
- Q60 pad 1: Net-(Q57-Pad3) -> XOUT
- Q60 pad 2: GND -> Net-(Q60-Pad2)
- Q60 pad 3: Net-(Q56-Pad3) -> ~XOUT
- Q61 pad 1: Net-(Q56-Pad3) -> Net-(Q57-Pad3)
- Q61 pad 2: GND -> Net-(Q61-Pad2)
- Q61 pad 3: Net-(Q57-Pad3) -> Net-(Q56-Pad1)
- Q62 pad 1: A -> Net-(Q62-Pad1)
- Q62 pad 3: ~A -> Net-(Q60-Pad2)
- Q63 pad 1: ~A -> WRX
- Q63 pad 3: A -> Net-(Q61-Pad2)
- Q64 pad 1: WRA -> Net-(Q56-Pad1)
- Q64 pad 2: GND -> Net-(Q64-Pad2)
- Q64 pad 3: Net-(Q56-Pad2) -> Net-(Q62-Pad1)
- Q65 pad 1: WRA -> Net-(Q57-Pad1)
- Q65 pad 2: GND -> Net-(Q65-Pad2)
- Q65 pad 3: Net-(Q57-Pad2) -> Net-(Q64-Pad2)
- Q66 pad 1: CLK2 -> WRX
- Q66 pad 3: Net-(Q58-Pad2) -> Net-(Q65-Pad2)
- Q67 pad 1: CLK2 -> Net-(Q62-Pad1)
- Q67 pad 2: GND -> Net-(Q67-Pad2)
- Q67 pad 3: Net-(Q59-Pad2) -> Net-(Q57-Pad1)
- Q70 pad 1: NP -> Net-(Q70-Pad1)
- Q70 pad 2: GND -> Net-(Q70-Pad2)
- Q70 pad 3: ~NP -> SOUT
- Q71 pad 1: ~NP -> Net-(Q71-Pad1)
- Q71 pad 2: GND -> Net-(Q71-Pad2)
- Q71 pad 3: NP -> Net-(Q71-Pad3)
- Q72 pad 1: P -> ~SOUT
- Q72 pad 3: ~P -> Net-(Q70-Pad2)
- Q73 pad 1: ~P -> Net-(Q70-Pad1)
- Q73 pad 3: P -> Net-(Q71-Pad2)
- Q74 pad 1: PIN_NEXT -> SOUT
- Q74 pad 3: Net-(Q74-Pad3) -> ~SOUT
- Q75 pad 1: PIN_X -> Net-(Q71-Pad3)
- Q75 pad 3: Net-(Q74-Pad3) -> Net-(Q70-Pad1)
- Q76 pad 1: Net-(Q74-Pad3) -> Net-(Q76-Pad1)
- Q76 pad 2: GND -> RST
- Q76 pad 3: Net-(Q76-Pad3) -> Net-(Q74-Pad2)
- Q77 pad 1: PNEXT -> WRS
- Q77 pad 2: GND -> RST
- Q77 pad 3: Net-(Q74-Pad2) -> Net-(Q75-Pad2)
- Q78 pad 1: X -> Net-(Q70-Pad1)
- Q78 pad 2: GND -> Net-(Q78-Pad2)
- Q78 pad 3: Net-(Q75-Pad2) -> Net-(Q76-Pad1)
- Q79 pad 1: Net-(Q76-Pad3) -> Net-(Q71-Pad1)
- Q79 pad 3: ~NP -> Net-(Q78-Pad2)
- Q8 pad 1: Net-(Q14-Pad1) -> Net-(Q11-Pad1)
- Q8 pad 2: Net-(Q12-Pad3) -> Net-(Q10-Pad3)
- Q8 pad 3: Net-(Q6-Pad1) -> AOUT
- Q80 pad 1: Net-(Q74-Pad3) -> WRS
- Q80 pad 2: Net-(Q80-Pad2) -> GND
- Q80 pad 3: NP -> Net-(Q79-Pad2)
- Q81 pad 1: NP -> Net-(Q76-Pad1)
- Q81 pad 3: ~P -> Net-(Q71-Pad1)
- Q82 pad 1: ~NP -> SIN
- Q82 pad 2: Net-(Q82-Pad2) -> RST
- Q82 pad 3: P -> Net-(Q81-Pad2)
- Q9 pad 1: Net-(Q15-Pad3) -> Net-(Q17-Pad1)
- Q9 pad 2: GND -> Net-(Q11-Pad3)
- Q9 pad 3: Net-(Q5-Pad2) -> Net-(Q13-Pad1)
- R10 pad 2: Net-(Q12-Pad1) -> Net-(Q14-Pad1)
- R11 pad 2: Net-(Q15-Pad3) -> Net-(Q17-Pad1)
- R12 pad 2: Net-(Q10-Pad1) -> Net-(D2-Pad2)
- R13 pad 2: FOUT -> P
- R14 pad 2: Net-(Q29-Pad1) -> Net-(Q33-Pad3)
- R15 pad 2: Net-(Q51-Pad1) -> ~P
- R16 pad 2: Net-(D1-Pad2) -> Net-(Q32-Pad1)
- R17 pad 2: Net-(Q56-Pad3) -> Net-(Q38-Pad1)
- R18 pad 2: Net-(Q57-Pad3) -> Net-(Q33-Pad1)
- R19 pad 2: ~XIN -> /X Register/X DFF/D
- R20 pad 2: Net-(D2-Pad2) -> Net-(D3-Pad2)
- R21 pad 2: Net-(Q74-Pad3) -> ~DBUS
- R22 pad 2: Net-(Q76-Pad3) -> XOUT
- R23 pad 2: ~NP -> Net-(Q57-Pad3)
- R24 pad 2: NP -> ~XOUT
- R25 pad 2: P -> Net-(Q56-Pad1)
- R26 pad 2: Net-(Q89-Pad3) -> Net-(Q62-Pad1)
- R27 pad 2: PNEXT -> Net-(Q57-Pad1)
- R29 pad 2: PCOUT -> SOUT
- R3 pad 2: ~ALU_OUT -> SW
- R30 pad 2: Net-(Q94-Pad1) -> Net-(Q71-Pad3)
- R31 pad 2: Net-(Q101-Pad3) -> ~SOUT
- R32 pad 2: Net-(Q102-Pad3) -> Net-(Q70-Pad1)
- R33 pad 2: ~X -> Net-(Q76-Pad1)
- R34 pad 2: Net-(D3-Pad2) -> Net-(Q71-Pad1)
- R35 pad 2: XIN -> ~SW
- R4 pad 2: SW -> RST
- R5 pad 2: Net-(Q14-Pad1) -> Net-(D1-Pad2)
- R6 pad 2: ALU_OUT -> AOUT
- R7 pad 2: Net-(Q5-Pad1) -> Net-(Q13-Pad1)
- R8 pad 2: Net-(Q6-Pad1) -> /A Register/A DFF/~Q
Routing:
- net AOUT: track 0.00 -> 149.9 mm, vias 0 -> 4
- net XOUT: track 0.00 -> 137.5 mm, vias 0 -> 7
- net AIN: track 0.00 -> 96.1 mm, vias 0 -> 3
- net ~XOUT: track 0.00 -> 95.8 mm, vias 0 -> 5
- net INCP_CLK: track 0.00 -> 74.2 mm, vias 0 -> 5
- net ~XIN: track 0.00 -> 50.5 mm, vias 0 -> 3
- net VCC: track 0.00 -> 32.1 mm
- net /A Register/A DFF/~Q: track 0.00 -> 15.3 mm
- net Net-(Q26-Pad2): track 0.00 -> 12.3 mm
- net CLRP: track 0.00 -> 9.19 mm
- net Net-(D1-Pad1): track 0.00 -> 6.50 mm
- net Net-(Q10-Pad3): track 0.00 -> 5.79 mm
- net ~P: track 0.00 -> 3.67 mm
- net Net-(Q60-Pad2): track 0.00 -> 3.39 mm
- net Net-(Q52-Pad2): track 0.00 -> 3.39 mm
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- added copper zone on B.Cu, net GND
- added copper zone on F.Cu, net GND
Other:
- board outline added: 100 x 75 mm
- board text added: "+ +"
- board text added: "- -"
- board text added: "AO AI"
- board text added: "DB AB"
- board text added: "Q2 Slice v0"
- board text added: "RP SI"
- board text added: "RX WA"
- board text added: "WP RA"
- board text added: "WS ~SO~"
- board text added: "WX DP"
- board text added: "XI WS"
- board text added: "XP SO"
- board text added: "XZ ~SW~"
- board text added: "~PO~ PI"
- board text added: "~RS~ XO"
- board text added: "~XO~ ~XI"

Commit message: Updates
Parts:
- moved R35 30.9 mm to (171.0, 26.0), turned to 90 degrees
Routing:
- net ~XIN: track 50.5 -> 36.1 mm
- net AOUT: track 149.9 -> 135.8 mm
- net AIN: track 96.1 -> 82.6 mm
- net INCP_CLK: track 74.2 -> 60.9 mm
- net ~XOUT: track 95.8 -> 84.7 mm
- net XOUT: track 137.5 -> 127.2 mm
- net ~P: track 3.67 -> 0.00 mm
Other:
- board text added: "AB ~SW"
- board text added: "DB NC"
- board text added: "DP RP"
- board text added: "PC ~PO"
- board text added: "RA RX"
- board text added: "SI XP"
- board text added: "SO XZ"
- board text added: "WA XD"
- board text added: "WS XS"
- board text added: "XO NC"
- board text added: "~RS~ ~WP~"
- board text added: "~SO~ WX"
- board text removed: "DB AB"
- board text removed: "RP SI"
- board text removed: "RX WA"
- board text removed: "WP RA"
- board text removed: "WS ~SO~"
- board text removed: "WX DP"
- board text removed: "XI WS"
- board text removed: "XP SO"
- board text removed: "XZ ~SW~"
- board text removed: "~PO~ PI"
- board text removed: "~RS~ XO"

Commit message: Updates.
Parts:
- moved R4 48.3 mm to (179.0, 98.0), turned to 90 degrees
- moved C1 43.9 mm to (190.5, 57.5)
- moved D1 43.9 mm to (97.0, 93.5)
- moved D2 43.9 mm to (97.0, 64.0)
- moved D3 43.9 mm to (97.0, 107.5)
- moved D4 43.9 mm to (97.0, 50.5)
- moved J1 43.9 mm to (191.0, 63.0)
- moved Q1 43.9 mm to (175.5, 64.0)
- moved Q10 43.9 mm to (111.0, 93.5)
- moved Q11 43.9 mm to (111.0, 110.0)
- moved Q12 43.9 mm to (120.5, 99.0)
- moved Q13 43.9 mm to (120.5, 110.0)
- moved Q14 43.9 mm to (126.5, 99.0)
- moved Q15 43.9 mm to (126.5, 110.0)
- moved Q16 43.9 mm to (105.0, 104.5)
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Routing:
- net VCC: track 31.8 -> 429.2 mm, vias 0 -> 27
- net GND: track 0.00 -> 388.1 mm, vias 0 -> 16
- net SOUT: track 0.00 -> 162.4 mm, vias 0 -> 6
- net DBUS: track 0.00 -> 161.0 mm, vias 0 -> 5
- net WRA: track 0.00 -> 130.0 mm, vias 0 -> 5
- net WRS: track 0.00 -> 119.6 mm, vias 0 -> 5
- net RST: track 0.00 -> 117.5 mm, vias 0 -> 6
- net ~P: track 0.00 -> 117.2 mm, vias 0 -> 5
- net ~SOUT: track 0.00 -> 115.7 mm, vias 0 -> 3
- net ABUS: track 2.92 -> 97.3 mm, vias 0 -> 3
- net SIN: track 0.00 -> 88.0 mm, vias 0 -> 3
- net WRX: track 0.00 -> 83.0 mm, vias 0 -> 4
- net RDA_DBUS: track 0.00 -> 79.3 mm, vias 0 -> 3
- net ~SW: track 0.00 -> 79.0 mm, vias 0 -> 5
- net ~RST: track 0.00 -> 65.9 mm, vias 0 -> 6
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Other:
- outline, holes or cut-outs redrawn
- board text added: "A Register"
- board text added: "P Register"
- board text added: "S Register"
- board text added: "X Register"

Commit message: Updates.
Connections:
- J1 pad 27: DBUS -> ABUS
- J1 pad 29: ABUS -> DBUS
Routing:
- net ABUS: track 97.3 -> 96.3 mm
Other:
- board text added: "AB NC"
- board text added: "DB ~SW"
- board text removed: "AB ~SW"
- board text removed: "DB NC"
Changed lines of the file:
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@@
     (thickness 1.6)
     (drawings 33)
-    (tracks 1098)
+    (tracks 1099)
     (zones 0)
     (modules 123)
@@
       (net 11 ~SW))
     (pad 29 thru_hole oval (at 0 35.56) (size 1.7 1.7) (drill 1) (layers *.Cu *.Mask)
-      (net 10 ABUS))
+      (net 4 DBUS))
     (pad 28 thru_hole oval (at 2.54 33.02) (size 1.7 1.7) (drill 1) (layers *.Cu *.Mask))
     (pad 27 thru_hole oval (at 0 33.02) (size 1.7 1.7) (drill 1) (layers *.Cu *.Mask)
-      (net 4 DBUS))
+      (net 10 ABUS))
     (pad 26 thru_hole oval (at 2.54 30.48) (size 1.7 1.7) (drill 1) (layers *.Cu *.Mask)
       (net 12 WRX))
@@
     (effects (font (size 1 1) (thickness 0.15)))
   )
-  (gr_text "AB ~SW" (at 186.25 98.5) (layer F.SilkS)
+  (gr_text "DB ~SW" (at 186.25 98.5) (layer F.SilkS)
     (effects (font (size 1 1) (thickness 0.15)))
   )
@@
     (effects (font (size 1 1) (thickness 0.15)))
   )
-  (gr_text "DB NC" (at 186.25 96) (layer F.SilkS)
+  (gr_text "AB NC" (at 186.25 96) (layer F.SilkS)
     (effects (font (size 1 1) (thickness 0.15)))
   )
@@
   (segment (start 179.3 59.525) (end 178.050001 58.275001) (width 0.25) (layer F.Cu) (net 4))
   (segment (start 180 59.525) (end 179.3 59.525) (width 0.25) (layer F.Cu) (net 4))
-  (segment (start 182.295 96.02) (end 182.275 96) (width 0.25) (layer B.Cu) (net 4))
-  (via (at 182.275 96) (size 0.8) (drill 0.4) (layers F.Cu B.Cu) (net 4))
-  (segment (start 191 96.02) (end 182.295 96.02) (width 0.25) (layer B.Cu) (net 4))
   (via (at 182.275 105.5) (size 0.8) (drill 0.4) (layers F.Cu B.Cu) (net 4))
-  (segment (start 182.275 96) (end 182.275 105.5) (width 0.25) (layer F.Cu) (net 4))
   (via (at 179 105.5) (size 0.8) (drill 0.4) (layers F.Cu B.Cu) (net 4))
   (segment (start 182.275 105.5) (end 179 105.5) (width 0.25) (layer B.Cu) (net 4))
@@
   (segment (start 172.674999 109.775001) (end 177 105.45) (width 0.25) (layer F.Cu) (net 4))
   (segment (start 124 114.5) (end 165.435002 114.5) (width 0.25) (layer F.Cu) (net 4))
+  (segment (start 182.31 98.56) (end 182.275 98.525) (width 0.25) (layer B.Cu) (net 4))
+  (segment (start 191 98.56) (end 182.31 98.56) (width 0.25) (layer B.Cu) (net 4))
+  (segment (start 182.275 98.525) (end 182.275 105.5) (width 0.25) (layer F.Cu) (net 4))
+  (via (at 182.275 98.525) (size 0.8) (drill 0.4) (layers F.Cu B.Cu) (net 4))
+  (segment (start 182.275 96) (end 182.275 98.525) (width 0.25) (layer F.Cu) (net 4))
   (segment (start 192.364999 66.715001) (end 188.284999 66.715001) (width 0.25) (layer B.Cu) (net 5))
   (segment (start 193.54 65.54) (end 192.364999 66.715001) (width 0.25) (layer B.Cu) (net 5))
@@
   (segment (start 179.5 94.298002) (end 179.5 91.5) (width 0.25) (layer B.Cu) (net 10))
   (via (at 179.5 91.5) (size 0.8) (drill 0.4) (layers F.Cu B.Cu) (net 10))
-  (segment (start 183.761998 98.56) (end 179.5 94.298002) (width 0.25) (layer B.Cu) (net 10))
-  (segment (start 191 98.56) (end 183.761998 98.56) (width 0.25) (layer B.Cu) (net 10))
   (segment (start 148.475 91.5) (end 147.5 92.475) (width 0.25) (layer F.Cu) (net 10))
   (segment (start 179.5 91.5) (end 148.475 91.5) (width 0.25) (layer F.Cu) (net 10))
@@
   (segment (start 149 54) (end 150.725001 55.725001) (width 0.25) (layer B.Cu) (net 10))
   (segment (start 150 95.5) (end 150 93.5) (width 0.25) (layer F.Cu) (net 10))
+  (segment (start 181.221998 96.02) (end 191 96.02) (width 0.25) (layer B.Cu) (net 10))
+  (segment (start 179.5 94.298002) (end 181.221998 96.02) (width 0.25) (layer B.Cu) (net 10))
   (via (at 185.5 99.5) (size 0.8) (drill 0.4) (layers F.Cu B.Cu) (net 11))
   (segment (start 192.364999 99.735001) (end 185.735001 99.735001) (width 0.25) (layer B.Cu) (net 11))

Commit message: Schematic updates.
Parts:
- C1: value C -> 0.1u
- R1, R10, R11, R13, R14, R15, R16, R17, R18, R19, R2, R21, R22, R23, R24, R25, R26, R27, R29, R3, R30, R31, R32, R33, R34, R35, R4, R6, R7, R8, R9: value R -> 10k
- R12, R20, R28, R5: value R -> 1k
Changed lines of the file:
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@@
       (drillshape 0)
       (scaleselection 1)
-      (outputdirectory ""))
+      (outputdirectory "plot"))
   )
   (net 0 "")
@@
       (effects (font (size 1 1) (thickness 0.15)))
     )
-    (fp_text value R (at 0 1.65 90) (layer F.Fab) hide
+    (fp_text value 10k (at 0 1.65 90) (layer F.Fab) hide
       (effects (font (size 1 1) (thickness 0.15)))
     )
@@
       (effects (font (size 1 1) (thickness 0.15)))
     )
-    (fp_text value R (at 0 1.65 90) (layer F.Fab) hide
+    (fp_text value 10k (at 0 1.65 90) (layer F.Fab) hide
       (effects (font (size 1 1) (thickness 0.15)))
     )
@@
       (effects (font (size 1 1) (thickness 0.15)))
     )
-    (fp_text value R (at 0 1.65 90) (layer F.Fab) hide
+    (fp_text value 1k (at 0 1.65 90) (layer F.Fab) hide
       (effects (font (size 1 1) (thickness 0.15)))
     )
@@
       (effects (font (size 1 1) (thickness 0.15)))
     )
-    (fp_text value R (at 0 1.65 90) (layer F.Fab) hide
+    (fp_text value 1k (at 0 1.65 90) (layer F.Fab) hide
       (effects (font (size 1 1) (thickness 0.15)))
     )
@@
       (effects (font (size 1 1) (thickness 0.15)))
     )
-    (fp_text value R (at 0 1.65 90) (layer F.Fab) hide
+    (fp_text value 1k (at 0 1.65 90) (layer F.Fab) hide
       (effects (font (size 1 1) (thickness 0.15)))
     )
@@
       (effects (font (size 1 1) (thickness 0.15)))
     )
-    (fp_text value R (at 0 1.65 90) (layer F.Fab) hide
+    (fp_text value 1k (at 0 1.65 90) (layer F.Fab) hide
       (effects (font (size 1 1) (thickness 0.15)))
     )
@@
       (effects (font (size 1 1) (thickness 0.15)))
     )
-    (fp_text value R (at 0 1.65) (layer F.Fab) hide
+    (fp_text value 10k (at 0 1.65) (layer F.Fab) hide
       (effects (font (size 1 1) (thickness 0.15)))
     )
@@
       (effects (font (size 1 1) (thickness 0.15)))
     )
-    (fp_text value R (at 0 1.65 90) (layer F.Fab) hide
+    (fp_text value 10k (at 0 1.65 90) (layer F.Fab) hide
       (effects (font (size 1 1) (thickness 0.15)))
     )
@@
       (effects (font (size 1 1) (thickness 0.15)))
     )
-    (fp_text value R (at 0 1.65 90) (layer F.Fab) hide
+    (fp_text value 10k (at 0 1.65 90) (layer F.Fab) hide
       (effects (font (size 1 1) (thickness 0.15)))
     )
@@
       (effects (font (size 1 1) (thickness 0.15)))
     )
-    (fp_text value R (at 0 1.65 90) (layer F.Fab) hide
+    (fp_text value 10k (at 0 1.65 90) (layer F.Fab) hide
       (effects (font (size 1 1) (thickness 0.15)))
     )
@@
       (effects (font (size 1 1) (thickness 0.15)))
     )
-    (fp_text value R (at 0 1.65 90) (layer F.Fab) hide
+    (fp_text value 10k (at 0 1.65 90) (layer F.Fab) hide
       (effects (font (size 1 1) (thickness 0.15)))
     )
@@
       (effects (font (size 1 1) (thickness 0.15)))
     )
-    (fp_text value R (at 0 1.65 90) (layer F.Fab) hide
+    (fp_text value 10k (at 0 1.65 90) (layer F.Fab) hide
       (effects (font (size 1 1) (thickness 0.15)))
     )
@@
       (effects (font (size 1 1) (thickness 0.15)))
     )
-    (fp_text value R (at 0 1.65 90) (layer F.Fab) hide
+    (fp_text value 10k (at 0 1.65 90) (layer F.Fab) hide
       (effects (font (size 1 1) (thickness 0.15)))
     )
@@
       (effects (font (size 1 1) (thickness 0.15)))
     )
-    (fp_text value R (at 0 1.65 90) (layer F.Fab) hide
+    (fp_text value 10k (at 0 1.65 90) (layer F.Fab) hide
       (effects (font (size 1 1) (thickness 0.15)))
     )
@@
       (effects (font (size 1 1) (thickness 0.15)))
     )
-    (fp_text value R (at 0 1.65 90) (layer F.Fab) hide
+    (fp_text value 10k (at 0 1.65 90) (layer F.Fab) hide
       (effects (font (size 1 1) (thickness 0.15)))
     )
@@
       (effects (font (size 1 1) (thickness 0.15)))
     )
-    (fp_text value R (at 0 1.65 90) (layer F.Fab) hide
+    (fp_text value 10k (at 0 1.65 90) (layer F.Fab) hide
       (effects (font (size 1 1) (thickness 0.15)))
     )
@@
       (effects (font (size 1 1) (thickness 0.15)))
     )
-    (fp_text value R (at 0 1.65 90) (layer F.Fab) hide
+    (fp_text value 10k (at 0 1.65 90) (layer F.Fab) hide
       (effects (font (size 1 1) (thickness 0.15)))
     )
@@
       (effects (font (size 1 1) (thickness 0.15)))
     )
-    (fp_text value R (at 0 1.65 90) (layer F.Fab) hide
+    (fp_text value 10k (at 0 1.65 90) (layer F.Fab) hide
       (effects (font (size 1 1) (thickness 0.15)))
     )
@@
       (effects (font (size 1 1) (thickness 0.15)))
     )
-    (fp_text value R (at 0 1.65 90) (layer F.Fab) hide
+    (fp_text value 10k (at 0 1.65 90) (layer F.Fab) hide
       (effects (font (size 1 1) (thickness 0.15)))
     )
@@
       (effects (font (size 1 1) (thickness 0.15)))
     )
-    (fp_text value R (at 0 1.65 90) (layer F.Fab) hide
+    (fp_text value 10k (at 0 1.65 90) (layer F.Fab) hide
       (effects (font (size 1 1) (thickness 0.15)))
     )
@@
       (effects (font (size 1 1) (thickness 0.15)))
     )
-    (fp_text value R (at 0 1.65 90) (layer F.Fab) hide
+    (fp_text value 10k (at 0 1.65 90) (layer F.Fab) hide
       (effects (font (size 1 1) (thickness 0.15)))
     )
@@
       (effects (font (size 1 1) (thickness 0.15)))
     )
-    (fp_text value R (at 0 1.65 90) (layer F.Fab) hide
+    (fp_text value 10k (at 0 1.65 90) (layer F.Fab) hide
       (effects (font (size 1 1) (thickness 0.15)))
     )
@@
       (effects (font (size 1 1) (thickness 0.15)))
     )
-    (fp_text value R (at 0 1.65 90) (layer F.Fab) hide
+    (fp_text value 10k (at 0 1.65 90) (layer F.Fab) hide
       (effects (font (size 1 1) (thickness 0.15)))
     )
@@
       (effects (font (size 1 1) (thickness 0.15)))
     )
-    (fp_text value R (at 0 1.65 90) (layer F.Fab) hide
+    (fp_text value 10k (at 0 1.65 90) (layer F.Fab) hide
       (effects (font (size 1 1) (thickness 0.15)))
     )
@@
       (effects (font (size 1 1) (thickness 0.15)))
     )
-    (fp_text value R (at 0 1.65 90) (layer F.Fab) hide
+    (fp_text value 10k (at 0 1.65 90) (layer F.Fab) hide
       (effects (font (size 1 1) (thickness 0.15)))
     )
@@
       (effects (font (size 1 1) (thickness 0.15)))
     )
-    (fp_text value R (at 0 1.65 90) (layer F.Fab) hide
+    (fp_text value 10k (at 0 1.65 90) (layer F.Fab) hide
       (effects (font (size 1 1) (thickness 0.15)))
     )
@@
       (effects (font (size 1 1) (thickness 0.15)))
     )
-    (fp_text value R (at 0 1.65 90) (layer F.Fab) hide
+    (fp_text value 10k (at 0 1.65 90) (layer F.Fab) hide
       (effects (font (size 1 1) (thickness 0.15)))
     )
@@
       (effects (font (size 1 1) (thickness 0.15)))
     )
-    (fp_text value R (at 0 1.65 90) (layer F.Fab) hide
+    (fp_text value 10k (at 0 1.65 90) (layer F.Fab) hide
       (effects (font (size 1 1) (thickness 0.15)))
     )
@@
       (effects (font (size 1 1) (thickness 0.15)))
     )
-    (fp_text value R (at 0 1.65 90) (layer F.Fab) hide
+    (fp_text value 10k (at 0 1.65 90) (layer F.Fab) hide
       (effects (font (size 1 1) (thickness 0.15)))
     )
@@
       (effects (font (size 1 1) (thickness 0.15)))
     )
-    (fp_text value R (at 0 1.65 90) (layer F.Fab) hide
+    (fp_text value 10k (at 0 1.65 90) (layer F.Fab) hide
       (effects (font (size 1 1) (thickness 0.15)))
     )
@@
       (effects (font (size 1 1) (thickness 0.15)))
     )
-    (fp_text value R (at 0 1.65 90) (layer F.Fab) hide
+    (fp_text value 10k (at 0 1.65 90) (layer F.Fab) hide
       (effects (font (size 1 1) (thickness 0.15)))
     )
@@
       (effects (font (size 1 1) (thickness 0.15)))
     )
-    (fp_text value R (at 0 1.65) (layer F.Fab) hide
+    (fp_text value 10k (at 0 1.65) (layer F.Fab) hide
       (effects (font (size 1 1) (thickness 0.15)))
     )
@@
       (effects (font (size 1 1) (thickness 0.15)))
     )
-    (fp_text value R (at 0 1.65) (layer F.Fab) hide
+    (fp_text value 10k (at 0 1.65) (layer F.Fab) hide
       (effects (font (size 1 1) (thickness 0.15)))
     )
@@
       (effects (font (size 1 1) (thickness 0.15)))
     )
-    (fp_text value R (at 0 1.65 90) (layer F.Fab) hide
+    (fp_text value 10k (at 0 1.65 90) (layer F.Fab) hide
       (effects (font (size 1 1) (thickness 0.15)))
     )
@@
       (effects (font (size 1 1) (thickness 0.15)))
     )
-    (fp_text value R (at 0 1.65 90) (layer F.Fab) hide
+    (fp_text value 10k (at 0 1.65 90) (layer F.Fab) hide
       (effects (font (size 1 1) (thickness 0.15)))
     )
@@
       (effects (font (size 1 1) (thickness 0.15)))
     )
-    (fp_text value C (at 0 1.65 90) (layer F.Fab) hide
+    (fp_text value 0.1u (at 0 1.65 90) (layer F.Fab) hide
       (effects (font (size 1 1) (thickness 0.15)))
     )
