File: pcb/control/control.kicad_pcb (KiCad board)
At the start: 2 copper layers, 221 parts, among them J1 Top, J2 Bottom, Q1 2N7002, Q10 2N7002, Q100 2N7002, Q101 2N7002, Q102 2N7002, Q103 2N7002, Q104 2N7002, Q105 2N7002, Q106 2N7002, Q107 2N7002, Q108 2N7002, Q109 2N7002, Q11 2N7002, Q110 2N7002, Q111 2N7002, Q112 2N7002, Q113 2N7002, Q114 2N7002, Q115 2N7002, Q116 2N7002, Q117 2N7002, Q118 2N7002, Q119 2N7002, Q12 2N7002, Q120 2N7002, Q121 2N7002, Q122 2N7002, Q123 2N7002, Q124 2N7002, Q125 2N7002, Q126 2N7002, Q127 2N7002, Q128 2N7002, Q129 2N7002, Q13 2N7002, Q130 2N7002, Q131 2N7002, Q132 2N7002, Q133 2N7002, Q134 2N7002, Q135 2N7002, Q136 2N7002, Q137 2N7002, Q138 2N7002, Q139 2N7002, Q14 2N7002, Q140 2N7002, Q141 2N7002, Q142 2N7002, Q143 2N7002, Q144 2N7002, Q15 2N7002, Q16 2N7002, Q17 2N7002, Q18 2N7002, Q19 2N7002, Q2 2N7002, Q20 2N7002, Q21 2N7002, Q22 2N7002, Q23 2N7002, Q24 2N7002, Q25 2N7002, Q26 2N7002, Q27 2N7002, Q28 2N7002, Q29 2N7002, Q3 2N7002, Q30 2N7002, Q31 2N7002, Q32 2N7002, Q33 2N7002, Q34 2N7002, Q35 2N7002, Q36 2N7002, Q37 2N7002, Q38 2N7002, Q39 2N7002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

Commit message: New design
Parts:
- removed D1, D2, D3, D4, D5, D6: LED, LED_SMD:LED_0805_2012Metric_Pad1.15x1.40mm_HandSolder
- removed J2: Bottom, Connector_Harwin:Harwin_M20-89020xx_1x20_P2.54mm_Horizontal
- removed Q100, Q101, Q102, Q103, Q104, Q105, Q106, Q107, Q108, Q109, Q110, Q111, Q112, Q113, Q114, Q115, Q116, Q117, Q118, Q119, Q120, Q121, Q122, Q123, Q124, Q125, Q126, Q127, Q128, Q129, Q130, Q131, Q132, Q133, Q134, Q135, Q136, Q137, Q138, Q139, Q140, Q141, Q142, Q143, Q144, Q59, Q60, Q61, Q62, Q63, Q64, Q65, Q66, Q67, Q68, Q69, Q70, Q71, Q72, Q73, Q74, Q75, Q76, Q77, Q78, Q79, Q80, Q81, Q82, Q83, Q84, Q85, Q86, Q87, Q88, Q89, Q90, Q91, Q92, Q93, Q94, Q95, Q96, Q97, Q98, Q99: 2N7002, Package_TO_SOT_SMD:SOT-23
- removed the Q11 at (193.0, 129.6)
- removed the Q3 at (179.1, 132.3)
- removed the Q4 at (193.3, 120.5)
- removed the Q5 at (183.8, 129.4)
- removed the Q6 at (188.6, 126.4)
- removed the Q7 at (193.3, 125.1)
- removed the Q8 at (183.5, 133.9)
- removed the R1 at (194.7, 155.8)
- removed the R2 at (169.0, 73.3)
- removed R24, R25, R26, R27, R28, R29, R30, R31, R32, R33, R34, R35, R36, R37, R38, R39, R40, R41, R42, R43, R44, R45, R46, R47, R48, R49, R50, R51, R52, R53, R54, R55, R56, R57, R58, R59, R60, R61, R62, R63, R64, R65, R66, R67, R68, R69: R, Resistor_SMD:R_0805_2012Metric_Pad1.15x1.40mm_HandSolder
- removed the R3 at (188.7, 122.7)
- removed the R4 at (184.0, 125.6)
- added Q39: 2N7002, Package_TO_SOT_SMD:SOT-23_Handsoldering, F.Cu at (138.0, 119.0)
- added Q40: 2N7002, Package_TO_SOT_SMD:SOT-23_Handsoldering, F.Cu at (150.9, 109.9)
- added Q41: 2N7002, Package_TO_SOT_SMD:SOT-23_Handsoldering, F.Cu at (150.9, 114.5)
- added Q42: 2N7002, Package_TO_SOT_SMD:SOT-23_Handsoldering, F.Cu at (163.8, 119.0)
- added Q47: 2N7002, Package_TO_SOT_SMD:SOT-23_Handsoldering, F.Cu at (183.2, 105.3)
- added Q49: 2N7002, Package_TO_SOT_SMD:SOT-23_Handsoldering, F.Cu at (170.2, 100.8)
- added Q51: 2N7002, Package_TO_SOT_SMD:SOT-23_Handsoldering, F.Cu at (176.7, 96.2)
- added R20: R, Resistor_SMD:R_0805_2012Metric_Pad1.15x1.40mm_HandSolder, F.Cu at (182.3, 109.1)
- added R21: R, Resistor_SMD:R_0805_2012Metric_Pad1.15x1.40mm_HandSolder, F.Cu at (188.8, 101.3)
- J1: value Top -> Conn_02x32_Odd_Even; footprint Connector_Harwin:Harwin_M20-89020xx_1x20_P2.54mm_Horizontal -> Connector_PinHeader_2.54mm:PinHeader_2x32_P2.54mm_Horizontal
- Q1, Q10, Q12, Q13, Q14, Q15, Q16, Q17, Q18, Q19, Q2, Q20, Q21, Q22, Q23, Q24, Q25, Q26, Q27, Q28, Q29, Q30, Q31, Q32, Q33, Q34, Q35, Q36, Q37, Q38, Q43, Q44, Q45, Q46, Q48, Q50, Q52, Q53, Q54, Q55, Q56, Q57, Q58, Q9: footprint Package_TO_SOT_SMD:SOT-23 -> Package_TO_SOT_SMD:SOT-23_Handsoldering
- Q11: renamed from Q51; footprint Package_TO_SOT_SMD:SOT-23 -> Package_TO_SOT_SMD:SOT-23_Handsoldering
- Q3: renamed from Q39; footprint Package_TO_SOT_SMD:SOT-23 -> Package_TO_SOT_SMD:SOT-23_Handsoldering
- Q4: renamed from Q40; footprint Package_TO_SOT_SMD:SOT-23 -> Package_TO_SOT_SMD:SOT-23_Handsoldering
- Q5: renamed from Q41; footprint Package_TO_SOT_SMD:SOT-23 -> Package_TO_SOT_SMD:SOT-23_Handsoldering
- Q6: renamed from Q42; footprint Package_TO_SOT_SMD:SOT-23 -> Package_TO_SOT_SMD:SOT-23_Handsoldering
- Q7: renamed from Q47; footprint Package_TO_SOT_SMD:SOT-23 -> Package_TO_SOT_SMD:SOT-23_Handsoldering
- Q8: renamed from Q49; footprint Package_TO_SOT_SMD:SOT-23 -> Package_TO_SOT_SMD:SOT-23_Handsoldering
- moved Q1 99.8 mm to (136.5, 83.1)
- moved R18 93.0 mm to (188.8, 98.4)
- moved R19 87.4 mm to (188.8, 104.3)
- moved Q27 77.3 mm to (183.2, 100.8)
- moved R17 75.5 mm to (175.8, 118.2)
- moved R16 75.1 mm to (170.4, 122.8)
- moved R15 71.1 mm to (165.7, 122.8)
- moved R6 69.7 mm to (131.9, 79.3)
- moved Q13 69.5 mm to (150.5, 74.2)
- moved Q37 66.3 mm to (176.7, 114.5)
- moved Q12 66.2 mm to (154.9, 74.2)
- moved Q43 65.0 mm to (176.7, 109.9)
- moved Q45 64.5 mm to (170.2, 96.2)
- moved Q50 62.9 mm to (163.8, 100.8)
- moved R12 62.5 mm to (188.8, 95.5)
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- renumbered R20 to R1, R21 to R2, R22 to R3, R23 to R4
Connections:
- J1 pad 1: VCC -> GND
- J1 pad 10: PIN_X -> ~S1
- J1 pad 11: WRP -> RDM
- J1 pad 12: WROUT -> (no net)
- J1 pad 13: RDSW_DBUS -> WRM
- J1 pad 14: HALT -> ~S2
- J1 pad 15: CLK2 -> (no net)
- J1 pad 16: CLK1 -> (no net)
- J1 pad 17: RST -> XLIN_DBUS
- J1 pad 18: F -> ~S3
- J1 pad 19: FIN -> STATE_ALU
- J1 pad 2: PIN_NEXT -> GND
- J1 pad 20: GND -> (no net)
- J1 pad 3: RDX_ABUS -> INCP_CLK
- J1 pad 4: XHIN_ABUS -> S0
- J1 pad 5: XHIN_DBUS -> ~WRP
- J1 pad 6: WRX -> ~S0
- J1 pad 7: WRA -> RDP_ABUS
- J1 pad 8: RDA_DBUS -> S1
- J1 pad 9: PIN_NEXT -> (no net)
- Q1 pad 1: Net-(Q1-Pad1) -> OP2
- Q1 pad 3: ~F -> ~STATE_LOAD
- Q10 pad 1: ~S1 -> XLIN_DBUS
- Q10 pad 3: Net-(Q10-Pad3) -> STATE_ALU
- Q11 pad 1: ~OP5 -> ~S2
- Q11 pad 2: GND -> Net-(Q11-Pad2)
- Q11 pad 3: Net-(Q47-Pad2) -> Net-(Q11-Pad3)
- Q12 pad 1: S1 -> ~OP5
- Q13 pad 1: RDX_ABUS -> ~S3
- Q13 pad 3: PIN_NEXT -> Net-(Q11-Pad2)
- Q14 pad 1: ~STATE_EXEC -> RDX_ABUS
- Q14 pad 3: PIN_X -> RDP_ABUS
- Q15 pad 1: Net-(Q15-Pad1) -> RDX_ABUS
- Q15 pad 2: Net-(Q15-Pad2) -> GND
- Q15 pad 3: ~S0 -> WRO
- Q16 pad 1: S0 -> ~WS
- Q16 pad 3: ~S0 -> WRO
- Q17 pad 1: ~S0 -> RDX_ABUS
- Q17 pad 3: S0 -> XHIN_ZERO
- Q18 pad 1: Net-(Q18-Pad1) -> ~DBUS6
- Q18 pad 2: Net-(Q15-Pad2) -> GND
- Q18 pad 3: S0 -> XHIN_ZERO
- Q19 pad 1: RST -> RDX_ABUS
- Q19 pad 3: S0 -> XHIN_P
- Q2 pad 1: CLK1 -> OP1
- Q2 pad 2: GND -> Net-(Q2-Pad2)
- Q2 pad 3: ~CLK1 -> ~STATE_DEREF
- Q20 pad 1: ~S0 -> DBUS6
- Q20 pad 2: Net-(Q20-Pad2) -> GND
- Q20 pad 3: Net-(Q18-Pad1) -> XHIN_P
- Q21 pad 1: Net-(Q15-Pad1) -> OP5
- Q21 pad 2: GND -> Net-(Q21-Pad2)
- Q21 pad 3: Net-(Q18-Pad1) -> RUN
- Q22 pad 1: Net-(Q18-Pad1) -> ~OP4
- Q22 pad 2: GND -> Net-(Q22-Pad2)
- Q22 pad 3: Net-(Q15-Pad1) -> Net-(Q21-Pad2)
- Q23 pad 1: Net-(Q23-Pad1) -> ~STATE_LOAD
- Q23 pad 2: Net-(Q20-Pad2) -> Net-(Q23-Pad2)
- Q23 pad 3: Net-(Q15-Pad1) -> XHIN_DBUS
- Q24 pad 1: CLK2 -> OP3
- Q24 pad 2: GND -> Net-(Q24-Pad2)
- Q24 pad 3: Net-(Q15-Pad2) -> Net-(Q22-Pad2)
- Q25 pad 1: ~S0 -> ~STATE_DEREF
- Q25 pad 3: Net-(Q23-Pad1) -> Net-(Q23-Pad2)
- Q26 pad 1: CLK1 -> WS
- Q26 pad 2: GND -> Net-(Q26-Pad2)
- Q26 pad 3: Net-(Q20-Pad2) -> Net-(Q24-Pad2)
- Q27 pad 1: Net-(Q27-Pad1) -> RDA_DBUS
- Q27 pad 2: Net-(Q27-Pad2) -> GND
- Q27 pad 3: ~S1 -> Net-(Q26-Pad2)
- Q28 pad 1: S1 -> XLIN_DBUS
- Q28 pad 3: ~S1 -> WRA
- Q29 pad 1: ~S1 -> ~WS
- Q29 pad 3: S1 -> WRA
- Q3 pad 1: ~OP3 -> ~S0
- Q3 pad 3: ~FUNC0 -> RDX_ABUS
- Q30 pad 1: Net-(Q30-Pad1) -> RDX_ABUS
- Q30 pad 2: Net-(Q27-Pad2) -> INCP_DB
- Q30 pad 3: S1 -> INCP_CLK
- Q31 pad 1: RST -> ~WS
- Q31 pad 2: GND -> INCP_DB
- Q31 pad 3: S1 -> INCP_CLK
- Q32 pad 1: NEXT_S1 -> XLIN_DBUS
- Q32 pad 3: Net-(Q30-Pad1) -> WRF
- Q33 pad 1: Net-(Q27-Pad1) -> ~WS
- Q33 pad 3: Net-(Q30-Pad1) -> WRF
- Q34 pad 1: Net-(Q30-Pad1) -> RDM
- Q34 pad 3: Net-(Q27-Pad1) -> Net-(Q32-Pad2)
- Q35 pad 1: Net-(Q35-Pad1) -> OP5
- Q35 pad 2: Net-(Q32-Pad2) -> GND
- Q35 pad 3: Net-(Q27-Pad1) -> Net-(Q32-Pad2)
- Q36 pad 1: CLK2 -> DBUS6
- Q36 pad 3: Net-(Q27-Pad2) -> ~DBUS6
- Q37 pad 1: NEXT_S1 -> WS
- Q37 pad 3: Net-(Q35-Pad1) -> ~WS
- Q38 pad 1: CLK1 -> XLIN_DBUS
- Q38 pad 2: GND -> Net-(Q38-Pad2)
- Q38 pad 3: Net-(Q32-Pad2) -> WRX
- Q4 pad 1: OP3 -> S0
- Q4 pad 3: ~FUNC1 -> Net-(Q1-Pad2)
- Q43 pad 1: ~OP3 -> XLIN_DBUS
- Q43 pad 2: Net-(Q43-Pad2) -> Net-(Q42-Pad2)
- Q43 pad 3: ~FUNC4 -> FOUT
- Q44 pad 1: OP3 -> RDX_ABUS
- Q44 pad 2: Net-(Q43-Pad2) -> GND
- Q44 pad 3: ~FUNC5 -> Net-(Q41-Pad2)
- Q45 pad 1: ~OP3 -> ~WS
- Q45 pad 3: ~FUNC6 -> ~WRP
- Q46 pad 1: OP3 -> OP4
- Q46 pad 2: Net-(Q45-Pad2) -> GND
- Q46 pad 3: ~FUNC7 -> Net-(Q42-Pad2)
- Q48 pad 1: OP4 -> OP3
- Q5 pad 1: ~OP3 -> ~S0
- Q5 pad 3: ~FUNC2 -> Net-(Q2-Pad2)
- Q50 pad 1: ~OP4 -> OP4
- Q50 pad 2: Net-(Q48-Pad2) -> Net-(Q50-Pad2)
- Q50 pad 3: Net-(Q43-Pad2) -> Net-(Q48-Pad2)
- Q52 pad 2: GND -> Net-(Q52-Pad2)
- Q52 pad 3: Net-(Q48-Pad2) -> Net-(Q50-Pad2)
- Q53 pad 1: ~FUNC0 -> RDA_DBUS
- Q53 pad 3: FUNC0 -> Net-(Q52-Pad2)
- Q54 pad 1: ~FUNC1 -> ~OP5
- Q54 pad 3: FUNC1 -> Net-(Q51-Pad2)
- Q55 pad 1: ~FUNC2 -> OP4
- Q55 pad 3: AND -> Net-(Q51-Pad2)
- Q56 pad 1: ~FUNC3 -> OP3
- Q56 pad 3: FUNC3 -> Net-(Q51-Pad2)
- Q57 pad 1: ~FUNC4 -> RDM
- Q57 pad 3: FUNC4 -> Net-(Q51-Pad2)
- Q58 pad 1: ~FUNC5 -> ~WS
- Q58 pad 3: ADD -> Net-(Q51-Pad2)
- Q6 pad 1: OP3 -> S0
- Q6 pad 3: ~FUNC3 -> RDM
- Q7 pad 1: OP4 -> S1
- Q7 pad 2: Net-(Q47-Pad2) -> Net-(Q11-Pad3)
- Q8 pad 1: ~OP4 -> ~S1
- Q8 pad 2: Net-(Q47-Pad2) -> Net-(Q11-Pad3)
- Q9 pad 1: S0 -> Net-(Q11-Pad3)
- Q9 pad 3: ~STATE_EXEC -> XLIN_DBUS
- R1 pad 2: ~FUNC0 -> RDX_ABUS
- R10 pad 2: ~S0 -> XHIN_ZERO
- R11 pad 2: S0 -> XHIN_P
- R12 pad 2: Net-(Q18-Pad1) -> XHIN_DBUS
- R13 pad 2: Net-(Q15-Pad1) -> WRA
- R14 pad 2: Net-(Q23-Pad1) -> INCP_CLK
- R15 pad 2: ~S1 -> WRF
- R16 pad 2: S1 -> ~DBUS6
- R17 pad 2: Net-(Q30-Pad1) -> ~WS
- R18 pad 2: Net-(Q27-Pad1) -> WRX
- R19 pad 2: Net-(Q35-Pad1) -> FOUT
- R2 pad 2: ~FUNC1 -> ~STATE_LOAD
- R3 pad 2: ~FUNC2 -> ~STATE_DEREF
- R4 pad 2: ~FUNC3 -> RDM
- R5 pad 2: NEXT_S1 -> XLIN_DBUS
- R6 pad 2: ~STATE_DEREF -> STATE_ALU
- R7 pad 2: ~STATE_EXEC -> Net-(Q11-Pad3)
- R8 pad 2: PIN_NEXT -> RDP_ABUS
- R9 pad 2: PIN_X -> WRO

Commit message: Updates
Parts:
- moved R8 101.9 mm to (138.5, 91.0), turned to 270 degrees
- moved Q14 100.6 mm to (134.5, 91.0)
- moved R7 97.8 mm to (118.5, 107.5), turned to 270 degrees
- moved R5 80.5 mm to (138.5, 118.5), turned to 270 degrees
- moved Q9 79.7 mm to (134.5, 118.5)
- moved Q53 67.2 mm to (153.5, 85.5)
- moved Q47 65.7 mm to (122.5, 80.0)
- moved Q46 63.8 mm to (116.5, 80.0)
- moved Q54 60.3 mm to (104.5, 85.5)
- moved Q55 58.6 mm to (110.5, 85.5)
- moved Q56 57.3 mm to (116.5, 85.5)
- moved Q57 56.3 mm to (122.5, 85.5)
- moved R19 55.8 mm to (138.5, 80.0), turned to 270 degrees
- moved R21 52.7 mm to (138.5, 85.5), turned to 270 degrees
- moved Q42 52.6 mm to (128.5, 80.0)
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Routing:
- net VCC: track 0.00 -> 668.4 mm, vias 0 -> 2
- net GND: track 0.00 -> 316.2 mm, vias 0 -> 22
- net OP3: track 0.00 -> 184.6 mm, vias 0 -> 6
- net ~WS: track 0.00 -> 172.9 mm, vias 0 -> 9
- net OP5: track 0.00 -> 166.5 mm, vias 0 -> 6
- net XLIN_DBUS: track 0.00 -> 164.3 mm, vias 0 -> 8
- net RDM: track 0.00 -> 155.4 mm, vias 0 -> 7
- net RDX_ABUS: track 0.00 -> 153.1 mm, vias 0 -> 8
- net RUN: track 0.00 -> 138.9 mm, vias 0 -> 3
- net OP4: track 0.00 -> 135.3 mm, vias 0 -> 3
- net ~OP4: track 0.00 -> 133.7 mm, vias 0 -> 3
- net WS: track 0.00 -> 131.9 mm, vias 0 -> 4
- net S0: track 0.00 -> 122.2 mm, vias 0 -> 4
- net XHIN_P: track 0.00 -> 116.6 mm, vias 0 -> 3
- net WRX: track 0.00 -> 114.9 mm, vias 0 -> 3
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- added copper zone on B.Cu, net GND
- added copper zone on F.Cu, net GND
Other:
- board outline added: 100 x 75 mm
- board text added: "+ +"
- board text added: "ALU"
- board text added: "FOUT"
- board text added: "INCP_CLK"
- board text added: "RDM"
- board text added: "RDP"
- board text added: "RDX"
- board text added: "WRA"
- board text added: "WRF"
- board text added: "WRM"
- board text added: "WRO"
- board text added: "WRX"
- board text added: "XHIN_DBUS"
- board text added: "XHIN_P"
- board text added: "XHIN_ZERO"
- board text added: "XLIN_DBUS"
- board text added: "~DEREF"
- board text added: "~HALT"
- board text added: "~LOAD"
- board text added: "~WRP"
- board text added: "~WS"

Commit message: Updates.
Parts:
- added Q59: 2N7002, Package_TO_SOT_SMD:SOT-23_Handsoldering, F.Cu at (110.5, 80.0)
- added Q60: 2N7002, Package_TO_SOT_SMD:SOT-23_Handsoldering, F.Cu at (104.5, 80.0)
Connections:
- J1 pad 11: RDM -> WS
- J1 pad 13: WRM -> RUN
- J1 pad 15: (no net) -> INCP_DB
- J1 pad 17: XLIN_DBUS -> (no net)
- J1 pad 19: STATE_ALU -> RDM
- J1 pad 21: (no net) -> WRM
- J1 pad 23: ~ALU_COUT -> (no net)
- J1 pad 25: (no net) -> XLIN_DBUS
- J1 pad 26: (no net) -> DBUS6
- J1 pad 27: (no net) -> STATE_ALU
- J1 pad 29: ~DEP_SW -> (no net)
- J1 pad 31: INCP_DB -> ~DEP_SW
- J1 pad 35: WRA -> ~X0
- J1 pad 36: WRO -> (no net)
- J1 pad 37: RDA_DBUS -> (no net)
- J1 pad 38: DBUS6 -> WRO
- J1 pad 41: (no net) -> WRA
- J1 pad 43: (no net) -> RDA_DBUS
- J1 pad 54: (no net) -> ~OP3
- J1 pad 59: WS -> (no net)
- J1 pad 61: RUN -> ~ALU_COUT
- Q46 pad 2: GND -> Net-(Q46-Pad2)
Routing:
- net ~X0: track 0.00 -> 109.1 mm, vias 0 -> 1
- net ~OP3: track 0.00 -> 89.3 mm, vias 0 -> 3
- net WS: track 131.9 -> 193.2 mm, vias 4 -> 6
- net RUN: track 138.9 -> 83.8 mm
- net RDM: track 155.4 -> 123.1 mm, vias 7 -> 6
- net DBUS6: track 103.1 -> 72.3 mm
- net INCP_DB: track 59.1 -> 40.6 mm
- net ~ALU_COUT: track 100.8 -> 82.8 mm, vias 2 -> 1
- net RDA_DBUS: track 80.0 -> 92.4 mm
- net STATE_ALU: track 78.0 -> 66.6 mm
- net XLIN_DBUS: track 164.3 -> 175.0 mm, vias 8 -> 9
- net Net-(Q46-Pad2): track 0.00 -> 9.39 mm
- net WRM: track 93.9 -> 85.1 mm
- net WRA: track 65.5 -> 71.7 mm
- net VCC: track 668.4 -> 673.6 mm
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Other:
- board text added: "Q2 Control v0"

Commit message: Signed immediates.
Parts:
- added Q61: 2N7002, Package_TO_SOT_SMD:SOT-23_Handsoldering, F.Cu at (177.5, 102.0)
- moved R16 11.0 mm to (161.0, 102.0)
- moved Q17 6.00 mm to (171.5, 102.0)
- moved Q36 2.50 mm to (165.5, 102.0)
Connections:
- J1 pad 24: (no net) -> DBUS5
- Q18 pad 2: GND -> Net-(Q18-Pad2)
Routing:
- net DBUS5: track 0.00 -> 61.5 mm, vias 0 -> 3
- net GND: track 313.7 -> 331.4 mm, vias 22 -> 25
- net VCC: track 673.6 -> 684.7 mm
- net ~DBUS6: track 13.7 -> 23.3 mm
- net XHIN_ZERO: track 105.9 -> 112.5 mm
- net Net-(Q18-Pad2): track 0.00 -> 3.39 mm
- net RDX_ABUS: track 153.1 -> 155.2 mm
- net XHIN_DBUS: track 114.8 -> 113.2 mm, vias 3 -> 1
- net DBUS6: track 72.3 -> 71.0 mm
Other:
- outline, holes or cut-outs redrawn
- board text added: "- -"
- board text added: "HD O4"
- board text added: "HP ~O4~"
- board text added: "HS O3"
- board text added: "HZ ~O3~"
- board text added: "IC S0"
- board text added: "IP S3"
- board text added: "LD D6"
- board text added: "LS NC"
- board text added: "NC D5"
- board text added: "NC O0"
- board text added: "NC O5"
- board text added: "NC WF"
- board text added: "NC WO"
- board text added: "NC ~F~"
- board text added: "NC ~O1~"
- board text added: "NC ~S1~"
- board text added: "NC ~S3~"
- board text added: "RA O1"
- board text added: "RM NC"
- board text added: "RN ~S2~"
- board text added: "RP S1"
- board text added: "RX O2"
- board text added: "WA ~O0~"
- board text added: "WM NC"
- board text added: "WS S2"
- board text added: "WX ~O2~"
- board text added: "~CO~ ~O5~"
- board text added: "~DS~ FO"
- board text added: "~WP~ ~S0~"
- board text added: "~X0~ NC"

Commit message: No load flag.
Parts:
- removed the Q21 at (183.5, 80.0)
- removed the Q22 at (177.5, 80.0)
- removed the Q24 at (171.5, 80.0)
- removed the Q26 at (165.5, 80.0)
- removed the Q27 at (159.5, 80.0)
- removed Q61: 2N7002, Package_TO_SOT_SMD:SOT-23_Handsoldering
- added Q12: 2N7002, Package_TO_SOT_SMD:SOT-23_Handsoldering, F.Cu at (128.5, 124.0)
- added Q15: 2N7002, Package_TO_SOT_SMD:SOT-23_Handsoldering, F.Cu at (122.5, 124.0)
- renumbered Q12 to Q13, Q13 to Q14, Q14 to Q16, Q15 to Q17, Q16 to Q18, Q17 to Q19, Q18 to Q20, Q23 to Q21, Q19 to Q22, Q20 to Q23, Q25 to Q24, Q28 to Q25, Q29 to Q26, Q30 to Q27, Q31 to Q28, Q36 to Q29, Q37 to Q30, Q32 to Q31, Q33 to Q32, Q38 to Q33, Q39 to Q34, Q45 to Q35, Q40 to Q36, Q34 to Q37, Q35 to Q38, Q41 to Q39, Q48 to Q40, Q49 to Q41, Q44 to Q42, Q50 to Q43, Q42 to Q44, Q43 to Q45, Q52 to Q46, Q53 to Q47, Q46 to Q48, Q47 to Q49, Q51 to Q50, Q59 to Q51, Q60 to Q52, Q54 to Q53, Q55 to Q54, Q56 to Q55, Q57 to Q56, Q58 to Q57, R12 to R11, R11 to R12, R16 to R15, R17 to R16, R15 to R17, R20 to R19, R19 to R20
Connections:
- net ~DBUS6 renamed ~DBUS7
- J1 pad 13: RUN -> (no net)
- J1 pad 24: DBUS5 -> DBUS7
- J1 pad 26: DBUS6 -> (no net)
- J1 pad 44: OP1 -> (no net)
- J1 pad 52: OP3 -> (no net)
- Q1 pad 1: OP2 -> ~OP5
- Q2 pad 1: OP1 -> OP2
- Q20 pad 2: Net-(Q18-Pad2) -> GND
- Q23 pad 1: DBUS6 -> DBUS7
- Q29 pad 1: DBUS6 -> DBUS7
- Q35 pad 1: ~WS -> WS
- Q40 pad 1: OP3 -> ~OP3
- Q55 pad 1: OP3 -> ~OP3
Routing:
- net OP3: track 184.8 -> 0.00 mm, vias 6 -> 0
- net GND: track 331.4 -> 423.4 mm, vias 25 -> 32
- net RUN: track 83.8 -> 0.00 mm, vias 3 -> 0
- net ~OP3: track 89.3 -> 170.1 mm, vias 3 -> 8
- net DBUS7: track 0.00 -> 71.4 mm, vias 0 -> 3
- net DBUS6: track 71.0 -> 0.00 mm, vias 2 -> 0
- net DBUS5: track 61.5 -> 0.00 mm, vias 3 -> 0
- net ~OP4: track 133.7 -> 77.3 mm, vias 3 -> 2
- net OP1: track 42.1 -> 0.00 mm, vias 1 -> 0
- net VCC: track 684.7 -> 649.2 mm, vias 2 -> 4
- net OP5: track 166.5 -> 133.3 mm, vias 6 -> 5
- net ~OP5: track 104.9 -> 133.4 mm, vias 5 -> 6
- net WS: track 193.2 -> 210.6 mm
- net Net-(Q12-Pad3): track 3.39 -> 13.2 mm, vias 0 -> 2
- net RDA_DBUS: track 92.4 -> 84.5 mm
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Other:
- board text added: "LD NC"
- board text added: "NC D7"
- board text added: "PC S0"
- board text removed: "IC S0"
- board text removed: "LD D6"
- board text removed: "NC D5"
- board text removed: "~HALT"

Commit message: More fixes
Parts:
- added Q58: 2N7002, Package_TO_SOT_SMD:SOT-23_Handsoldering, F.Cu at (152.5, 79.5)
- added R22: 10k, Resistor_SMD:R_0805_2012Metric_Pad1.15x1.40mm_HandSolder, F.Cu at (156.5, 79.5)
- R1, R10, R11, R12, R14, R15, R16, R17, R18, R19, R2, R20, R21, R3, R4, R5, R6, R7, R8, R9: value R -> 10k
- R13: value R -> 1k
Routing:
- net RDM: track 123.1 -> 154.6 mm, vias 6 -> 7
- net WS: track 210.6 -> 221.3 mm
- net VCC: track 649.2 -> 654.5 mm, vias 4 -> 6
- net RDA_DBUS: track 84.5 -> 88.8 mm
- net GND: track 423.4 -> 425.9 mm
- net FOUT: track 89.9 -> 88.2 mm, vias 1 -> 3
