File: pcb/q2v2/areg.kicad_sch (KiCad schematic)
At the start: 2 parts, among them Q1033 2N7002, Q1034 2N7002

Commit message: Smaller
Parts:
- Q110: renamed from Q1033; value 2N7002 -> 2N7002a
- Q111: renamed from Q1034; value 2N7002 -> 2N7002a
Changed lines of the file:
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@@
   (title_block
     (title "Q2 A Register Bit")
-    (date "2021-01-30")
+    (date "2021-02-05")
     (rev "1")
     (company "joewing.net")
@@
   (symbol (lib_id "power:GND") (at 96.52 86.36 270)
     (in_bom yes) (on_board yes)
-    (property "Reference" "#PWR0851" (id 0) (at 90.17 86.36 0)
+    (property "Reference" "#PWR0120" (id 0) (at 90.17 86.36 0)
       (effects (font (size 1.27 1.27)) hide)
     )
@@
   (symbol (lib_id "power:GND") (at 96.52 90.17 270)
     (in_bom yes) (on_board yes)
-    (property "Reference" "#PWR0852" (id 0) (at 90.17 90.17 0)
+    (property "Reference" "#PWR0121" (id 0) (at 90.17 90.17 0)
       (effects (font (size 1.27 1.27)) hide)
     )
@@
   (symbol (lib_id "power:GND") (at 154.94 97.79 0)
     (in_bom yes) (on_board yes)
-    (property "Reference" "#PWR0850" (id 0) (at 154.94 104.14 0)
+    (property "Reference" "#PWR0122" (id 0) (at 154.94 104.14 0)
       (effects (font (size 1.27 1.27)) hide)
     )
@@
   (symbol (lib_id "Transistor_FET:2N7002") (at 152.4 82.55 0)
     (in_bom yes) (on_board yes)
-    (property "Reference" "Q1033" (id 0) (at 157.6324 81.3816 0)
+    (property "Reference" "Q110" (id 0) (at 157.6324 81.3816 0)
       (effects (font (size 1.27 1.27)) (justify left))
     )
-    (property "Value" "2N7002" (id 1) (at 157.6324 83.693 0)
+    (property "Value" "2N7002a" (id 1) (at 157.6324 83.693 0)
       (effects (font (size 1.27 1.27)) (justify left))
     )
@@
   (symbol (lib_id "Transistor_FET:2N7002") (at 152.4 92.71 0)
     (in_bom yes) (on_board yes)
-    (property "Reference" "Q1034" (id 0) (at 157.6324 91.5416 0)
+    (property "Reference" "Q111" (id 0) (at 157.6324 91.5416 0)
       (effects (font (size 1.27 1.27)) (justify left))
     )
-    (property "Value" "2N7002" (id 1) (at 157.6324 93.853 0)
+    (property "Value" "2N7002a" (id 1) (at 157.6324 93.853 0)
       (effects (font (size 1.27 1.27)) (justify left))
     )
