File: pcb/q2v2/bit.kicad_sch (KiCad schematic)
At the start: 5 parts, among them Q1031 2N7002-2, Q1032 2N7002-2

Commit message: Smaller
Parts:
- Q1077: renamed from Q1031; value 2N7002-2 -> 2N7002b
- Q1078: renamed from Q1032; value 2N7002-2 -> 2N7002b
- renumbered C16 to C27, R429 to R476, R430 to R477
Changed lines of the file:
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@@
   (title_block
     (title "Q2 Bit Slice")
-    (date "2021-01-30")
+    (date "2021-02-05")
     (rev "1")
     (company "joewing.net")
@@
   (symbol (lib_id "power:VCC") (at 184.15 44.45 0)
     (in_bom yes) (on_board yes)
-    (property "Reference" "#PWR0847" (id 0) (at 184.15 48.26 0)
+    (property "Reference" "#PWR01000" (id 0) (at 184.15 48.26 0)
       (effects (font (size 1.27 1.27)) hide)
     )
@@
   (symbol (lib_id "power:VCC") (at 200.66 40.64 0)
     (in_bom yes) (on_board yes)
-    (property "Reference" "#PWR0844" (id 0) (at 200.66 44.45 0)
+    (property "Reference" "#PWR0999" (id 0) (at 200.66 44.45 0)
       (effects (font (size 1.27 1.27)) hide)
     )
@@
   (symbol (lib_id "power:VCC") (at 220.98 71.12 0)
     (in_bom yes) (on_board yes)
-    (property "Reference" "#PWR0843" (id 0) (at 220.98 74.93 0)
+    (property "Reference" "#PWR01002" (id 0) (at 220.98 74.93 0)
       (effects (font (size 1.27 1.27)) hide)
     )
@@
   (symbol (lib_id "power:GND") (at 184.15 52.07 0)
     (in_bom yes) (on_board yes)
-    (property "Reference" "#PWR0846" (id 0) (at 184.15 58.42 0)
+    (property "Reference" "#PWR01001" (id 0) (at 184.15 58.42 0)
       (effects (font (size 1.27 1.27)) hide)
     )
@@
   (symbol (lib_id "power:GND") (at 220.98 109.22 0)
     (in_bom yes) (on_board yes)
-    (property "Reference" "#PWR0845" (id 0) (at 220.98 115.57 0)
+    (property "Reference" "#PWR01003" (id 0) (at 220.98 115.57 0)
       (effects (font (size 1.27 1.27)) hide)
     )
@@
   (symbol (lib_id "Device:R") (at 200.66 44.45 0)
     (in_bom yes) (on_board yes)
-    (property "Reference" "R429" (id 0) (at 202.438 43.2816 0)
+    (property "Reference" "R476" (id 0) (at 202.438 43.2816 0)
       (effects (font (size 1.27 1.27)) (justify left))
     )
@@
   (symbol (lib_id "Device:R") (at 220.98 74.93 0)
     (in_bom yes) (on_board yes)
-    (property "Reference" "R430" (id 0) (at 222.758 73.7616 0)
+    (property "Reference" "R477" (id 0) (at 222.758 73.7616 0)
       (effects (font (size 1.27 1.27)) (justify left))
     )
@@
   (symbol (lib_id "Device:C") (at 184.15 48.26 0)
     (in_bom yes) (on_board yes)
-    (property "Reference" "C16" (id 0) (at 187.071 47.0916 0)
+    (property "Reference" "C27" (id 0) (at 187.071 47.0916 0)
       (effects (font (size 1.27 1.27)) (justify left))
     )
@@
   (symbol (lib_id "Transistor_FET:2N7002") (at 218.44 93.98 0)
     (in_bom yes) (on_board yes)
-    (property "Reference" "Q1031" (id 0) (at 223.6724 92.8116 0)
-      (effects (font (size 1.27 1.27)) (justify left))
-    )
-    (property "Value" "2N7002-2" (id 1) (at 223.672 95.123 0)
+    (property "Reference" "Q1077" (id 0) (at 223.6724 92.8116 0)
+      (effects (font (size 1.27 1.27)) (justify left))
+    )
+    (property "Value" "2N7002b" (id 1) (at 223.672 95.123 0)
       (effects (font (size 1.27 1.27)) (justify left))
     )
@@
   (symbol (lib_id "Transistor_FET:2N7002") (at 218.44 104.14 0)
     (in_bom yes) (on_board yes)
-    (property "Reference" "Q1032" (id 0) (at 223.6724 102.9716 0)
-      (effects (font (size 1.27 1.27)) (justify left))
-    )
-    (property "Value" "2N7002-2" (id 1) (at 223.672 105.283 0)
-      (effects (font (size 1.27 1.27)) (justify left))
-    )
+    (property "Reference" "Q1078" (id 0) (at 223.6724 102.9716 0)
+      (effects (font (size 1.27 1.27)) (justify left))
+    )
+    (property "Value" "2N7002b" (id 1) (at 223.672 105.283 0)
+      (effects (font (size 1.27 1.27)) (justify left))
+    )
