File: pcb/q2v2/dff.kicad_sch (KiCad schematic)
At the start: 22 parts, among them Q1100 2N7002, Q1101 2N7002, Q1102 2N7002, Q1103 2N7002, Q1104 2N7002-2, Q1105 2N7002, Q1106 2N7002, Q1107 2N7002, Q1108 2N7002, Q1109 2N7002, Q1110 2N7002, Q1111 2N7002, Q1112 2N7002, Q1113 2N7002

Commit message: Smaller
Parts:
- Q136: renamed from Q1100; value 2N7002 -> 2N7002a
- Q137: renamed from Q1101; value 2N7002 -> 2N7002a
- Q138: renamed from Q1102; value 2N7002 -> 2N7002a
- Q139: renamed from Q1103; value 2N7002 -> 2N7002a
- Q140: renamed from Q1104; value 2N7002-2 -> 2N7002b
- Q141: renamed from Q1105; value 2N7002 -> 2N7002a
- Q142: renamed from Q1106; value 2N7002 -> 2N7002a
- Q143: renamed from Q1107; value 2N7002 -> 2N7002a
- Q144: renamed from Q1108; value 2N7002 -> 2N7002a
- Q145: renamed from Q1109; value 2N7002 -> 2N7002a
- Q146: renamed from Q1110; value 2N7002 -> 2N7002a
- Q147: renamed from Q1111; value 2N7002 -> 2N7002a
- Q148: renamed from Q1112; value 2N7002 -> 2N7002a
- Q149: renamed from Q1113; value 2N7002 -> 2N7002a
- renumbered D48 to D8, R456 to R56, R457 to R57, R458 to R58, R459 to R59, R460 to R60, R461 to R61, R462 to R62
