File: pcb/q2v2/fpbit.kicad_sch (KiCad schematic)
At the start: 7 parts, among them Q1132 2N7002-2, Q1133 2N7002-2, SW17 SW

Commit message: Smaller
Parts:
- Q993: renamed from Q1132; value 2N7002-2 -> 2N7002b
- Q994: renamed from Q1133; value 2N7002-2 -> 2N7002b
- renumbered D59 to D66, D60 to D67, R486 to R440, R487 to R441, SW17 to SW32
Changed lines of the file:
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@@
   (title_block
     (title "Front Panel Bit")
-    (date "2021-01-30")
+    (date "2021-02-05")
     (rev "1")
     (company "joewing.net")
@@
   (symbol (lib_id "power:VCC") (at 88.9 60.96 0)
     (in_bom yes) (on_board yes)
-    (property "Reference" "#PWR0997" (id 0) (at 88.9 64.77 0)
+    (property "Reference" "#PWR0930" (id 0) (at 88.9 64.77 0)
       (effects (font (size 1.27 1.27)) hide)
     )
@@
   (symbol (lib_id "power:VCC") (at 116.84 60.96 0)
     (in_bom yes) (on_board yes)
-    (property "Reference" "#PWR0998" (id 0) (at 116.84 64.77 0)
+    (property "Reference" "#PWR0931" (id 0) (at 116.84 64.77 0)
       (effects (font (size 1.27 1.27)) hide)
     )
@@
   (symbol (lib_id "power:GND") (at 88.9 86.36 0)
     (in_bom yes) (on_board yes)
-    (property "Reference" "#PWR0999" (id 0) (at 88.9 92.71 0)
+    (property "Reference" "#PWR0932" (id 0) (at 88.9 92.71 0)
       (effects (font (size 1.27 1.27)) hide)
     )
@@
   (symbol (lib_id "power:GND") (at 88.9 109.22 0)
     (in_bom yes) (on_board yes)
-    (property "Reference" "#PWR01001" (id 0) (at 88.9 115.57 0)
+    (property "Reference" "#PWR0934" (id 0) (at 88.9 115.57 0)
       (effects (font (size 1.27 1.27)) hide)
     )
@@
   (symbol (lib_id "power:GND") (at 116.84 86.36 0)
     (in_bom yes) (on_board yes)
-    (property "Reference" "#PWR01000" (id 0) (at 116.84 92.71 0)
+    (property "Reference" "#PWR0933" (id 0) (at 116.84 92.71 0)
       (effects (font (size 1.27 1.27)) hide)
     )
@@
   (symbol (lib_id "Device:R") (at 88.9 72.39 0)
     (in_bom yes) (on_board yes)
-    (property "Reference" "R486" (id 0) (at 90.678 71.2216 0)
+    (property "Reference" "R440" (id 0) (at 90.678 71.2216 0)
       (effects (font (size 1.27 1.27)) (justify left))
     )
@@
   (symbol (lib_id "Device:R") (at 116.84 72.39 0)
     (in_bom yes) (on_board yes)
-    (property "Reference" "R487" (id 0) (at 118.618 71.2216 0)
+    (property "Reference" "R441" (id 0) (at 118.618 71.2216 0)
       (effects (font (size 1.27 1.27)) (justify left))
     )
@@
   (symbol (lib_id "Device:LED") (at 88.9 64.77 90)
     (in_bom yes) (on_board yes)
-    (property "Reference" "D59" (id 0) (at 91.8718 63.7794 90)
+    (property "Reference" "D66" (id 0) (at 91.8718 63.7794 90)
       (effects (font (size 1.27 1.27)) (justify right))
     )
@@
   (symbol (lib_id "Device:LED") (at 116.84 64.77 90)
     (in_bom yes) (on_board yes)
-    (property "Reference" "D60" (id 0) (at 119.8118 63.7794 90)
+    (property "Reference" "D67" (id 0) (at 119.8118 63.7794 90)
       (effects (font (size 1.27 1.27)) (justify right))
     )
@@
   (symbol (lib_id "Switch:SW_SPST") (at 88.9 104.14 90)
     (in_bom yes) (on_board yes)
-    (property "Reference" "SW17" (id 0) (at 91.1352 102.9716 90)
+    (property "Reference" "SW32" (id 0) (at 91.1352 102.9716 90)
       (effects (font (size 1.27 1.27)) (justify right))
     )
@@
   (symbol (lib_id "Transistor_FET:2N7002") (at 86.36 81.28 0)
     (in_bom yes) (on_board yes)
-    (property "Reference" "Q1132" (id 0) (at 91.5924 80.1116 0)
-      (effects (font (size 1.27 1.27)) (justify left))
-    )
-    (property "Value" "2N7002-2" (id 1) (at 91.5924 82.423 0)
+    (property "Reference" "Q993" (id 0) (at 91.5924 80.1116 0)
+      (effects (font (size 1.27 1.27)) (justify left))
+    )
+    (property "Value" "2N7002b" (id 1) (at 91.5924 82.423 0)
       (effects (font (size 1.27 1.27)) (justify left))
     )
@@
   (symbol (lib_id "Transistor_FET:2N7002") (at 114.3 81.28 0)
     (in_bom yes) (on_board yes)
-    (property "Reference" "Q1133" (id 0) (at 119.5324 80.1116 0)
-      (effects (font (size 1.27 1.27)) (justify left))
-    )
-    (property "Value" "2N7002-2" (id 1) (at 119.532 82.423 0)
-      (effects (font (size 1.27 1.27)) (justify left))
-    )
+    (property "Reference" "Q994" (id 0) (at 119.5324 80.1116 0)
+      (effects (font (size 1.27 1.27)) (justify left))
+    )
+    (property "Value" "2N7002b" (id 1) (at 119.532 82.423 0)
+      (effects (font (size 1.27 1.27)) (justify left))
+    )
