File: pcb/q2v2/frontpanel.kicad_sch (KiCad schematic)
At the start: 45 parts, among them Q1117 2N7002-2, Q1123 2N7002-2, Q1127 2N7002-2, Q1146 2N7002-2, Q1147 2N7002, Q1148 2N7002-2, Q1149 2N7002-2, Q1150 2N7002-2, Q1151 2N7002-2, Q1152 2N7002-2, Q1153 2N7002-2, Q1154 2N7002-2, Q1155 2N7002-2, Q1156 2N7002-2, Q1157 2N7002-2, SW1 Input, SW10 Input, SW11 Input, SW14 Input, SW15 Input, SW25 Input, SW26 Input, SW27 Input, SW28 Input, SW29 Input, SW30 Input, SW31 Input, SW4 Reset, SW5 Deposit, SW6 Run, SW7 Halt, SW8 Next

Commit message: Smaller
Parts:
- C24: renamed from C5; value 0.1u -> 0.47u; LCSC C49678 -> C13967
- C25: renamed from C23; value 0.1u -> 0.47u; LCSC C49678 -> C13967
- Q956: renamed from Q1123; value 2N7002-2 -> 2N7002b
- Q957: renamed from Q1127; value 2N7002-2 -> 2N7002b
- Q958: renamed from Q1117; value 2N7002-2 -> 2N7002b
- Q959: renamed from Q1146; value 2N7002-2 -> 2N7002b
- Q960: renamed from Q1147; value 2N7002 -> 2N7002a
- Q961: renamed from Q1148; value 2N7002-2 -> 2N7002b
- Q962: renamed from Q1149; value 2N7002-2 -> 2N7002b
- Q963: renamed from Q1150; value 2N7002-2 -> 2N7002b
- Q964: renamed from Q1151; value 2N7002-2 -> 2N7002b
- Q965: renamed from Q1152; value 2N7002-2 -> 2N7002b
- Q966: renamed from Q1153; value 2N7002-2 -> 2N7002b
- Q967: renamed from Q1154; value 2N7002-2 -> 2N7002b
- Q968: renamed from Q1155; value 2N7002-2 -> 2N7002b
- Q969: renamed from Q1156; value 2N7002-2 -> 2N7002b
- Q970: renamed from Q1157; value 2N7002-2 -> 2N7002b
- renumbered D74 to D43, R102 to R410, R476 to R411, R477 to R412, R103 to R413, R104 to R414, R478 to R415, R481 to R416, R112 to R417, RV1 to RV3, SW14 to SW12, SW15 to SW13, SW25 to SW14, SW26 to SW15, SW27 to SW16, SW28 to SW17, SW29 to SW18, SW30 to SW19, SW31 to SW20, SW7 to SW4, SW4 to SW5, SW5 to SW6, SW6 to SW7, SW1 to SW9
Other:
- moved on the sheet: R414, SW8
