File: pcb/q2v2/logic.kicad_sch (KiCad schematic)
At the start: 66 parts, among them Q177 2N7002, Q183 2N7002, Q184 2N7002, Q185 2N7002, Q186 2N7002, Q187 2N7002, Q188 2N7002, Q189 2N7002, Q190 2N7002, Q191 2N7002, Q192 2N7002, Q193 2N7002, Q194 2N7002, Q195 2N7002, Q196 2N7002, Q197 2N7002, Q198 2N7002, Q199 2N7002, Q200 2N7002, Q201 2N7002, Q202 2N7002, Q203 2N7002, Q204 2N7002, Q205 2N7002, Q206 2N7002, Q207 2N7002, Q208 2N7002, Q209 2N7002, Q210 2N7002, Q211 2N7002, Q212 2N7002, Q213 2N7002, Q214 2N7002, Q215 2N7002, Q216 2N7002, Q217 2N7002, Q218 2N7002, Q219 2N7002, Q220 2N7002, Q221 2N7002, Q222 2N7002, Q223 2N7002, Q224 2N7002, Q225 2N7002, Q240 2N7002, Q241 2N7002, Q242 2N7002

Commit message: Smaller
Parts:
- Q179: renamed from Q177; value 2N7002 -> 2N7002a
- Q180: renamed from Q189; value 2N7002 -> 2N7002a
- Q181: renamed from Q183; value 2N7002 -> 2N7002a
- Q182: renamed from Q190; value 2N7002 -> 2N7002a
- Q183: renamed from Q191; value 2N7002 -> 2N7002a
- Q184: renamed from Q187; value 2N7002 -> 2N7002a
- Q185: renamed from Q188; value 2N7002 -> 2N7002a
- Q186: renamed from Q185; value 2N7002 -> 2N7002a
- Q187: renamed from Q186; value 2N7002 -> 2N7002a
- Q188: renamed from Q192; value 2N7002 -> 2N7002a
- Q189: renamed from Q197; value 2N7002 -> 2N7002a
- Q190: renamed from Q193; value 2N7002 -> 2N7002a
- Q191: renamed from Q194; value 2N7002 -> 2N7002a
- Q192: renamed from Q199; value 2N7002 -> 2N7002a
- Q193: renamed from Q200; value 2N7002 -> 2N7002a
- Q194: renamed from Q195; value 2N7002 -> 2N7002a
- Q195: renamed from Q196; value 2N7002 -> 2N7002a
- Q196: renamed from Q205; value 2N7002 -> 2N7002a
- Q197: renamed from Q206; value 2N7002 -> 2N7002a
- Q198, Q201, Q202, Q204, Q221, Q222, Q223, Q224, Q225: value 2N7002 -> 2N7002a
- Q199: renamed from Q240; value 2N7002 -> 2N7002a
- Q200: renamed from Q241; value 2N7002 -> 2N7002a
- Q203: renamed from Q242; value 2N7002 -> 2N7002a
- Q205: renamed from Q207; value 2N7002 -> 2N7002a
- Q206: renamed from Q203; value 2N7002 -> 2N7002a
- Q207: renamed from Q210; value 2N7002 -> 2N7002a
- Q208: renamed from Q184; value 2N7002 -> 2N7002a
- Q209: renamed from Q212; value 2N7002 -> 2N7002a
- Q210: renamed from Q213; value 2N7002 -> 2N7002a
- Q211: renamed from Q208; value 2N7002 -> 2N7002a
- Q212: renamed from Q209; value 2N7002 -> 2N7002a
- Q213: renamed from Q216; value 2N7002 -> 2N7002a
- Q214: renamed from Q217; value 2N7002 -> 2N7002a
- Q215: renamed from Q211; value 2N7002 -> 2N7002a
- Q216: renamed from Q214; value 2N7002 -> 2N7002a
- Q217: renamed from Q219; value 2N7002 -> 2N7002a
- Q218: renamed from Q220; value 2N7002 -> 2N7002a
- Q219: renamed from Q215; value 2N7002 -> 2N7002a
- Q220: renamed from Q218; value 2N7002 -> 2N7002a
- R81: renamed from R79; value 1k -> 4.7k; LCSC C17513 -> C17673
- R91: renamed from R89; value 10k -> 1k; LCSC C17414 -> C17513
- renumbered C6 to C7, R77 to R76, R82 to R77, R80 to R78, R81 to R79, R75 to R80, R85 to R82, R87 to R84, R84 to R85, R88 to R87, R106 to R88, R107 to R89, R78 to R90, R90 to R92, R91 to R93
Connections:
- net OP4 renamed O1
- net OP5 renamed O2
- net ~OP3 renamed ~O0
- net ~OP5 renamed ~O2
Other:
- note added: "Clock fanout to 12 DFFs (24 gates)"
- note added: "Fanout to 12 gates."
- note added: "Fanout to 8 gates"
- note added: "Set ABUS to P to fetch the instruction."
- note added: "Set DBUS = A"
- note added: "Set P = X Fanout to 24 gates"
- note added: "Write operand Saves the top 4 bits of DBUS to the top 4 bits of the state register."
- note removed: "1k resistor here for fast pullup Clock fanout to 12 DFFs (24 gates)"
- note removed: "Fanout to 12 gates"
- note removed: "Write operand Saves the top 6 bits of DBUS to the top 6 bits of the state register."
