File: pcb/q2v2/memory.kicad_sch (KiCad schematic)
At the start: 51 parts, among them Q1015 2N7002, Q1016 2N7002, Q1098 2N7002, Q1099 2N7002, Q1114 2N7002, Q1115 2N7002, Q1116 2N7002, Q1118 2N7002, Q1126 2N7002, Q249 2N7002, Q250 2N7002, Q601 2N7002, Q683 2N7002, Q684 2N7002, Q766 2N7002, Q767 2N7002, Q849 2N7002, Q850 2N7002, Q932 2N7002, Q933 2N7002, SW32 Write Protect, SW33 ROM Bank, U1 28C256, U2 6264, U3 6264, U4 28C256

Commit message: Smaller
Parts:
- Q772: renamed from Q1126; value 2N7002 -> 2N7002a
- Q773: renamed from Q249; value 2N7002 -> 2N7002a
- Q774: renamed from Q250; value 2N7002 -> 2N7002a
- Q775: renamed from Q1118; value 2N7002 -> 2N7002a
- Q776: renamed from Q601; value 2N7002 -> 2N7002a
- Q777: renamed from Q683; value 2N7002 -> 2N7002a
- Q778: renamed from Q684; value 2N7002 -> 2N7002a
- Q779: renamed from Q1098; value 2N7002 -> 2N7002a
- Q780: renamed from Q766; value 2N7002 -> 2N7002a
- Q781: renamed from Q1114; value 2N7002 -> 2N7002a
- Q782: renamed from Q767; value 2N7002 -> 2N7002a
- Q783: renamed from Q849; value 2N7002 -> 2N7002a
- Q784: renamed from Q850; value 2N7002 -> 2N7002a
- Q785: renamed from Q932; value 2N7002 -> 2N7002a
- Q786: renamed from Q1115; value 2N7002 -> 2N7002a
- Q787: renamed from Q1116; value 2N7002 -> 2N7002a
- Q788: renamed from Q933; value 2N7002 -> 2N7002a
- Q789: renamed from Q1015; value 2N7002 -> 2N7002a
- Q790: renamed from Q1016; value 2N7002 -> 2N7002a
- Q791: renamed from Q1099; value 2N7002 -> 2N7002a
- U2: footprint Package_SO:SOIC-28W_7.5x18.7mm_P1.27mm -> q2:SOIC127P1210X305-28N
- U4: renamed from U3; footprint Package_SO:SOIC-28W_7.5x18.7mm_P1.27mm -> q2:SOIC127P1210X305-28N
- renumbered C19 to C18, C20 to C19, C21 to C20, C22 to C21, R470 to R321, R465 to R322, R463 to R323, R94 to R324, R105 to R325, R501 to R326, R464 to R327, R502 to R328, R1 to R329, R471 to R330, R503 to R331, R469 to R332, R504 to R333, R467 to R334, R472 to R335, R473 to R336, R505 to R337, R506 to R338, R507 to R339, R508 to R340, R509 to R341, SW32 to SW2, SW33 to SW3, U4 to U3
Other:
- note removed: "LY6264SL ?"
