File: pcb/q2v2/xreg.kicad_sch (KiCad schematic)
At the start: 12 parts, among them Q1049 2N7002, Q1050 2N7002, Q1051 2N7002, Q1052 2N7002, Q1053 2N7002, Q1054 2N7002, Q1055 2N7002, Q1056 2N7002, Q1057 2N7002, Q1058 2N7002

Commit message: Smaller
Parts:
- Q126: renamed from Q1049; value 2N7002 -> 2N7002a
- Q127: renamed from Q1050; value 2N7002 -> 2N7002a
- Q128: renamed from Q1051; value 2N7002 -> 2N7002a
- Q129: renamed from Q1052; value 2N7002 -> 2N7002a
- Q130: renamed from Q1053; value 2N7002 -> 2N7002a
- Q131: renamed from Q1054; value 2N7002 -> 2N7002a
- Q132: renamed from Q1055; value 2N7002 -> 2N7002a
- Q133: renamed from Q1056; value 2N7002 -> 2N7002a
- Q134: renamed from Q1057; value 2N7002 -> 2N7002a
- Q135: renamed from Q1058; value 2N7002 -> 2N7002a
- renumbered R438 to R54, R439 to R55
Changed lines of the file:
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@@
   (title_block
     (title "Q2 X Register Bit")
-    (date "2021-01-30")
+    (date "2021-02-05")
     (rev "1")
     (company "joewing.net")
@@
   (symbol (lib_id "power:VCC") (at 67.31 104.14 0)
     (in_bom yes) (on_board yes)
-    (property "Reference" "#PWR0868" (id 0) (at 67.31 107.95 0)
+    (property "Reference" "#PWR0140" (id 0) (at 67.31 107.95 0)
       (effects (font (size 1.27 1.27)) hide)
     )
@@
   (symbol (lib_id "power:VCC") (at 135.89 46.99 0)
     (in_bom yes) (on_board yes)
-    (property "Reference" "#PWR0863" (id 0) (at 135.89 50.8 0)
+    (property "Reference" "#PWR0132" (id 0) (at 135.89 50.8 0)
       (effects (font (size 1.27 1.27)) hide)
     )
@@
   (symbol (lib_id "power:GND") (at 67.31 87.63 0)
     (in_bom yes) (on_board yes)
-    (property "Reference" "#PWR0869" (id 0) (at 67.31 93.98 0)
+    (property "Reference" "#PWR0135" (id 0) (at 67.31 93.98 0)
       (effects (font (size 1.27 1.27)) hide)
     )
@@
   (symbol (lib_id "power:GND") (at 67.31 130.81 0)
     (in_bom yes) (on_board yes)
-    (property "Reference" "#PWR0867" (id 0) (at 67.31 137.16 0)
+    (property "Reference" "#PWR0141" (id 0) (at 67.31 137.16 0)
       (effects (font (size 1.27 1.27)) hide)
     )
@@
   (symbol (lib_id "power:GND") (at 93.98 95.25 0)
     (in_bom yes) (on_board yes)
-    (property "Reference" "#PWR0866" (id 0) (at 93.98 101.6 0)
+    (property "Reference" "#PWR0136" (id 0) (at 93.98 101.6 0)
       (effects (font (size 1.27 1.27)) hide)
     )
@@
   (symbol (lib_id "power:GND") (at 119.38 96.52 0)
     (in_bom yes) (on_board yes)
-    (property "Reference" "#PWR0865" (id 0) (at 119.38 102.87 0)
+    (property "Reference" "#PWR0138" (id 0) (at 119.38 102.87 0)
       (effects (font (size 1.27 1.27)) hide)
     )
@@
   (symbol (lib_id "power:GND") (at 148.59 96.52 0)
     (in_bom yes) (on_board yes)
-    (property "Reference" "#PWR0864" (id 0) (at 148.59 102.87 0)
+    (property "Reference" "#PWR0139" (id 0) (at 148.59 102.87 0)
       (effects (font (size 1.27 1.27)) hide)
     )
@@
   (symbol (lib_id "power:GND") (at 205.74 63.5 90)
     (in_bom yes) (on_board yes)
-    (property "Reference" "#PWR0871" (id 0) (at 212.09 63.5 0)
+    (property "Reference" "#PWR0133" (id 0) (at 212.09 63.5 0)
       (effects (font (size 1.27 1.27)) hide)
     )
@@
   (symbol (lib_id "power:GND") (at 205.74 68.58 90)
     (in_bom yes) (on_board yes)
-    (property "Reference" "#PWR0870" (id 0) (at 212.09 68.58 0)
+    (property "Reference" "#PWR0134" (id 0) (at 212.09 68.58 0)
       (effects (font (size 1.27 1.27)) hide)
     )
@@
   (symbol (lib_id "power:GND") (at 240.03 95.25 0)
     (in_bom yes) (on_board yes)
-    (property "Reference" "#PWR0862" (id 0) (at 240.03 101.6 0)
+    (property "Reference" "#PWR0137" (id 0) (at 240.03 101.6 0)
       (effects (font (size 1.27 1.27)) hide)
     )
@@
   (symbol (lib_id "Device:R") (at 67.31 107.95 0)
     (in_bom yes) (on_board yes)
-    (property "Reference" "R439" (id 0) (at 69.088 106.7816 0)
+    (property "Reference" "R55" (id 0) (at 69.088 106.7816 0)
       (effects (font (size 1.27 1.27)) (justify left))
     )
@@
   (symbol (lib_id "Device:R") (at 135.89 50.8 0)
     (in_bom yes) (on_board yes)
-    (property "Reference" "R438" (id 0) (at 137.668 49.6316 0)
+    (property "Reference" "R54" (id 0) (at 137.668 49.6316 0)
       (effects (font (size 1.27 1.27)) (justify left))
     )
@@
   (symbol (lib_id "Transistor_FET:2N7002") (at 64.77 82.55 0)
     (in_bom yes) (on_board yes)
-    (property "Reference" "Q1053" (id 0) (at 70.0024 81.3816 0)
-      (effects (font (size 1.27 1.27)) (justify left))
-    )
-    (property "Value" "2N7002" (id 1) (at 70.0024 83.693 0)
+    (property "Reference" "Q130" (id 0) (at 70.0024 81.3816 0)
+      (effects (font (size 1.27 1.27)) (justify left))
+    )
+    (property "Value" "2N7002a" (id 1) (at 70.0024 83.693 0)
       (effects (font (size 1.27 1.27)) (justify left))
     )
@@
   (symbol (lib_id "Transistor_FET:2N7002") (at 64.77 125.73 0)
     (in_bom yes) (on_board yes)
-    (property "Reference" "Q1058" (id 0) (at 70.0024 124.5616 0)
-      (effects (font (size 1.27 1.27)) (justify left))
-    )
-    (property "Value" "2N7002" (id 1) (at 70.0024 126.873 0)
+    (property "Reference" "Q135" (id 0) (at 70.0024 124.5616 0)
+      (effects (font (size 1.27 1.27)) (justify left))
+    )
+    (property "Value" "2N7002a" (id 1) (at 70.0024 126.873 0)
       (effects (font (size 1.27 1.27)) (justify left))
     )
@@
   (symbol (lib_id "Transistor_FET:2N7002") (at 91.44 80.01 0)
     (in_bom yes) (on_board yes)
-    (property "Reference" "Q1049" (id 0) (at 96.6724 78.8416 0)
-      (effects (font (size 1.27 1.27)) (justify left))
-    )
-    (property "Value" "2N7002" (id 1) (at 96.6724 81.153 0)
+    (property "Reference" "Q126" (id 0) (at 96.6724 78.8416 0)
+      (effects (font (size 1.27 1.27)) (justify left))
+    )
+    (property "Value" "2N7002a" (id 1) (at 96.6724 81.153 0)
       (effects (font (size 1.27 1.27)) (justify left))
     )
@@
   (symbol (lib_id "Transistor_FET:2N7002") (at 91.44 90.17 0)
     (in_bom yes) (on_board yes)
-    (property "Reference" "Q1054" (id 0) (at 96.6724 89.0016 0)
-      (effects (font (size 1.27 1.27)) (justify left))
-    )
-    (property "Value" "2N7002" (id 1) (at 96.6724 91.313 0)
+    (property "Reference" "Q131" (id 0) (at 96.6724 89.0016 0)
+      (effects (font (size 1.27 1.27)) (justify left))
+    )
+    (property "Value" "2N7002a" (id 1) (at 96.6724 91.313 0)
       (effects (font (size 1.27 1.27)) (justify left))
     )
@@
   (symbol (lib_id "Transistor_FET:2N7002") (at 116.84 81.28 0)
     (in_bom yes) (on_board yes)
-    (property "Reference" "Q1051" (id 0) (at 122.0724 80.1116 0)
-      (effects (font (size 1.27 1.27)) (justify left))
-    )
-    (property "Value" "2N7002" (id 1) (at 122.0724 82.423 0)
+    (property "Reference" "Q128" (id 0) (at 122.0724 80.1116 0)
+      (effects (font (size 1.27 1.27)) (justify left))
+    )
+    (property "Value" "2N7002a" (id 1) (at 122.0724 82.423 0)
       (effects (font (size 1.27 1.27)) (justify left))
     )
@@
   (symbol (lib_id "Transistor_FET:2N7002") (at 116.84 91.44 0)
     (in_bom yes) (on_board yes)
-    (property "Reference" "Q1056" (id 0) (at 122.0724 90.2716 0)
-      (effects (font (size 1.27 1.27)) (justify left))
-    )
-    (property "Value" "2N7002" (id 1) (at 122.0724 92.583 0)
+    (property "Reference" "Q133" (id 0) (at 122.0724 90.2716 0)
+      (effects (font (size 1.27 1.27)) (justify left))
+    )
+    (property "Value" "2N7002a" (id 1) (at 122.0724 92.583 0)
       (effects (font (size 1.27 1.27)) (justify left))
     )
@@
   (symbol (lib_id "Transistor_FET:2N7002") (at 146.05 81.28 0)
     (in_bom yes) (on_board yes)
-    (property "Reference" "Q1052" (id 0) (at 151.2824 80.1116 0)
-      (effects (font (size 1.27 1.27)) (justify left))
-    )
-    (property "Value" "2N7002" (id 1) (at 151.2824 82.423 0)
+    (property "Reference" "Q129" (id 0) (at 151.2824 80.1116 0)
+      (effects (font (size 1.27 1.27)) (justify left))
+    )
+    (property "Value" "2N7002a" (id 1) (at 151.2824 82.423 0)
       (effects (font (size 1.27 1.27)) (justify left))
     )
@@
   (symbol (lib_id "Transistor_FET:2N7002") (at 146.05 91.44 0)
     (in_bom yes) (on_board yes)
-    (property "Reference" "Q1057" (id 0) (at 151.2824 90.2716 0)
-      (effects (font (size 1.27 1.27)) (justify left))
-    )
-    (property "Value" "2N7002" (id 1) (at 151.2824 92.583 0)
+    (property "Reference" "Q134" (id 0) (at 151.2824 90.2716 0)
+      (effects (font (size 1.27 1.27)) (justify left))
+    )
+    (property "Value" "2N7002a" (id 1) (at 151.2824 92.583 0)
       (effects (font (size 1.27 1.27)) (justify left))
     )
@@
   (symbol (lib_id "Transistor_FET:2N7002") (at 237.49 80.01 0)
     (in_bom yes) (on_board yes)
-    (property "Reference" "Q1050" (id 0) (at 242.7224 78.8416 0)
-      (effects (font (size 1.27 1.27)) (justify left))
-    )
-    (property "Value" "2N7002" (id 1) (at 242.7224 81.153 0)
+    (property "Reference" "Q127" (id 0) (at 242.7224 78.8416 0)
+      (effects (font (size 1.27 1.27)) (justify left))
+    )
+    (property "Value" "2N7002a" (id 1) (at 242.7224 81.153 0)
       (effects (font (size 1.27 1.27)) (justify left))
     )
@@
   (symbol (lib_id "Transistor_FET:2N7002") (at 237.49 90.17 0)
     (in_bom yes) (on_board yes)
-    (property "Reference" "Q1055" (id 0) (at 242.7224 89.0016 0)
-      (effects (font (size 1.27 1.27)) (justify left))
-    )
-    (property "Value" "2N7002" (id 1) (at 242.7224 91.313 0)
-      (effects (font (size 1.27 1.27)) (justify left))
-    )
+    (property "Reference" "Q132" (id 0) (at 242.7224 89.0016 0)
+      (effects (font (size 1.27 1.27)) (justify left))
+    )
+    (property "Value" "2N7002a" (id 1) (at 242.7224 91.313 0)
+      (effects (font (size 1.27 1.27)) (justify left))
+    )
