File: pcb/xreg.kicad_sch (KiCad schematic)
At the start: 12 parts, among them Q126 2N7002a, Q127 2N7002a, Q128 2N7002a, Q129 2N7002a, Q130 2N7002a, Q131 2N7002a, Q132 2N7002a, Q133 2N7002a, Q134 2N7002a, Q135 2N7002a

Commit message: Pi programmer.
Parts:
- renumbered Q126 to Q1079, Q127 to Q1080, Q128 to Q1081, Q129 to Q1082, Q130 to Q1083, Q131 to Q1084, Q132 to Q1085, Q133 to Q1086, Q134 to Q1087, Q135 to Q1088, R54 to R481, R55 to R482
Changed lines of the file:
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@@
   (symbol (lib_id "power:VCC") (at 67.31 104.14 0)
     (in_bom yes) (on_board yes)
-    (property "Reference" "#PWR0140" (id 0) (at 67.31 107.95 0)
+    (property "Reference" "#PWR0989" (id 0) (at 67.31 107.95 0)
       (effects (font (size 1.27 1.27)) hide)
     )
@@
   (symbol (lib_id "power:VCC") (at 135.89 46.99 0)
     (in_bom yes) (on_board yes)
-    (property "Reference" "#PWR0132" (id 0) (at 135.89 50.8 0)
+    (property "Reference" "#PWR0981" (id 0) (at 135.89 50.8 0)
       (effects (font (size 1.27 1.27)) hide)
     )
@@
   (symbol (lib_id "power:GND") (at 67.31 87.63 0)
     (in_bom yes) (on_board yes)
-    (property "Reference" "#PWR0135" (id 0) (at 67.31 93.98 0)
+    (property "Reference" "#PWR0984" (id 0) (at 67.31 93.98 0)
       (effects (font (size 1.27 1.27)) hide)
     )
@@
   (symbol (lib_id "power:GND") (at 67.31 130.81 0)
     (in_bom yes) (on_board yes)
-    (property "Reference" "#PWR0141" (id 0) (at 67.31 137.16 0)
+    (property "Reference" "#PWR0990" (id 0) (at 67.31 137.16 0)
       (effects (font (size 1.27 1.27)) hide)
     )
@@
   (symbol (lib_id "power:GND") (at 93.98 95.25 0)
     (in_bom yes) (on_board yes)
-    (property "Reference" "#PWR0136" (id 0) (at 93.98 101.6 0)
+    (property "Reference" "#PWR0985" (id 0) (at 93.98 101.6 0)
       (effects (font (size 1.27 1.27)) hide)
     )
@@
   (symbol (lib_id "power:GND") (at 119.38 96.52 0)
     (in_bom yes) (on_board yes)
-    (property "Reference" "#PWR0138" (id 0) (at 119.38 102.87 0)
+    (property "Reference" "#PWR0987" (id 0) (at 119.38 102.87 0)
       (effects (font (size 1.27 1.27)) hide)
     )
@@
   (symbol (lib_id "power:GND") (at 148.59 96.52 0)
     (in_bom yes) (on_board yes)
-    (property "Reference" "#PWR0139" (id 0) (at 148.59 102.87 0)
+    (property "Reference" "#PWR0988" (id 0) (at 148.59 102.87 0)
       (effects (font (size 1.27 1.27)) hide)
     )
@@
   (symbol (lib_id "power:GND") (at 205.74 63.5 90)
     (in_bom yes) (on_board yes)
-    (property "Reference" "#PWR0133" (id 0) (at 212.09 63.5 0)
+    (property "Reference" "#PWR0982" (id 0) (at 212.09 63.5 0)
       (effects (font (size 1.27 1.27)) hide)
     )
@@
   (symbol (lib_id "power:GND") (at 205.74 68.58 90)
     (in_bom yes) (on_board yes)
-    (property "Reference" "#PWR0134" (id 0) (at 212.09 68.58 0)
+    (property "Reference" "#PWR0983" (id 0) (at 212.09 68.58 0)
       (effects (font (size 1.27 1.27)) hide)
     )
@@
   (symbol (lib_id "power:GND") (at 240.03 95.25 0)
     (in_bom yes) (on_board yes)
-    (property "Reference" "#PWR0137" (id 0) (at 240.03 101.6 0)
+    (property "Reference" "#PWR0986" (id 0) (at 240.03 101.6 0)
       (effects (font (size 1.27 1.27)) hide)
     )
@@
   (symbol (lib_id "Device:R") (at 67.31 107.95 0)
     (in_bom yes) (on_board yes)
-    (property "Reference" "R55" (id 0) (at 69.088 106.7816 0)
+    (property "Reference" "R482" (id 0) (at 69.088 106.7816 0)
       (effects (font (size 1.27 1.27)) (justify left))
     )
@@
   (symbol (lib_id "Device:R") (at 135.89 50.8 0)
     (in_bom yes) (on_board yes)
-    (property "Reference" "R54" (id 0) (at 137.668 49.6316 0)
+    (property "Reference" "R481" (id 0) (at 137.668 49.6316 0)
       (effects (font (size 1.27 1.27)) (justify left))
     )
@@
   (symbol (lib_id "Transistor_FET:2N7002") (at 64.77 82.55 0)
     (in_bom yes) (on_board yes)
-    (property "Reference" "Q130" (id 0) (at 70.0024 81.3816 0)
+    (property "Reference" "Q1083" (id 0) (at 70.0024 81.3816 0)
       (effects (font (size 1.27 1.27)) (justify left))
     )
@@
   (symbol (lib_id "Transistor_FET:2N7002") (at 64.77 125.73 0)
     (in_bom yes) (on_board yes)
-    (property "Reference" "Q135" (id 0) (at 70.0024 124.5616 0)
+    (property "Reference" "Q1088" (id 0) (at 70.0024 124.5616 0)
       (effects (font (size 1.27 1.27)) (justify left))
     )
@@
   (symbol (lib_id "Transistor_FET:2N7002") (at 91.44 80.01 0)
     (in_bom yes) (on_board yes)
-    (property "Reference" "Q126" (id 0) (at 96.6724 78.8416 0)
+    (property "Reference" "Q1079" (id 0) (at 96.6724 78.8416 0)
       (effects (font (size 1.27 1.27)) (justify left))
     )
@@
   (symbol (lib_id "Transistor_FET:2N7002") (at 91.44 90.17 0)
     (in_bom yes) (on_board yes)
-    (property "Reference" "Q131" (id 0) (at 96.6724 89.0016 0)
+    (property "Reference" "Q1084" (id 0) (at 96.6724 89.0016 0)
       (effects (font (size 1.27 1.27)) (justify left))
     )
@@
   (symbol (lib_id "Transistor_FET:2N7002") (at 116.84 81.28 0)
     (in_bom yes) (on_board yes)
-    (property "Reference" "Q128" (id 0) (at 122.0724 80.1116 0)
+    (property "Reference" "Q1081" (id 0) (at 122.0724 80.1116 0)
       (effects (font (size 1.27 1.27)) (justify left))
     )
@@
   (symbol (lib_id "Transistor_FET:2N7002") (at 116.84 91.44 0)
     (in_bom yes) (on_board yes)
-    (property "Reference" "Q133" (id 0) (at 122.0724 90.2716 0)
+    (property "Reference" "Q1086" (id 0) (at 122.0724 90.2716 0)
       (effects (font (size 1.27 1.27)) (justify left))
     )
@@
   (symbol (lib_id "Transistor_FET:2N7002") (at 146.05 81.28 0)
     (in_bom yes) (on_board yes)
-    (property "Reference" "Q129" (id 0) (at 151.2824 80.1116 0)
+    (property "Reference" "Q1082" (id 0) (at 151.2824 80.1116 0)
       (effects (font (size 1.27 1.27)) (justify left))
     )
@@
   (symbol (lib_id "Transistor_FET:2N7002") (at 146.05 91.44 0)
     (in_bom yes) (on_board yes)
-    (property "Reference" "Q134" (id 0) (at 151.2824 90.2716 0)
+    (property "Reference" "Q1087" (id 0) (at 151.2824 90.2716 0)
       (effects (font (size 1.27 1.27)) (justify left))
     )
@@
   (symbol (lib_id "Transistor_FET:2N7002") (at 237.49 80.01 0)
     (in_bom yes) (on_board yes)
-    (property "Reference" "Q127" (id 0) (at 242.7224 78.8416 0)
+    (property "Reference" "Q1080" (id 0) (at 242.7224 78.8416 0)
       (effects (font (size 1.27 1.27)) (justify left))
     )
@@
   (symbol (lib_id "Transistor_FET:2N7002") (at 237.49 90.17 0)
     (in_bom yes) (on_board yes)
-    (property "Reference" "Q132" (id 0) (at 242.7224 89.0016 0)
-      (effects (font (size 1.27 1.27)) (justify left))
-    )
+    (property "Reference" "Q1085" (id 0) (at 242.7224 89.0016 0)
+      (effects (font (size 1.27 1.27)) (justify left))
+    )

Commit message: Fixes
Parts:
- renumbered Q1079 to Q1077, Q1080 to Q1078, Q1081 to Q1079, Q1082 to Q1080, Q1083 to Q1081, Q1084 to Q1082, Q1085 to Q1083, Q1086 to Q1084, Q1087 to Q1085, Q1088 to Q1086, R481 to R467, R482 to R468
Changed lines of the file:
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@@
   (symbol (lib_id "power:VCC") (at 67.31 104.14 0)
     (in_bom yes) (on_board yes)
-    (property "Reference" "#PWR0989" (id 0) (at 67.31 107.95 0)
+    (property "Reference" "#PWR0985" (id 0) (at 67.31 107.95 0)
       (effects (font (size 1.27 1.27)) hide)
     )
@@
   (symbol (lib_id "power:VCC") (at 135.89 46.99 0)
     (in_bom yes) (on_board yes)
-    (property "Reference" "#PWR0981" (id 0) (at 135.89 50.8 0)
+    (property "Reference" "#PWR0977" (id 0) (at 135.89 50.8 0)
       (effects (font (size 1.27 1.27)) hide)
     )
@@
   (symbol (lib_id "power:GND") (at 67.31 87.63 0)
     (in_bom yes) (on_board yes)
-    (property "Reference" "#PWR0984" (id 0) (at 67.31 93.98 0)
+    (property "Reference" "#PWR0980" (id 0) (at 67.31 93.98 0)
       (effects (font (size 1.27 1.27)) hide)
     )
@@
   (symbol (lib_id "power:GND") (at 67.31 130.81 0)
     (in_bom yes) (on_board yes)
-    (property "Reference" "#PWR0990" (id 0) (at 67.31 137.16 0)
+    (property "Reference" "#PWR0986" (id 0) (at 67.31 137.16 0)
       (effects (font (size 1.27 1.27)) hide)
     )
@@
   (symbol (lib_id "power:GND") (at 93.98 95.25 0)
     (in_bom yes) (on_board yes)
-    (property "Reference" "#PWR0985" (id 0) (at 93.98 101.6 0)
+    (property "Reference" "#PWR0981" (id 0) (at 93.98 101.6 0)
       (effects (font (size 1.27 1.27)) hide)
     )
@@
   (symbol (lib_id "power:GND") (at 119.38 96.52 0)
     (in_bom yes) (on_board yes)
-    (property "Reference" "#PWR0987" (id 0) (at 119.38 102.87 0)
+    (property "Reference" "#PWR0983" (id 0) (at 119.38 102.87 0)
       (effects (font (size 1.27 1.27)) hide)
     )
@@
   (symbol (lib_id "power:GND") (at 148.59 96.52 0)
     (in_bom yes) (on_board yes)
-    (property "Reference" "#PWR0988" (id 0) (at 148.59 102.87 0)
+    (property "Reference" "#PWR0984" (id 0) (at 148.59 102.87 0)
       (effects (font (size 1.27 1.27)) hide)
     )
@@
   (symbol (lib_id "power:GND") (at 205.74 63.5 90)
     (in_bom yes) (on_board yes)
-    (property "Reference" "#PWR0982" (id 0) (at 212.09 63.5 0)
+    (property "Reference" "#PWR0978" (id 0) (at 212.09 63.5 0)
       (effects (font (size 1.27 1.27)) hide)
     )
@@
   (symbol (lib_id "power:GND") (at 205.74 68.58 90)
     (in_bom yes) (on_board yes)
-    (property "Reference" "#PWR0983" (id 0) (at 212.09 68.58 0)
+    (property "Reference" "#PWR0979" (id 0) (at 212.09 68.58 0)
       (effects (font (size 1.27 1.27)) hide)
     )
@@
   (symbol (lib_id "power:GND") (at 240.03 95.25 0)
     (in_bom yes) (on_board yes)
-    (property "Reference" "#PWR0986" (id 0) (at 240.03 101.6 0)
+    (property "Reference" "#PWR0982" (id 0) (at 240.03 101.6 0)
       (effects (font (size 1.27 1.27)) hide)
     )
@@
   (symbol (lib_id "Device:R") (at 67.31 107.95 0)
     (in_bom yes) (on_board yes)
-    (property "Reference" "R482" (id 0) (at 69.088 106.7816 0)
+    (property "Reference" "R468" (id 0) (at 69.088 106.7816 0)
       (effects (font (size 1.27 1.27)) (justify left))
     )
@@
   (symbol (lib_id "Device:R") (at 135.89 50.8 0)
     (in_bom yes) (on_board yes)
-    (property "Reference" "R481" (id 0) (at 137.668 49.6316 0)
+    (property "Reference" "R467" (id 0) (at 137.668 49.6316 0)
       (effects (font (size 1.27 1.27)) (justify left))
     )
@@
   (symbol (lib_id "Transistor_FET:2N7002") (at 64.77 82.55 0)
     (in_bom yes) (on_board yes)
-    (property "Reference" "Q1083" (id 0) (at 70.0024 81.3816 0)
+    (property "Reference" "Q1081" (id 0) (at 70.0024 81.3816 0)
       (effects (font (size 1.27 1.27)) (justify left))
     )
@@
   (symbol (lib_id "Transistor_FET:2N7002") (at 64.77 125.73 0)
     (in_bom yes) (on_board yes)
-    (property "Reference" "Q1088" (id 0) (at 70.0024 124.5616 0)
+    (property "Reference" "Q1086" (id 0) (at 70.0024 124.5616 0)
       (effects (font (size 1.27 1.27)) (justify left))
     )
@@
   (symbol (lib_id "Transistor_FET:2N7002") (at 91.44 80.01 0)
     (in_bom yes) (on_board yes)
-    (property "Reference" "Q1079" (id 0) (at 96.6724 78.8416 0)
+    (property "Reference" "Q1077" (id 0) (at 96.6724 78.8416 0)
       (effects (font (size 1.27 1.27)) (justify left))
     )
@@
   (symbol (lib_id "Transistor_FET:2N7002") (at 91.44 90.17 0)
     (in_bom yes) (on_board yes)
-    (property "Reference" "Q1084" (id 0) (at 96.6724 89.0016 0)
+    (property "Reference" "Q1082" (id 0) (at 96.6724 89.0016 0)
       (effects (font (size 1.27 1.27)) (justify left))
     )
@@
   (symbol (lib_id "Transistor_FET:2N7002") (at 116.84 81.28 0)
     (in_bom yes) (on_board yes)
-    (property "Reference" "Q1081" (id 0) (at 122.0724 80.1116 0)
+    (property "Reference" "Q1079" (id 0) (at 122.0724 80.1116 0)
       (effects (font (size 1.27 1.27)) (justify left))
     )
@@
   (symbol (lib_id "Transistor_FET:2N7002") (at 116.84 91.44 0)
     (in_bom yes) (on_board yes)
-    (property "Reference" "Q1086" (id 0) (at 122.0724 90.2716 0)
+    (property "Reference" "Q1084" (id 0) (at 122.0724 90.2716 0)
       (effects (font (size 1.27 1.27)) (justify left))
     )
@@
   (symbol (lib_id "Transistor_FET:2N7002") (at 146.05 81.28 0)
     (in_bom yes) (on_board yes)
-    (property "Reference" "Q1082" (id 0) (at 151.2824 80.1116 0)
+    (property "Reference" "Q1080" (id 0) (at 151.2824 80.1116 0)
       (effects (font (size 1.27 1.27)) (justify left))
     )
@@
   (symbol (lib_id "Transistor_FET:2N7002") (at 146.05 91.44 0)
     (in_bom yes) (on_board yes)
-    (property "Reference" "Q1087" (id 0) (at 151.2824 90.2716 0)
+    (property "Reference" "Q1085" (id 0) (at 151.2824 90.2716 0)
       (effects (font (size 1.27 1.27)) (justify left))
     )
@@
   (symbol (lib_id "Transistor_FET:2N7002") (at 237.49 80.01 0)
     (in_bom yes) (on_board yes)
-    (property "Reference" "Q1080" (id 0) (at 242.7224 78.8416 0)
+    (property "Reference" "Q1078" (id 0) (at 242.7224 78.8416 0)
       (effects (font (size 1.27 1.27)) (justify left))
     )
@@
   (symbol (lib_id "Transistor_FET:2N7002") (at 237.49 90.17 0)
     (in_bom yes) (on_board yes)
-    (property "Reference" "Q1085" (id 0) (at 242.7224 89.0016 0)
-      (effects (font (size 1.27 1.27)) (justify left))
-    )
+    (property "Reference" "Q1083" (id 0) (at 242.7224 89.0016 0)
+      (effects (font (size 1.27 1.27)) (justify left))
+    )

Commit message: Cleanups.
Parts:
- renumbered Q1077 to Q1076, Q1078 to Q1077, Q1079 to Q1078, Q1080 to Q1079, Q1081 to Q1080, Q1082 to Q1081, Q1083 to Q1082, Q1084 to Q1083, Q1085 to Q1084, Q1086 to Q1085, R467 to R465, R468 to R466
Changed lines of the file:
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@@
   (symbol (lib_id "power:VCC") (at 67.31 104.14 0)
     (in_bom yes) (on_board yes)
-    (property "Reference" "#PWR0985" (id 0) (at 67.31 107.95 0)
+    (property "Reference" "#PWR0981" (id 0) (at 67.31 107.95 0)
       (effects (font (size 1.27 1.27)) hide)
     )
@@
   (symbol (lib_id "power:VCC") (at 135.89 46.99 0)
     (in_bom yes) (on_board yes)
-    (property "Reference" "#PWR0977" (id 0) (at 135.89 50.8 0)
+    (property "Reference" "#PWR0973" (id 0) (at 135.89 50.8 0)
       (effects (font (size 1.27 1.27)) hide)
     )
@@
   (symbol (lib_id "power:GND") (at 67.31 87.63 0)
     (in_bom yes) (on_board yes)
-    (property "Reference" "#PWR0980" (id 0) (at 67.31 93.98 0)
+    (property "Reference" "#PWR0976" (id 0) (at 67.31 93.98 0)
       (effects (font (size 1.27 1.27)) hide)
     )
@@
   (symbol (lib_id "power:GND") (at 67.31 130.81 0)
     (in_bom yes) (on_board yes)
-    (property "Reference" "#PWR0986" (id 0) (at 67.31 137.16 0)
+    (property "Reference" "#PWR0982" (id 0) (at 67.31 137.16 0)
       (effects (font (size 1.27 1.27)) hide)
     )
@@
   (symbol (lib_id "power:GND") (at 93.98 95.25 0)
     (in_bom yes) (on_board yes)
-    (property "Reference" "#PWR0981" (id 0) (at 93.98 101.6 0)
+    (property "Reference" "#PWR0977" (id 0) (at 93.98 101.6 0)
       (effects (font (size 1.27 1.27)) hide)
     )
@@
   (symbol (lib_id "power:GND") (at 119.38 96.52 0)
     (in_bom yes) (on_board yes)
-    (property "Reference" "#PWR0983" (id 0) (at 119.38 102.87 0)
+    (property "Reference" "#PWR0979" (id 0) (at 119.38 102.87 0)
       (effects (font (size 1.27 1.27)) hide)
     )
@@
   (symbol (lib_id "power:GND") (at 148.59 96.52 0)
     (in_bom yes) (on_board yes)
-    (property "Reference" "#PWR0984" (id 0) (at 148.59 102.87 0)
+    (property "Reference" "#PWR0980" (id 0) (at 148.59 102.87 0)
       (effects (font (size 1.27 1.27)) hide)
     )
@@
   (symbol (lib_id "power:GND") (at 205.74 63.5 90)
     (in_bom yes) (on_board yes)
-    (property "Reference" "#PWR0978" (id 0) (at 212.09 63.5 0)
+    (property "Reference" "#PWR0974" (id 0) (at 212.09 63.5 0)
       (effects (font (size 1.27 1.27)) hide)
     )
@@
   (symbol (lib_id "power:GND") (at 205.74 68.58 90)
     (in_bom yes) (on_board yes)
-    (property "Reference" "#PWR0979" (id 0) (at 212.09 68.58 0)
+    (property "Reference" "#PWR0975" (id 0) (at 212.09 68.58 0)
       (effects (font (size 1.27 1.27)) hide)
     )
@@
   (symbol (lib_id "power:GND") (at 240.03 95.25 0)
     (in_bom yes) (on_board yes)
-    (property "Reference" "#PWR0982" (id 0) (at 240.03 101.6 0)
+    (property "Reference" "#PWR0978" (id 0) (at 240.03 101.6 0)
       (effects (font (size 1.27 1.27)) hide)
     )
@@
   (symbol (lib_id "Device:R") (at 67.31 107.95 0)
     (in_bom yes) (on_board yes)
-    (property "Reference" "R468" (id 0) (at 69.088 106.7816 0)
+    (property "Reference" "R466" (id 0) (at 69.088 106.7816 0)
       (effects (font (size 1.27 1.27)) (justify left))
     )
@@
   (symbol (lib_id "Device:R") (at 135.89 50.8 0)
     (in_bom yes) (on_board yes)
-    (property "Reference" "R467" (id 0) (at 137.668 49.6316 0)
+    (property "Reference" "R465" (id 0) (at 137.668 49.6316 0)
       (effects (font (size 1.27 1.27)) (justify left))
     )
@@
   (symbol (lib_id "Transistor_FET:2N7002") (at 64.77 82.55 0)
     (in_bom yes) (on_board yes)
-    (property "Reference" "Q1081" (id 0) (at 70.0024 81.3816 0)
+    (property "Reference" "Q1080" (id 0) (at 70.0024 81.3816 0)
       (effects (font (size 1.27 1.27)) (justify left))
     )
@@
   (symbol (lib_id "Transistor_FET:2N7002") (at 64.77 125.73 0)
     (in_bom yes) (on_board yes)
-    (property "Reference" "Q1086" (id 0) (at 70.0024 124.5616 0)
+    (property "Reference" "Q1085" (id 0) (at 70.0024 124.5616 0)
       (effects (font (size 1.27 1.27)) (justify left))
     )
@@
   (symbol (lib_id "Transistor_FET:2N7002") (at 91.44 80.01 0)
     (in_bom yes) (on_board yes)
-    (property "Reference" "Q1077" (id 0) (at 96.6724 78.8416 0)
+    (property "Reference" "Q1076" (id 0) (at 96.6724 78.8416 0)
       (effects (font (size 1.27 1.27)) (justify left))
     )
@@
   (symbol (lib_id "Transistor_FET:2N7002") (at 91.44 90.17 0)
     (in_bom yes) (on_board yes)
-    (property "Reference" "Q1082" (id 0) (at 96.6724 89.0016 0)
+    (property "Reference" "Q1081" (id 0) (at 96.6724 89.0016 0)
       (effects (font (size 1.27 1.27)) (justify left))
     )
@@
   (symbol (lib_id "Transistor_FET:2N7002") (at 116.84 81.28 0)
     (in_bom yes) (on_board yes)
-    (property "Reference" "Q1079" (id 0) (at 122.0724 80.1116 0)
+    (property "Reference" "Q1078" (id 0) (at 122.0724 80.1116 0)
       (effects (font (size 1.27 1.27)) (justify left))
     )
@@
   (symbol (lib_id "Transistor_FET:2N7002") (at 116.84 91.44 0)
     (in_bom yes) (on_board yes)
-    (property "Reference" "Q1084" (id 0) (at 122.0724 90.2716 0)
+    (property "Reference" "Q1083" (id 0) (at 122.0724 90.2716 0)
       (effects (font (size 1.27 1.27)) (justify left))
     )
@@
   (symbol (lib_id "Transistor_FET:2N7002") (at 146.05 81.28 0)
     (in_bom yes) (on_board yes)
-    (property "Reference" "Q1080" (id 0) (at 151.2824 80.1116 0)
+    (property "Reference" "Q1079" (id 0) (at 151.2824 80.1116 0)
       (effects (font (size 1.27 1.27)) (justify left))
     )
@@
   (symbol (lib_id "Transistor_FET:2N7002") (at 146.05 91.44 0)
     (in_bom yes) (on_board yes)
-    (property "Reference" "Q1085" (id 0) (at 151.2824 90.2716 0)
+    (property "Reference" "Q1084" (id 0) (at 151.2824 90.2716 0)
       (effects (font (size 1.27 1.27)) (justify left))
     )
@@
   (symbol (lib_id "Transistor_FET:2N7002") (at 237.49 80.01 0)
     (in_bom yes) (on_board yes)
-    (property "Reference" "Q1078" (id 0) (at 242.7224 78.8416 0)
+    (property "Reference" "Q1077" (id 0) (at 242.7224 78.8416 0)
       (effects (font (size 1.27 1.27)) (justify left))
     )
@@
   (symbol (lib_id "Transistor_FET:2N7002") (at 237.49 90.17 0)
     (in_bom yes) (on_board yes)
-    (property "Reference" "Q1083" (id 0) (at 242.7224 89.0016 0)
-      (effects (font (size 1.27 1.27)) (justify left))
-    )
+    (property "Reference" "Q1082" (id 0) (at 242.7224 89.0016 0)
+      (effects (font (size 1.27 1.27)) (justify left))
+    )
