File: pcb/bit.kicad_sch (KiCad schematic)
At the start: 5 parts, among them Q1077 2N7002b, Q1078 2N7002b

Commit message: Pi programmer.
Parts:
- renumbered C27 to C23, Q1077 to Q912, Q1078 to Q913, R476 to R411, R477 to R412
Changed lines of the file:
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@@
   (symbol (lib_id "power:VCC") (at 184.15 44.45 0)
     (in_bom yes) (on_board yes)
-    (property "Reference" "#PWR01000" (id 0) (at 184.15 48.26 0)
+    (property "Reference" "#PWR0847" (id 0) (at 184.15 48.26 0)
       (effects (font (size 1.27 1.27)) hide)
     )
@@
   (symbol (lib_id "power:VCC") (at 200.66 40.64 0)
     (in_bom yes) (on_board yes)
-    (property "Reference" "#PWR0999" (id 0) (at 200.66 44.45 0)
+    (property "Reference" "#PWR0846" (id 0) (at 200.66 44.45 0)
       (effects (font (size 1.27 1.27)) hide)
     )
@@
   (symbol (lib_id "power:VCC") (at 220.98 71.12 0)
     (in_bom yes) (on_board yes)
-    (property "Reference" "#PWR01002" (id 0) (at 220.98 74.93 0)
+    (property "Reference" "#PWR0849" (id 0) (at 220.98 74.93 0)
       (effects (font (size 1.27 1.27)) hide)
     )
@@
   (symbol (lib_id "power:GND") (at 184.15 52.07 0)
     (in_bom yes) (on_board yes)
-    (property "Reference" "#PWR01001" (id 0) (at 184.15 58.42 0)
+    (property "Reference" "#PWR0848" (id 0) (at 184.15 58.42 0)
       (effects (font (size 1.27 1.27)) hide)
     )
@@
   (symbol (lib_id "power:GND") (at 220.98 109.22 0)
     (in_bom yes) (on_board yes)
-    (property "Reference" "#PWR01003" (id 0) (at 220.98 115.57 0)
+    (property "Reference" "#PWR0850" (id 0) (at 220.98 115.57 0)
       (effects (font (size 1.27 1.27)) hide)
     )
@@
   (symbol (lib_id "Device:R") (at 200.66 44.45 0)
     (in_bom yes) (on_board yes)
-    (property "Reference" "R476" (id 0) (at 202.438 43.2816 0)
+    (property "Reference" "R411" (id 0) (at 202.438 43.2816 0)
       (effects (font (size 1.27 1.27)) (justify left))
     )
@@
   (symbol (lib_id "Device:R") (at 220.98 74.93 0)
     (in_bom yes) (on_board yes)
-    (property "Reference" "R477" (id 0) (at 222.758 73.7616 0)
+    (property "Reference" "R412" (id 0) (at 222.758 73.7616 0)
       (effects (font (size 1.27 1.27)) (justify left))
     )
@@
   (symbol (lib_id "Device:C") (at 184.15 48.26 0)
     (in_bom yes) (on_board yes)
-    (property "Reference" "C27" (id 0) (at 187.071 47.0916 0)
+    (property "Reference" "C23" (id 0) (at 187.071 47.0916 0)
       (effects (font (size 1.27 1.27)) (justify left))
     )
@@
   (symbol (lib_id "Transistor_FET:2N7002") (at 218.44 93.98 0)
     (in_bom yes) (on_board yes)
-    (property "Reference" "Q1077" (id 0) (at 223.6724 92.8116 0)
+    (property "Reference" "Q912" (id 0) (at 223.6724 92.8116 0)
       (effects (font (size 1.27 1.27)) (justify left))
     )
@@
   (symbol (lib_id "Transistor_FET:2N7002") (at 218.44 104.14 0)
     (in_bom yes) (on_board yes)
-    (property "Reference" "Q1078" (id 0) (at 223.6724 102.9716 0)
+    (property "Reference" "Q913" (id 0) (at 223.6724 102.9716 0)
       (effects (font (size 1.27 1.27)) (justify left))
     )

Commit message: Fixes
Parts:
- renumbered Q912 to Q910, Q913 to Q911, R411 to R397, R412 to R398
Changed lines of the file:
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@@
   (symbol (lib_id "power:VCC") (at 184.15 44.45 0)
     (in_bom yes) (on_board yes)
-    (property "Reference" "#PWR0847" (id 0) (at 184.15 48.26 0)
+    (property "Reference" "#PWR0843" (id 0) (at 184.15 48.26 0)
       (effects (font (size 1.27 1.27)) hide)
     )
@@
   (symbol (lib_id "power:VCC") (at 200.66 40.64 0)
     (in_bom yes) (on_board yes)
-    (property "Reference" "#PWR0846" (id 0) (at 200.66 44.45 0)
+    (property "Reference" "#PWR0842" (id 0) (at 200.66 44.45 0)
       (effects (font (size 1.27 1.27)) hide)
     )
@@
   (symbol (lib_id "power:VCC") (at 220.98 71.12 0)
     (in_bom yes) (on_board yes)
-    (property "Reference" "#PWR0849" (id 0) (at 220.98 74.93 0)
+    (property "Reference" "#PWR0845" (id 0) (at 220.98 74.93 0)
       (effects (font (size 1.27 1.27)) hide)
     )
@@
   (symbol (lib_id "power:GND") (at 184.15 52.07 0)
     (in_bom yes) (on_board yes)
-    (property "Reference" "#PWR0848" (id 0) (at 184.15 58.42 0)
+    (property "Reference" "#PWR0844" (id 0) (at 184.15 58.42 0)
       (effects (font (size 1.27 1.27)) hide)
     )
@@
   (symbol (lib_id "power:GND") (at 220.98 109.22 0)
     (in_bom yes) (on_board yes)
-    (property "Reference" "#PWR0850" (id 0) (at 220.98 115.57 0)
+    (property "Reference" "#PWR0846" (id 0) (at 220.98 115.57 0)
       (effects (font (size 1.27 1.27)) hide)
     )
@@
   (symbol (lib_id "Device:R") (at 200.66 44.45 0)
     (in_bom yes) (on_board yes)
-    (property "Reference" "R411" (id 0) (at 202.438 43.2816 0)
+    (property "Reference" "R397" (id 0) (at 202.438 43.2816 0)
       (effects (font (size 1.27 1.27)) (justify left))
     )
@@
   (symbol (lib_id "Device:R") (at 220.98 74.93 0)
     (in_bom yes) (on_board yes)
-    (property "Reference" "R412" (id 0) (at 222.758 73.7616 0)
+    (property "Reference" "R398" (id 0) (at 222.758 73.7616 0)
       (effects (font (size 1.27 1.27)) (justify left))
     )
@@
   (symbol (lib_id "Transistor_FET:2N7002") (at 218.44 93.98 0)
     (in_bom yes) (on_board yes)
-    (property "Reference" "Q912" (id 0) (at 223.6724 92.8116 0)
+    (property "Reference" "Q910" (id 0) (at 223.6724 92.8116 0)
       (effects (font (size 1.27 1.27)) (justify left))
     )
@@
   (symbol (lib_id "Transistor_FET:2N7002") (at 218.44 104.14 0)
     (in_bom yes) (on_board yes)
-    (property "Reference" "Q913" (id 0) (at 223.6724 102.9716 0)
+    (property "Reference" "Q911" (id 0) (at 223.6724 102.9716 0)
       (effects (font (size 1.27 1.27)) (justify left))
     )

Commit message: Cleanups.
Parts:
- renumbered Q910 to Q909, Q911 to Q910, R397 to R395, R398 to R396
Changed lines of the file:
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@@
   (symbol (lib_id "power:VCC") (at 184.15 44.45 0)
     (in_bom yes) (on_board yes)
-    (property "Reference" "#PWR0843" (id 0) (at 184.15 48.26 0)
+    (property "Reference" "#PWR0839" (id 0) (at 184.15 48.26 0)
       (effects (font (size 1.27 1.27)) hide)
     )
@@
   (symbol (lib_id "power:VCC") (at 200.66 40.64 0)
     (in_bom yes) (on_board yes)
-    (property "Reference" "#PWR0842" (id 0) (at 200.66 44.45 0)
+    (property "Reference" "#PWR0838" (id 0) (at 200.66 44.45 0)
       (effects (font (size 1.27 1.27)) hide)
     )
@@
   (symbol (lib_id "power:VCC") (at 220.98 71.12 0)
     (in_bom yes) (on_board yes)
-    (property "Reference" "#PWR0845" (id 0) (at 220.98 74.93 0)
+    (property "Reference" "#PWR0841" (id 0) (at 220.98 74.93 0)
       (effects (font (size 1.27 1.27)) hide)
     )
@@
   (symbol (lib_id "power:GND") (at 184.15 52.07 0)
     (in_bom yes) (on_board yes)
-    (property "Reference" "#PWR0844" (id 0) (at 184.15 58.42 0)
+    (property "Reference" "#PWR0840" (id 0) (at 184.15 58.42 0)
       (effects (font (size 1.27 1.27)) hide)
     )
@@
   (symbol (lib_id "power:GND") (at 220.98 109.22 0)
     (in_bom yes) (on_board yes)
-    (property "Reference" "#PWR0846" (id 0) (at 220.98 115.57 0)
+    (property "Reference" "#PWR0842" (id 0) (at 220.98 115.57 0)
       (effects (font (size 1.27 1.27)) hide)
     )
@@
   (symbol (lib_id "Device:R") (at 200.66 44.45 0)
     (in_bom yes) (on_board yes)
-    (property "Reference" "R397" (id 0) (at 202.438 43.2816 0)
+    (property "Reference" "R395" (id 0) (at 202.438 43.2816 0)
       (effects (font (size 1.27 1.27)) (justify left))
     )
@@
   (symbol (lib_id "Device:R") (at 220.98 74.93 0)
     (in_bom yes) (on_board yes)
-    (property "Reference" "R398" (id 0) (at 222.758 73.7616 0)
+    (property "Reference" "R396" (id 0) (at 222.758 73.7616 0)
       (effects (font (size 1.27 1.27)) (justify left))
     )
@@
   (symbol (lib_id "Transistor_FET:2N7002") (at 218.44 93.98 0)
     (in_bom yes) (on_board yes)
-    (property "Reference" "Q910" (id 0) (at 223.6724 92.8116 0)
+    (property "Reference" "Q909" (id 0) (at 223.6724 92.8116 0)
       (effects (font (size 1.27 1.27)) (justify left))
     )
@@
   (symbol (lib_id "Transistor_FET:2N7002") (at 218.44 104.14 0)
     (in_bom yes) (on_board yes)
-    (property "Reference" "Q911" (id 0) (at 223.6724 102.9716 0)
+    (property "Reference" "Q910" (id 0) (at 223.6724 102.9716 0)
       (effects (font (size 1.27 1.27)) (justify left))
     )

Commit message: Buttons.
Parts:
- renumbered R395 to R396, R396 to R397
Changed lines of the file:
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@@
   (symbol (lib_id "Device:R") (at 200.66 44.45 0)
     (in_bom yes) (on_board yes)
-    (property "Reference" "R395" (id 0) (at 202.438 43.2816 0)
+    (property "Reference" "R396" (id 0) (at 202.438 43.2816 0)
       (effects (font (size 1.27 1.27)) (justify left))
     )
@@
   (symbol (lib_id "Device:R") (at 220.98 74.93 0)
     (in_bom yes) (on_board yes)
-    (property "Reference" "R396" (id 0) (at 222.758 73.7616 0)
+    (property "Reference" "R397" (id 0) (at 222.758 73.7616 0)
       (effects (font (size 1.27 1.27)) (justify left))
     )
