File: pcb/memory.kicad_sch (KiCad schematic)
At the start: 38 parts, among them Q690 2N7002a, Q691 2N7002a, Q692 2N7002a, Q693 2N7002a, Q694 2N7002a, Q695 2N7002a, Q696 2N7002a, Q697 2N7002a, Q698 2N7002a, Q699 2N7002a, Q700 2N7002a, Q701 2N7002a, Q702 2N7002a, Q703 2N7002a, Q704 2N7002a, Q705 2N7002a, Q706 2N7002a, Q707 2N7002a, Q708 2N7002a, U1 6264, U2 6264

Commit message: Fixes
Parts:
- BT1: footprint Battery:BatteryHolder_Keystone_107_1x23mm -> Battery:BatteryHolder_ComfortableElectronic_CH273-2450_1x2450
- renumbered Q690 to Q688, Q691 to Q689, Q692 to Q690, Q693 to Q691, Q694 to Q692, Q695 to Q693, Q696 to Q694, Q697 to Q695, Q698 to Q696, Q699 to Q697, Q700 to Q698, Q701 to Q699, Q702 to Q700, Q703 to Q701, Q704 to Q702, Q705 to Q703, Q706 to Q704, Q707 to Q705, Q708 to Q706
Changed lines of the file:
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@@
   (symbol (lib_id "power:PWR_FLAG") (at 163.83 50.8 0) (unit 1)
     (in_bom yes) (on_board yes)
-    (property "Reference" "#FLG?" (id 0) (at 163.83 48.895 0)
+    (property "Reference" "#FLG01" (id 0) (at 163.83 48.895 0)
       (effects (font (size 1.27 1.27)) hide)
     )
@@
   (symbol (lib_id "power:VCC") (at 80.01 119.38 0) (unit 1)
     (in_bom yes) (on_board yes)
-    (property "Reference" "#PWR0614" (id 0) (at 80.01 123.19 0)
+    (property "Reference" "#PWR0612" (id 0) (at 80.01 123.19 0)
       (effects (font (size 1.27 1.27)) hide)
     )
@@
   (symbol (lib_id "power:VCC") (at 109.22 120.65 0) (unit 1)
     (in_bom yes) (on_board yes)
-    (property "Reference" "#PWR0615" (id 0) (at 109.22 124.46 0)
+    (property "Reference" "#PWR0613" (id 0) (at 109.22 124.46 0)
       (effects (font (size 1.27 1.27)) hide)
     )
@@
   (symbol (lib_id "power:GND") (at 36.83 185.42 0) (unit 1)
     (in_bom yes) (on_board yes)
-    (property "Reference" "#PWR0620" (id 0) (at 36.83 191.77 0)
+    (property "Reference" "#PWR0618" (id 0) (at 36.83 191.77 0)
       (effects (font (size 1.27 1.27)) hide)
     )
@@
   (symbol (lib_id "power:GND") (at 80.01 144.78 0) (unit 1)
     (in_bom yes) (on_board yes)
-    (property "Reference" "#PWR0618" (id 0) (at 80.01 151.13 0)
+    (property "Reference" "#PWR0616" (id 0) (at 80.01 151.13 0)
       (effects (font (size 1.27 1.27)) hide)
     )
@@
   (symbol (lib_id "power:GND") (at 109.22 146.05 0) (unit 1)
     (in_bom yes) (on_board yes)
-    (property "Reference" "#PWR0619" (id 0) (at 109.22 152.4 0)
+    (property "Reference" "#PWR0617" (id 0) (at 109.22 152.4 0)
       (effects (font (size 1.27 1.27)) hide)
     )
@@
   (symbol (lib_id "power:GND") (at 163.83 110.49 270) (unit 1)
     (in_bom yes) (on_board yes)
-    (property "Reference" "#PWR0612" (id 0) (at 157.48 110.49 0)
+    (property "Reference" "#PWR0610" (id 0) (at 157.48 110.49 0)
       (effects (font (size 1.27 1.27)) hide)
     )
@@
   (symbol (lib_id "power:GND") (at 173.99 125.73 0) (unit 1)
     (in_bom yes) (on_board yes)
-    (property "Reference" "#PWR0616" (id 0) (at 173.99 132.08 0)
+    (property "Reference" "#PWR0614" (id 0) (at 173.99 132.08 0)
       (effects (font (size 1.27 1.27)) hide)
     )
@@
   (symbol (lib_id "power:GND") (at 233.68 111.76 270) (unit 1)
     (in_bom yes) (on_board yes)
-    (property "Reference" "#PWR0613" (id 0) (at 227.33 111.76 0)
+    (property "Reference" "#PWR0611" (id 0) (at 227.33 111.76 0)
       (effects (font (size 1.27 1.27)) hide)
     )
@@
   (symbol (lib_id "power:GND") (at 243.84 127 0) (unit 1)
     (in_bom yes) (on_board yes)
-    (property "Reference" "#PWR0617" (id 0) (at 243.84 133.35 0)
+    (property "Reference" "#PWR0615" (id 0) (at 243.84 133.35 0)
       (effects (font (size 1.27 1.27)) hide)
     )
@@
       (effects (font (size 1.27 1.27)) (justify left))
     )
-    (property "Footprint" "Battery:BatteryHolder_Keystone_107_1x23mm" (id 2) (at 243.84 45.466 90)
+    (property "Footprint" "Battery:BatteryHolder_ComfortableElectronic_CH273-2450_1x2450" (id 2) (at 243.84 45.466 90)
       (effects (font (size 1.27 1.27)) hide)
     )
@@
   (symbol (lib_id "Transistor_FET:2N7002") (at 34.29 68.58 0) (unit 1)
     (in_bom yes) (on_board yes)
-    (property "Reference" "Q694" (id 0) (at 39.5224 67.4116 0)
+    (property "Reference" "Q692" (id 0) (at 39.5224 67.4116 0)
       (effects (font (size 1.27 1.27)) (justify left))
     )
@@
   (symbol (lib_id "Transistor_FET:2N7002") (at 34.29 78.74 0) (unit 1)
     (in_bom yes) (on_board yes)
-    (property "Reference" "Q695" (id 0) (at 39.5224 77.5716 0)
+    (property "Reference" "Q693" (id 0) (at 39.5224 77.5716 0)
       (effects (font (size 1.27 1.27)) (justify left))
     )
@@
   (symbol (lib_id "Transistor_FET:2N7002") (at 34.29 88.9 0) (unit 1)
     (in_bom yes) (on_board yes)
-    (property "Reference" "Q697" (id 0) (at 39.5224 87.7316 0)
+    (property "Reference" "Q695" (id 0) (at 39.5224 87.7316 0)
       (effects (font (size 1.27 1.27)) (justify left))
     )
@@
   (symbol (lib_id "Transistor_FET:2N7002") (at 34.29 99.06 0) (unit 1)
     (in_bom yes) (on_board yes)
-    (property "Reference" "Q698" (id 0) (at 39.5224 97.8916 0)
+    (property "Reference" "Q696" (id 0) (at 39.5224 97.8916 0)
       (effects (font (size 1.27 1.27)) (justify left))
     )
@@
   (symbol (lib_id "Transistor_FET:2N7002") (at 34.29 109.22 0) (unit 1)
     (in_bom yes) (on_board yes)
-    (property "Reference" "Q699" (id 0) (at 39.5224 108.0516 0)
+    (property "Reference" "Q697" (id 0) (at 39.5224 108.0516 0)
       (effects (font (size 1.27 1.27)) (justify left))
     )
@@
   (symbol (lib_id "Transistor_FET:2N7002") (at 34.29 119.38 0) (unit 1)
     (in_bom yes) (on_board yes)
-    (property "Reference" "Q700" (id 0) (at 39.5224 118.2116 0)
+    (property "Reference" "Q698" (id 0) (at 39.5224 118.2116 0)
       (effects (font (size 1.27 1.27)) (justify left))
     )
@@
   (symbol (lib_id "Transistor_FET:2N7002") (at 34.29 129.54 0) (unit 1)
     (in_bom yes) (on_board yes)
-    (property "Reference" "Q701" (id 0) (at 39.5224 128.3716 0)
+    (property "Reference" "Q699" (id 0) (at 39.5224 128.3716 0)
       (effects (font (size 1.27 1.27)) (justify left))
     )
@@
   (symbol (lib_id "Transistor_FET:2N7002") (at 34.29 139.7 0) (unit 1)
     (in_bom yes) (on_board yes)
-    (property "Reference" "Q702" (id 0) (at 39.5224 138.5316 0)
+    (property "Reference" "Q700" (id 0) (at 39.5224 138.5316 0)
       (effects (font (size 1.27 1.27)) (justify left))
     )
@@
   (symbol (lib_id "Transistor_FET:2N7002") (at 34.29 149.86 0) (unit 1)
     (in_bom yes) (on_board yes)
-    (property "Reference" "Q705" (id 0) (at 39.5224 148.6916 0)
+    (property "Reference" "Q703" (id 0) (at 39.5224 148.6916 0)
       (effects (font (size 1.27 1.27)) (justify left))
     )
@@
   (symbol (lib_id "Transistor_FET:2N7002") (at 34.29 160.02 0) (unit 1)
     (in_bom yes) (on_board yes)
-    (property "Reference" "Q706" (id 0) (at 39.5224 158.8516 0)
+    (property "Reference" "Q704" (id 0) (at 39.5224 158.8516 0)
       (effects (font (size 1.27 1.27)) (justify left))
     )
@@
   (symbol (lib_id "Transistor_FET:2N7002") (at 34.29 170.18 0) (unit 1)
     (in_bom yes) (on_board yes)
-    (property "Reference" "Q707" (id 0) (at 39.5224 169.0116 0)
+    (property "Reference" "Q705" (id 0) (at 39.5224 169.0116 0)
       (effects (font (size 1.27 1.27)) (justify left))
     )
@@
   (symbol (lib_id "Transistor_FET:2N7002") (at 34.29 180.34 0) (unit 1)
     (in_bom yes) (on_board yes)
-    (property "Reference" "Q708" (id 0) (at 39.5224 179.1716 0)
+    (property "Reference" "Q706" (id 0) (at 39.5224 179.1716 0)
       (effects (font (size 1.27 1.27)) (justify left))
     )
@@
   (symbol (lib_id "Transistor_FET:2N7002") (at 54.61 49.53 0) (unit 1)
     (in_bom yes) (on_board yes)
-    (property "Reference" "Q692" (id 0) (at 59.8424 48.3616 0)
+    (property "Reference" "Q690" (id 0) (at 59.8424 48.3616 0)
       (effects (font (size 1.27 1.27)) (justify left))
     )
@@
   (symbol (lib_id "Transistor_FET:2N7002") (at 73.66 40.64 0) (unit 1)
     (in_bom yes) (on_board yes)
-    (property "Reference" "Q691" (id 0) (at 78.8924 39.4716 0)
+    (property "Reference" "Q689" (id 0) (at 78.8924 39.4716 0)
       (effects (font (size 1.27 1.27)) (justify left))
     )
@@
   (symbol (lib_id "Transistor_FET:2N7002") (at 77.47 139.7 0) (unit 1)
     (in_bom yes) (on_board yes)
-    (property "Reference" "Q703" (id 0) (at 82.7024 138.5316 0)
+    (property "Reference" "Q701" (id 0) (at 82.7024 138.5316 0)
       (effects (font (size 1.27 1.27)) (justify left))
     )
@@
   (symbol (lib_id "Transistor_FET:2N7002") (at 99.06 49.53 0) (unit 1)
     (in_bom yes) (on_board yes)
-    (property "Reference" "Q693" (id 0) (at 104.2924 48.3616 0)
+    (property "Reference" "Q691" (id 0) (at 104.2924 48.3616 0)
       (effects (font (size 1.27 1.27)) (justify left))
     )
@@
   (symbol (lib_id "Transistor_FET:2N7002") (at 106.68 140.97 0) (unit 1)
     (in_bom yes) (on_board yes)
-    (property "Reference" "Q704" (id 0) (at 111.9124 139.8016 0)
+    (property "Reference" "Q702" (id 0) (at 111.9124 139.8016 0)
       (effects (font (size 1.27 1.27)) (justify left))
     )
@@
   (symbol (lib_id "Transistor_FET:2N7002") (at 118.11 39.37 0) (unit 1)
     (in_bom yes) (on_board yes)
-    (property "Reference" "Q690" (id 0) (at 123.3424 38.2016 0)
+    (property "Reference" "Q688" (id 0) (at 123.3424 38.2016 0)
       (effects (font (size 1.27 1.27)) (justify left))
     )
@@
   (symbol (lib_id "Transistor_FET:2N7002") (at 123.19 82.55 0) (unit 1)
     (in_bom yes) (on_board yes)
-    (property "Reference" "Q696" (id 0) (at 128.4224 81.3816 0)
-      (effects (font (size 1.27 1.27)) (justify left))
-    )
+    (property "Reference" "Q694" (id 0) (at 128.4224 81.3816 0)
+      (effects (font (size 1.27 1.27)) (justify left))
+    )

Commit message: Cleanups.
Parts:
- added Q1125: 2N7002a, Package_TO_SOT_SMD:SOT-23, symbol Transistor_FET:2N7002
- added R483: 10k, Resistor_SMD:R_0805_2012Metric, symbol Device:R
- renumbered D31 to D30, D32 to D31, R287 to R286, R288 to R287, R289 to R288, R290 to R289, R291 to R290, R292 to R291, R293 to R292, R294 to R293, R295 to R294, R296 to R295, R297 to R296, R298 to R297
Connections:
- net GND: now also Q1125.2 (S); no longer Q694.2 (S)
- net VCC: now also Q1125.1 (G), R483.1; no longer R296.1
- net at C17.2, C18.2, D30.1 (K)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: now also R296.1; no longer U1.26 (A13), U2.26 (A13)
- new net: R483.2, U1.26 (A13), U2.26 (A13)
- new net: Q1125.3 (D), Q694.2 (S)
Other:
- moved on the sheet: BT1, C17, C18, D30, D31, Q694, Q701, Q702, R291, R292, R293, R294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

Commit message: Buttons.
Parts:
- removed Q1125: 2N7002a, Package_TO_SOT_SMD:SOT-23, symbol Transistor_FET:2N7002
- renumbered Q695 to Q694, Q696 to Q695, Q701 to Q696, Q694 to Q697, Q697 to Q698, Q698 to Q699, Q699 to Q700, Q700 to Q701, R296 to R291, R291 to R292, R292 to R293, R293 to R294, R294 to R295, R295 to R296, R483 to R297, R297 to R298
Connections:
- net GND: now also Q697.2 (S)

Commit message: Fix UUIDs.
Parts:
- renumbered Q688 to Q679, Q689 to Q680, Q690 to Q681, Q691 to Q682, Q692 to Q683, Q693 to Q684, Q694 to Q685, Q695 to Q686, Q696 to Q687, Q697 to Q688, Q698 to Q689, Q699 to Q690, Q700 to Q691, Q701 to Q692, Q702 to Q693, Q703 to Q694, Q704 to Q695, Q705 to Q696, Q706 to Q697

Commit message: New reset.
Parts:
- removed R297: 10k, Resistor_SMD:R_0805_2012Metric, symbol Device:R
- renumbered C17 to C16, C18 to C17, R298 to R297
Connections:
- net ~RST: now reaches U1.26 (A13), U2.26 (A13)

Commit message: Skip ALU state for jfc/jmp/sta.
Parts:
- D30, D31: value B5819W -> BAT43W; LCSC C8598 -> C19167
Changed lines of the file:
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@@
       (effects (font (size 1.27 1.27)) (justify right))
     )
-    (property "Value" "B5819W" (id 1) (at 176.0221 77.3493 90)
+    (property "Value" "BAT43W" (id 1) (at 176.0221 77.3493 90)
       (effects (font (size 1.27 1.27)) (justify right))
     )
@@
       (effects (font (size 1.27 1.27)) hide)
     )
-    (property "Datasheet" "https://datasheet.lcsc.com/szlcsc/Changjiang-Electronics-Tech-CJ-B5819W_C8598.pdf" (id 3) (at 173.99 76.2 0)
+    (property "Datasheet" "https://datasheet.lcsc.com/szlcsc/Changjiang-Electronics-Tech-CJ-BAT43W_C19167.pdf" (id 3) (at 173.99 76.2 0)
       (effects (font (size 1.27 1.27)) hide)
     )
-    (property "LCSC" "C8598" (id 4) (at 173.99 76.2 0)
+    (property "LCSC" "C19167" (id 4) (at 173.99 76.2 0)
       (effects (font (size 1.27 1.27)) hide)
     )
@@
       (effects (font (size 1.27 1.27)) (justify right))
     )
-    (property "Value" "B5819W" (id 1) (at 223.0121 76.0793 90)
+    (property "Value" "BAT43W" (id 1) (at 223.0121 76.0793 90)
       (effects (font (size 1.27 1.27)) (justify right))
     )
@@
       (effects (font (size 1.27 1.27)) hide)
     )
-    (property "Datasheet" "https://datasheet.lcsc.com/szlcsc/Changjiang-Electronics-Tech-CJ-B5819W_C8598.pdf" (id 3) (at 220.98 74.93 0)
+    (property "Datasheet" "https://datasheet.lcsc.com/szlcsc/Changjiang-Electronics-Tech-CJ-BAT43W_C19167.pdf" (id 3) (at 220.98 74.93 0)
       (effects (font (size 1.27 1.27)) hide)
     )
-    (property "LCSC" "C8598" (id 4) (at 220.98 74.93 0)
+    (property "LCSC" "C19167" (id 4) (at 220.98 74.93 0)
       (effects (font (size 1.27 1.27)) hide)
     )

Commit message: Cleanups.
Parts:
- added C25: 1u, Capacitor_SMD:C_0805_2012Metric, symbol Device:C
- added C26: 0.1u, Capacitor_SMD:C_0805_2012Metric, symbol Device:C
- added D90: BAT43W, Diode_SMD:D_SOD-123, symbol Diode:1N5819
- added R485: 10k, Resistor_SMD:R_0805_2012Metric, symbol Device:R
Connections:
- net GND: now also C25.2, C26.1
- net VCC: now also D90.1 (K), R485.1
- net at C16.2, C17.2, D30.1 (K)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: now also C25.1
- net ~RST: no longer names the net of U1.26 (A13), U2.26 (A13)
- net ~RST: now also C26.2, D90.2 (A), R485.2
Other:
- note added: "A13 (pin 26) is an active high chip enable. Here we hold it low for a moment after Vcc is applied and pull it low quickly when Vcc is removed to avoid spurious writes."
- note added: "Hold ~CE~ high even when Vcc is removed."
- moved on the sheet: C17

Commit message: Updates.
Parts:
- added R484: 10k, Resistor_SMD:R_0805_2012Metric, symbol Device:R
- added SW31: Bank, Connector_PinHeader_2.54mm:PinHeader_1x03_P2.54mm_Vertical, symbol Switch:SW_SPST
Connections:
- net GND: now also SW31.1 (A); no longer U1.2 (A12), U2.2 (A12)
- net VCC: now also R484.1
- new net BANK: R484.2, SW31.2 (B), U1.2 (A12), U2.2 (A12)
Changed lines of the file:
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@@
   (junction (at 57.15 40.64) (diameter 1.016) (color 0 0 0 0))
   (junction (at 57.15 59.69) (diameter 1.016) (color 0 0 0 0))
+  (junction (at 74.93 166.37) (diameter 0.9144) (color 0 0 0 0))
   (junction (at 76.2 34.29) (diameter 1.016) (color 0 0 0 0))
   (junction (at 99.06 99.06) (diameter 1.016) (color 0 0 0 0))
@@
     (stroke (width 0) (type solid) (color 0 0 0 0))
   )
+  (wire (pts (xy 74.93 165.1) (xy 74.93 166.37))
+    (stroke (width 0) (type solid) (color 0 0 0 0))
+  )
+  (wire (pts (xy 74.93 166.37) (xy 74.93 168.91))
+    (stroke (width 0) (type solid) (color 0 0 0 0))
+  )
+  (wire (pts (xy 74.93 166.37) (xy 80.01 166.37))
+    (stroke (width 0) (type solid) (color 0 0 0 0))
+  )
   (wire (pts (xy 76.2 33.02) (xy 76.2 34.29))
     (stroke (width 0) (type solid) (color 0 0 0 0))
@@
     (stroke (width 0) (type solid) (color 0 0 0 0))
   )
+  (wire (pts (xy 151.13 130.81) (xy 163.83 130.81))
+    (stroke (width 0) (type solid) (color 0 0 0 0))
+  )
   (wire (pts (xy 153.67 143.51) (xy 163.83 143.51))
     (stroke (width 0) (type solid) (color 0 0 0 0))
@@
   )
   (wire (pts (xy 220.98 88.9) (xy 243.84 88.9))
+    (stroke (width 0) (type solid) (color 0 0 0 0))
+  )
+  (wire (pts (xy 222.25 132.08) (xy 233.68 132.08))
     (stroke (width 0) (type solid) (color 0 0 0 0))
   )
@@
     (effects (font (size 1.27 1.27)) (justify left bottom))
   )
+  (label "BANK" (at 80.01 166.37 0)
+    (effects (font (size 1.27 1.27)) (justify left bottom))
+  )
+  (label "BANK" (at 151.13 130.81 180)
+    (effects (font (size 1.27 1.27)) (justify right bottom))
+  )
+  (label "BANK" (at 222.25 132.08 180)
+    (effects (font (size 1.27 1.27)) (justify right bottom))
+  )
   (global_label "ABUS0" (shape input) (at 29.21 68.58 180)
     (effects (font (size 1.27 1.27)) (justify right))
@@
     (pin "1")
   )
+  (symbol (lib_id "power:VCC") (at 74.93 157.48 0) (unit 1)
+    (in_bom yes) (on_board yes)
+    (property "Reference" "#PWR0587" (id 0) (at 74.93 161.29 0)
+      (effects (font (size 1.27 1.27)) hide)
+    )
+    (property "Value" "VCC" (id 1) (at 75.3618 153.0858 0))
+    (property "Footprint" "" (id 2) (at 74.93 157.48 0)
+      (effects (font (size 1.27 1.27)) hide)
+    )
+    (property "Datasheet" "" (id 3) (at 74.93 157.48 0)
+      (effects (font (size 1.27 1.27)) hide)
+    )
+    (pin "1")
+  )
   (symbol (lib_id "power:VCC") (at 76.2 25.4 0) (unit 1)
     (in_bom yes) (on_board yes)
@@
     (pin "1")
   )
+  (symbol (lib_id "power:GND") (at 74.93 179.07 0) (unit 1)
+    (in_bom yes) (on_board yes)
+    (property "Reference" "#PWR0986" (id 0) (at 74.93 185.42 0)
+      (effects (font (size 1.27 1.27)) hide)
+    )
+    (property "Value" "GND" (id 1) (at 75.057 183.4642 0))
+    (property "Footprint" "" (id 2) (at 74.93 179.07 0)
+      (effects (font (size 1.27 1.27)) hide)
+    )
+    (property "Datasheet" "" (id 3) (at 74.93 179.07 0)
+      (effects (font (size 1.27 1.27)) hide)
+    )
+    (pin "1")
+  )
   (symbol (lib_id "power:GND") (at 76.2 45.72 0) (unit 1)
     (in_bom yes) (on_board yes)
@@
     (pin "1")
   )
-  (symbol (lib_id "power:GND") (at 163.83 130.81 270) (unit 1)
-    (in_bom yes) (on_board yes)
-    (property "Reference" "#PWR0587" (id 0) (at 157.48 130.81 0)
-      (effects (font (size 1.27 1.27)) hide)
-    )
-    (property "Value" "GND" (id 1) (at 159.4358 130.937 0))
-    (property "Footprint" "" (id 2) (at 163.83 130.81 0)
-      (effects (font (size 1.27 1.27)) hide)
-    )
-    (property "Datasheet" "" (id 3) (at 163.83 130.81 0)
-      (effects (font (size 1.27 1.27)) hide)
-    )
-    (pin "1")
-  )
   (symbol (lib_id "power:GND") (at 163.83 135.89 270) (unit 1)
     (in_bom yes) (on_board yes)
@@
     (pin "1")
   )
-  (symbol (lib_id "power:GND") (at 233.68 132.08 270) (unit 1)
-    (in_bom yes) (on_board yes)
-    (property "Reference" "#PWR0588" (id 0) (at 227.33 132.08 0)
-      (effects (font (size 1.27 1.27)) hide)
-    )
-    (property "Value" "GND" (id 1) (at 229.2858 132.207 0))
-    (property "Footprint" "" (id 2) (at 233.68 132.08 0)
-      (effects (font (size 1.27 1.27)) hide)
-    )
-    (property "Datasheet" "" (id 3) (at 233.68 132.08 0)
-      (effects (font (size 1.27 1.27)) hide)
-    )
-    (pin "1")
-  )
   (symbol (lib_id "power:GND") (at 233.68 137.16 270) (unit 1)
     (in_bom yes) (on_board yes)
@@
     (pin "2")
   )
+  (symbol (lib_id "Device:R") (at 74.93 161.29 0) (unit 1)
+    (in_bom yes) (on_board yes)
+    (property "Reference" "R484" (id 0) (at 76.708 160.1216 0)
+      (effects (font (size 1.27 1.27)) (justify left))
+    )
+    (property "Value" "10k" (id 1) (at 76.708 162.433 0)
+      (effects (font (size 1.27 1.27)) (justify left))
+    )
+    (property "Footprint" "Resistor_SMD:R_0805_2012Metric" (id 2) (at 73.152 161.29 90)
+      (effects (font (size 1.27 1.27)) hide)
+    )
+    (property "Datasheet" "~" (id 3) (at 74.93 161.29 0)
+      (effects (font (size 1.27 1.27)) hide)
+    )
+    (property "LCSC" "C17414" (id 4) (at 74.93 161.29 0)
+      (effects (font (size 1.27 1.27)) hide)
+    )
+    (pin "1")
+    (pin "2")
+  )
   (symbol (lib_id "Device:R") (at 76.2 29.21 0) (unit 1)
     (in_bom yes) (on_board yes)
@@
       (effects (font (size 1.27 1.27)) hide)
     )
+    (pin "1")
+    (pin "2")
+  )
+  (symbol (lib_id "Switch:SW_SPST") (at 74.93 173.99 90) (unit 1)
+    (in_bom yes) (on_board yes)
+    (property "Reference" "SW31" (id 0) (at 77.1652 172.8216 90)
+      (effects (font (size 1.27 1.27)) (justify right))
+    )
+    (property "Value" "Bank" (id 1) (at 77.165 175.133 90)
+      (effects (font (size 1.27 1.27)) (justify right))
+    )
+    (property "Footprint" "Connector_PinHeader_2.54mm:PinHeader_1x03_P2.54mm_Vertical" (id 2) (at 74.93 173.99 0)
+      (effects (font (size 1.27 1.27)) hide)
+    )
+    (property "Datasheet" "~" (id 3) (at 74.93 173.99 0)
+      (effects (font (size 1.27 1.27)) hide)
+    )
