File: pcb/bit-high.kicad_sch (KiCad schematic)
At the start: 5 parts, among them Q693 2N7002K, Q694 2N7002K

Commit message: Update resistors.
Parts:
- renumbered Q693 to Q691, Q694 to Q692, R300 to R298, R301 to R299
Other:
- moved on the sheet: C21
Changed lines of the file:
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@@
     (effects (font (size 1.27 1.27)) (justify left))
-  )
-  (symbol (lib_id "power:VCC") (at 184.15 44.45 0)
-    (in_bom yes) (on_board yes)
-    (property "Reference" "#PWR0604" (id 0) (at 184.15 48.26 0)
-      (effects (font (size 1.27 1.27)) hide)
-    )
-    (property "Value" "VCC" (id 1) (at 184.5818 40.0558 0))
-    (property "Footprint" "" (id 2) (at 184.15 44.45 0)
-      (effects (font (size 1.27 1.27)) hide)
-    )
-    (property "Datasheet" "" (id 3) (at 184.15 44.45 0)
-      (effects (font (size 1.27 1.27)) hide)
-    )
-    (pin "1")
   )
   (symbol (lib_id "power:VCC") (at 200.66 40.64 0)
     (in_bom yes) (on_board yes)
-    (property "Reference" "#PWR0603" (id 0) (at 200.66 44.45 0)
+    (property "Reference" "#PWR0599" (id 0) (at 200.66 44.45 0)
       (effects (font (size 1.27 1.27)) hide)
     )
@@
     (pin "1")
   )
+  (symbol (lib_id "power:VCC") (at 219.71 40.64 0)
+    (in_bom yes) (on_board yes)
+    (property "Reference" "#PWR0600" (id 0) (at 219.71 44.45 0)
+      (effects (font (size 1.27 1.27)) hide)
+    )
+    (property "Value" "VCC" (id 1) (at 220.1418 36.2458 0))
+    (property "Footprint" "" (id 2) (at 219.71 40.64 0)
+      (effects (font (size 1.27 1.27)) hide)
+    )
+    (property "Datasheet" "" (id 3) (at 219.71 40.64 0)
+      (effects (font (size 1.27 1.27)) hide)
+    )
+    (pin "1")
+  )
   (symbol (lib_id "power:VCC") (at 220.98 71.12 0)
     (in_bom yes) (on_board yes)
-    (property "Reference" "#PWR0606" (id 0) (at 220.98 74.93 0)
+    (property "Reference" "#PWR0602" (id 0) (at 220.98 74.93 0)
       (effects (font (size 1.27 1.27)) hide)
     )
@@
   (symbol (lib_id "power:GND") (at 104.14 113.03 0)
     (in_bom yes) (on_board yes)
-    (property "Reference" "#PWR0608" (id 0) (at 104.14 119.38 0)
+    (property "Reference" "#PWR0604" (id 0) (at 104.14 119.38 0)
       (effects (font (size 1.27 1.27)) hide)
     )
@@
     (pin "1")
   )
-  (symbol (lib_id "power:GND") (at 184.15 52.07 0)
+  (symbol (lib_id "power:GND") (at 219.71 48.26 0)
     (in_bom yes) (on_board yes)
-    (property "Reference" "#PWR0605" (id 0) (at 184.15 58.42 0)
+    (property "Reference" "#PWR0601" (id 0) (at 219.71 54.61 0)
       (effects (font (size 1.27 1.27)) hide)
     )
-    (property "Value" "GND" (id 1) (at 184.277 56.4642 0))
-    (property "Footprint" "" (id 2) (at 184.15 52.07 0)
+    (property "Value" "GND" (id 1) (at 219.837 52.6542 0))
+    (property "Footprint" "" (id 2) (at 219.71 48.26 0)
       (effects (font (size 1.27 1.27)) hide)
     )
-    (property "Datasheet" "" (id 3) (at 184.15 52.07 0)
+    (property "Datasheet" "" (id 3) (at 219.71 48.26 0)
       (effects (font (size 1.27 1.27)) hide)
     )
@@
   (symbol (lib_id "power:GND") (at 220.98 109.22 0)
     (in_bom yes) (on_board yes)
-    (property "Reference" "#PWR0607" (id 0) (at 220.98 115.57 0)
+    (property "Reference" "#PWR0603" (id 0) (at 220.98 115.57 0)
       (effects (font (size 1.27 1.27)) hide)
     )
@@
   (symbol (lib_id "Device:R") (at 200.66 44.45 0)
     (in_bom yes) (on_board yes)
-    (property "Reference" "R300" (id 0) (at 202.438 43.2816 0)
+    (property "Reference" "R298" (id 0) (at 202.438 43.2816 0)
       (effects (font (size 1.27 1.27)) (justify left))
     )
@@
   (symbol (lib_id "Device:R") (at 220.98 74.93 0)
     (in_bom yes) (on_board yes)
-    (property "Reference" "R301" (id 0) (at 222.758 73.7616 0)
+    (property "Reference" "R299" (id 0) (at 222.758 73.7616 0)
       (effects (font (size 1.27 1.27)) (justify left))
     )
@@
     (pin "2")
   )
-  (symbol (lib_id "Device:C") (at 184.15 48.26 0)
+  (symbol (lib_id "Device:C") (at 219.71 44.45 0)
     (in_bom yes) (on_board yes)
-    (property "Reference" "C21" (id 0) (at 187.071 47.0916 0)
+    (property "Reference" "C21" (id 0) (at 222.631 43.2816 0)
       (effects (font (size 1.27 1.27)) (justify left))
     )
-    (property "Value" "0.1u" (id 1) (at 187.071 49.403 0)
+    (property "Value" "0.1u" (id 1) (at 222.631 45.593 0)
       (effects (font (size 1.27 1.27)) (justify left))
     )
-    (property "Footprint" "Capacitor_SMD:C_0805_2012Metric" (id 2) (at 185.1152 52.07 0)
+    (property "Footprint" "Capacitor_SMD:C_0805_2012Metric" (id 2) (at 220.6752 48.26 0)
       (effects (font (size 1.27 1.27)) hide)
     )
-    (property "Datasheet" "~" (id 3) (at 184.15 48.26 0)
+    (property "Datasheet" "~" (id 3) (at 219.71 44.45 0)
       (effects (font (size 1.27 1.27)) hide)
     )
-    (property "LCSC" "C49678" (id 4) (at 184.15 48.26 0)
+    (property "LCSC" "C49678" (id 4) (at 219.71 44.45 0)
       (effects (font (size 1.27 1.27)) hide)
     )
@@
   (symbol (lib_id "Transistor_FET:2N7002") (at 218.44 93.98 0)
     (in_bom yes) (on_board yes)
-    (property "Reference" "Q693" (id 0) (at 223.6724 92.8116 0)
+    (property "Reference" "Q691" (id 0) (at 223.6724 92.8116 0)
       (effects (font (size 1.27 1.27)) (justify left))
     )
@@
   (symbol (lib_id "Transistor_FET:2N7002") (at 218.44 104.14 0)
     (in_bom yes) (on_board yes)
-    (property "Reference" "Q694" (id 0) (at 223.6724 102.9716 0)
+    (property "Reference" "Q692" (id 0) (at 223.6724 102.9716 0)
       (effects (font (size 1.27 1.27)) (justify left))
     )
