File: pcb/preg.kicad_sch (KiCad schematic)
At the start: 13 parts, among them Q85 2N7002a, Q86 2N7002a, Q87 2N7002a, Q88 2N7002a, Q89 2N7002a, Q90 2N7002a, Q91 2N7002b, Q92 2N7002b, Q93 2N7002b, Q94 2N7002a, Q95 2N7002b

Commit message: Pi programmer.
Parts:
- renumbered Q85 to Q1114, Q86 to Q1115, Q87 to Q1116, Q88 to Q1117, Q89 to Q1118, Q90 to Q1119, Q91 to Q1120, Q92 to Q1121, Q93 to Q1122, Q94 to Q1123, Q95 to Q1124, R38 to R481, R39 to R482
Changed lines of the file:
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@@
   (symbol (lib_id "power:VCC") (at 85.09 156.21 0)
     (in_bom yes) (on_board yes)
-    (property "Reference" "#PWR0108" (id 0) (at 85.09 160.02 0)
+    (property "Reference" "#PWR01006" (id 0) (at 85.09 160.02 0)
       (effects (font (size 1.27 1.27)) hide)
     )
@@
   (symbol (lib_id "power:VCC") (at 109.22 156.21 0)
     (in_bom yes) (on_board yes)
-    (property "Reference" "#PWR0109" (id 0) (at 109.22 160.02 0)
+    (property "Reference" "#PWR01007" (id 0) (at 109.22 160.02 0)
       (effects (font (size 1.27 1.27)) hide)
     )
@@
   (symbol (lib_id "power:GND") (at 49.53 143.51 0)
     (in_bom yes) (on_board yes)
-    (property "Reference" "#PWR0104" (id 0) (at 49.53 149.86 0)
+    (property "Reference" "#PWR01002" (id 0) (at 49.53 149.86 0)
       (effects (font (size 1.27 1.27)) hide)
     )
@@
   (symbol (lib_id "power:GND") (at 73.66 143.51 0)
     (in_bom yes) (on_board yes)
-    (property "Reference" "#PWR0105" (id 0) (at 73.66 149.86 0)
+    (property "Reference" "#PWR01003" (id 0) (at 73.66 149.86 0)
       (effects (font (size 1.27 1.27)) hide)
     )
@@
   (symbol (lib_id "power:GND") (at 100.33 143.51 0)
     (in_bom yes) (on_board yes)
-    (property "Reference" "#PWR0106" (id 0) (at 100.33 149.86 0)
+    (property "Reference" "#PWR01004" (id 0) (at 100.33 149.86 0)
       (effects (font (size 1.27 1.27)) hide)
     )
@@
   (symbol (lib_id "power:GND") (at 109.22 177.8 0)
     (in_bom yes) (on_board yes)
-    (property "Reference" "#PWR0110" (id 0) (at 109.22 184.15 0)
+    (property "Reference" "#PWR01008" (id 0) (at 109.22 184.15 0)
       (effects (font (size 1.27 1.27)) hide)
     )
@@
   (symbol (lib_id "power:GND") (at 125.73 143.51 0)
     (in_bom yes) (on_board yes)
-    (property "Reference" "#PWR0107" (id 0) (at 125.73 149.86 0)
+    (property "Reference" "#PWR01005" (id 0) (at 125.73 149.86 0)
       (effects (font (size 1.27 1.27)) hide)
     )
@@
   (symbol (lib_id "power:GND") (at 149.86 93.98 0)
     (in_bom yes) (on_board yes)
-    (property "Reference" "#PWR0103" (id 0) (at 149.86 100.33 0)
+    (property "Reference" "#PWR01001" (id 0) (at 149.86 100.33 0)
       (effects (font (size 1.27 1.27)) hide)
     )
@@
   (symbol (lib_id "Device:R") (at 85.09 160.02 0)
     (in_bom yes) (on_board yes)
-    (property "Reference" "R38" (id 0) (at 86.868 158.8516 0)
+    (property "Reference" "R481" (id 0) (at 86.868 158.8516 0)
       (effects (font (size 1.27 1.27)) (justify left))
     )
@@
   (symbol (lib_id "Device:R") (at 109.22 160.02 0)
     (in_bom yes) (on_board yes)
-    (property "Reference" "R39" (id 0) (at 110.998 158.8516 0)
+    (property "Reference" "R482" (id 0) (at 110.998 158.8516 0)
       (effects (font (size 1.27 1.27)) (justify left))
     )
@@
   (symbol (lib_id "Transistor_FET:2N7002") (at 46.99 123.19 0)
     (in_bom yes) (on_board yes)
-    (property "Reference" "Q87" (id 0) (at 52.2224 122.0216 0)
+    (property "Reference" "Q1116" (id 0) (at 52.2224 122.0216 0)
       (effects (font (size 1.27 1.27)) (justify left))
     )
@@
   (symbol (lib_id "Transistor_FET:2N7002") (at 46.99 138.43 0)
     (in_bom yes) (on_board yes)
-    (property "Reference" "Q91" (id 0) (at 52.2224 137.2616 0)
+    (property "Reference" "Q1120" (id 0) (at 52.2224 137.2616 0)
       (effects (font (size 1.27 1.27)) (justify left))
     )
@@
   (symbol (lib_id "Transistor_FET:2N7002") (at 71.12 123.19 0)
     (in_bom yes) (on_board yes)
-    (property "Reference" "Q88" (id 0) (at 76.3524 122.0216 0)
+    (property "Reference" "Q1117" (id 0) (at 76.3524 122.0216 0)
       (effects (font (size 1.27 1.27)) (justify left))
     )
@@
   (symbol (lib_id "Transistor_FET:2N7002") (at 71.12 138.43 0)
     (in_bom yes) (on_board yes)
-    (property "Reference" "Q92" (id 0) (at 76.3524 137.2616 0)
+    (property "Reference" "Q1121" (id 0) (at 76.3524 137.2616 0)
       (effects (font (size 1.27 1.27)) (justify left))
     )
@@
   (symbol (lib_id "Transistor_FET:2N7002") (at 97.79 123.19 0)
     (in_bom yes) (on_board yes)
-    (property "Reference" "Q89" (id 0) (at 103.0224 122.0216 0)
+    (property "Reference" "Q1118" (id 0) (at 103.0224 122.0216 0)
       (effects (font (size 1.27 1.27)) (justify left))
     )
@@
   (symbol (lib_id "Transistor_FET:2N7002") (at 97.79 138.43 0)
     (in_bom yes) (on_board yes)
-    (property "Reference" "Q93" (id 0) (at 103.0224 137.2616 0)
+    (property "Reference" "Q1122" (id 0) (at 103.0224 137.2616 0)
       (effects (font (size 1.27 1.27)) (justify left))
     )
@@
   (symbol (lib_id "Transistor_FET:2N7002") (at 106.68 172.72 0)
     (in_bom yes) (on_board yes)
-    (property "Reference" "Q95" (id 0) (at 111.9124 171.5516 0)
+    (property "Reference" "Q1124" (id 0) (at 111.9124 171.5516 0)
       (effects (font (size 1.27 1.27)) (justify left))
     )
@@
   (symbol (lib_id "Transistor_FET:2N7002") (at 123.19 123.19 0)
     (in_bom yes) (on_board yes)
-    (property "Reference" "Q90" (id 0) (at 128.4224 122.0216 0)
+    (property "Reference" "Q1119" (id 0) (at 128.4224 122.0216 0)
       (effects (font (size 1.27 1.27)) (justify left))
     )
@@
   (symbol (lib_id "Transistor_FET:2N7002") (at 123.19 138.43 0)
     (in_bom yes) (on_board yes)
-    (property "Reference" "Q94" (id 0) (at 128.4224 137.2616 0)
+    (property "Reference" "Q1123" (id 0) (at 128.4224 137.2616 0)
       (effects (font (size 1.27 1.27)) (justify left))
     )
@@
   (symbol (lib_id "Transistor_FET:2N7002") (at 147.32 78.74 0)
     (in_bom yes) (on_board yes)
-    (property "Reference" "Q85" (id 0) (at 152.5524 77.5716 0)
+    (property "Reference" "Q1114" (id 0) (at 152.5524 77.5716 0)
       (effects (font (size 1.27 1.27)) (justify left))
     )
@@
   (symbol (lib_id "Transistor_FET:2N7002") (at 147.32 88.9 0)
     (in_bom yes) (on_board yes)
-    (property "Reference" "Q86" (id 0) (at 152.5524 87.7316 0)
-      (effects (font (size 1.27 1.27)) (justify left))
-    )
+    (property "Reference" "Q1115" (id 0) (at 152.5524 87.7316 0)
+      (effects (font (size 1.27 1.27)) (justify left))
+    )

Commit message: Buttons.
Parts:
- renumbered R481 to R482, R482 to R483
Changed lines of the file:
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@@
   (symbol (lib_id "Device:R") (at 85.09 160.02 0)
     (in_bom yes) (on_board yes)
-    (property "Reference" "R481" (id 0) (at 86.868 158.8516 0)
+    (property "Reference" "R482" (id 0) (at 86.868 158.8516 0)
       (effects (font (size 1.27 1.27)) (justify left))
     )
@@
   (symbol (lib_id "Device:R") (at 109.22 160.02 0)
     (in_bom yes) (on_board yes)
-    (property "Reference" "R482" (id 0) (at 110.998 158.8516 0)
+    (property "Reference" "R483" (id 0) (at 110.998 158.8516 0)
       (effects (font (size 1.27 1.27)) (justify left))
     )

Commit message: Fix UUIDs.
Parts:
- renumbered Q1114 to Q1093, Q1115 to Q1094, Q1116 to Q1095, Q1117 to Q1096, Q1118 to Q1097, Q1119 to Q1098, Q1120 to Q1099, Q1121 to Q1100, Q1122 to Q1101, Q1123 to Q1102, Q1124 to Q1103
Changed lines of the file:
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@@
   (symbol (lib_id "power:VCC") (at 85.09 156.21 0)
     (in_bom yes) (on_board yes)
-    (property "Reference" "#PWR01006" (id 0) (at 85.09 160.02 0)
+    (property "Reference" "#PWR0978" (id 0) (at 85.09 160.02 0)
       (effects (font (size 1.27 1.27)) hide)
     )
@@
   (symbol (lib_id "power:VCC") (at 109.22 156.21 0)
     (in_bom yes) (on_board yes)
-    (property "Reference" "#PWR01007" (id 0) (at 109.22 160.02 0)
+    (property "Reference" "#PWR0979" (id 0) (at 109.22 160.02 0)
       (effects (font (size 1.27 1.27)) hide)
     )
@@
   (symbol (lib_id "power:GND") (at 49.53 143.51 0)
     (in_bom yes) (on_board yes)
-    (property "Reference" "#PWR01002" (id 0) (at 49.53 149.86 0)
+    (property "Reference" "#PWR0974" (id 0) (at 49.53 149.86 0)
       (effects (font (size 1.27 1.27)) hide)
     )
@@
   (symbol (lib_id "power:GND") (at 73.66 143.51 0)
     (in_bom yes) (on_board yes)
-    (property "Reference" "#PWR01003" (id 0) (at 73.66 149.86 0)
+    (property "Reference" "#PWR0975" (id 0) (at 73.66 149.86 0)
       (effects (font (size 1.27 1.27)) hide)
     )
@@
   (symbol (lib_id "power:GND") (at 100.33 143.51 0)
     (in_bom yes) (on_board yes)
-    (property "Reference" "#PWR01004" (id 0) (at 100.33 149.86 0)
+    (property "Reference" "#PWR0976" (id 0) (at 100.33 149.86 0)
       (effects (font (size 1.27 1.27)) hide)
     )
@@
   (symbol (lib_id "power:GND") (at 109.22 177.8 0)
     (in_bom yes) (on_board yes)
-    (property "Reference" "#PWR01008" (id 0) (at 109.22 184.15 0)
+    (property "Reference" "#PWR0980" (id 0) (at 109.22 184.15 0)
       (effects (font (size 1.27 1.27)) hide)
     )
@@
   (symbol (lib_id "power:GND") (at 125.73 143.51 0)
     (in_bom yes) (on_board yes)
-    (property "Reference" "#PWR01005" (id 0) (at 125.73 149.86 0)
+    (property "Reference" "#PWR0977" (id 0) (at 125.73 149.86 0)
       (effects (font (size 1.27 1.27)) hide)
     )
@@
   (symbol (lib_id "power:GND") (at 149.86 93.98 0)
     (in_bom yes) (on_board yes)
-    (property "Reference" "#PWR01001" (id 0) (at 149.86 100.33 0)
+    (property "Reference" "#PWR0973" (id 0) (at 149.86 100.33 0)
       (effects (font (size 1.27 1.27)) hide)
     )
@@
   (symbol (lib_id "Transistor_FET:2N7002") (at 46.99 123.19 0)
     (in_bom yes) (on_board yes)
-    (property "Reference" "Q1116" (id 0) (at 52.2224 122.0216 0)
+    (property "Reference" "Q1095" (id 0) (at 52.2224 122.0216 0)
       (effects (font (size 1.27 1.27)) (justify left))
     )
@@
   (symbol (lib_id "Transistor_FET:2N7002") (at 46.99 138.43 0)
     (in_bom yes) (on_board yes)
-    (property "Reference" "Q1120" (id 0) (at 52.2224 137.2616 0)
+    (property "Reference" "Q1099" (id 0) (at 52.2224 137.2616 0)
       (effects (font (size 1.27 1.27)) (justify left))
     )
@@
   (symbol (lib_id "Transistor_FET:2N7002") (at 71.12 123.19 0)
     (in_bom yes) (on_board yes)
-    (property "Reference" "Q1117" (id 0) (at 76.3524 122.0216 0)
+    (property "Reference" "Q1096" (id 0) (at 76.3524 122.0216 0)
       (effects (font (size 1.27 1.27)) (justify left))
     )
@@
   (symbol (lib_id "Transistor_FET:2N7002") (at 71.12 138.43 0)
     (in_bom yes) (on_board yes)
-    (property "Reference" "Q1121" (id 0) (at 76.3524 137.2616 0)
+    (property "Reference" "Q1100" (id 0) (at 76.3524 137.2616 0)
       (effects (font (size 1.27 1.27)) (justify left))
     )
@@
   (symbol (lib_id "Transistor_FET:2N7002") (at 97.79 123.19 0)
     (in_bom yes) (on_board yes)
-    (property "Reference" "Q1118" (id 0) (at 103.0224 122.0216 0)
+    (property "Reference" "Q1097" (id 0) (at 103.0224 122.0216 0)
       (effects (font (size 1.27 1.27)) (justify left))
     )
@@
   (symbol (lib_id "Transistor_FET:2N7002") (at 97.79 138.43 0)
     (in_bom yes) (on_board yes)
-    (property "Reference" "Q1122" (id 0) (at 103.0224 137.2616 0)
+    (property "Reference" "Q1101" (id 0) (at 103.0224 137.2616 0)
       (effects (font (size 1.27 1.27)) (justify left))
     )
@@
   (symbol (lib_id "Transistor_FET:2N7002") (at 106.68 172.72 0)
     (in_bom yes) (on_board yes)
-    (property "Reference" "Q1124" (id 0) (at 111.9124 171.5516 0)
+    (property "Reference" "Q1103" (id 0) (at 111.9124 171.5516 0)
       (effects (font (size 1.27 1.27)) (justify left))
     )
@@
   (symbol (lib_id "Transistor_FET:2N7002") (at 123.19 123.19 0)
     (in_bom yes) (on_board yes)
-    (property "Reference" "Q1119" (id 0) (at 128.4224 122.0216 0)
+    (property "Reference" "Q1098" (id 0) (at 128.4224 122.0216 0)
       (effects (font (size 1.27 1.27)) (justify left))
     )
@@
   (symbol (lib_id "Transistor_FET:2N7002") (at 123.19 138.43 0)
     (in_bom yes) (on_board yes)
-    (property "Reference" "Q1123" (id 0) (at 128.4224 137.2616 0)
+    (property "Reference" "Q1102" (id 0) (at 128.4224 137.2616 0)
       (effects (font (size 1.27 1.27)) (justify left))
     )
@@
   (symbol (lib_id "Transistor_FET:2N7002") (at 147.32 78.74 0)
     (in_bom yes) (on_board yes)
-    (property "Reference" "Q1114" (id 0) (at 152.5524 77.5716 0)
+    (property "Reference" "Q1093" (id 0) (at 152.5524 77.5716 0)
       (effects (font (size 1.27 1.27)) (justify left))
     )
@@
   (symbol (lib_id "Transistor_FET:2N7002") (at 147.32 88.9 0)
     (in_bom yes) (on_board yes)
-    (property "Reference" "Q1115" (id 0) (at 152.5524 87.7316 0)
-      (effects (font (size 1.27 1.27)) (justify left))
-    )
+    (property "Reference" "Q1094" (id 0) (at 152.5524 87.7316 0)
+      (effects (font (size 1.27 1.27)) (justify left))
+    )

Commit message: New reset.
Parts:
- renumbered R482 to R481, R483 to R482
Changed lines of the file:
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@@
   (symbol (lib_id "power:VCC") (at 85.09 156.21 0)
     (in_bom yes) (on_board yes)
-    (property "Reference" "#PWR0978" (id 0) (at 85.09 160.02 0)
+    (property "Reference" "#PWR0977" (id 0) (at 85.09 160.02 0)
       (effects (font (size 1.27 1.27)) hide)
     )
@@
   (symbol (lib_id "power:VCC") (at 109.22 156.21 0)
     (in_bom yes) (on_board yes)
-    (property "Reference" "#PWR0979" (id 0) (at 109.22 160.02 0)
+    (property "Reference" "#PWR0978" (id 0) (at 109.22 160.02 0)
       (effects (font (size 1.27 1.27)) hide)
     )
@@
   (symbol (lib_id "power:GND") (at 49.53 143.51 0)
     (in_bom yes) (on_board yes)
-    (property "Reference" "#PWR0974" (id 0) (at 49.53 149.86 0)
+    (property "Reference" "#PWR0973" (id 0) (at 49.53 149.86 0)
       (effects (font (size 1.27 1.27)) hide)
     )
@@
   (symbol (lib_id "power:GND") (at 73.66 143.51 0)
     (in_bom yes) (on_board yes)
-    (property "Reference" "#PWR0975" (id 0) (at 73.66 149.86 0)
+    (property "Reference" "#PWR0974" (id 0) (at 73.66 149.86 0)
       (effects (font (size 1.27 1.27)) hide)
     )
@@
   (symbol (lib_id "power:GND") (at 100.33 143.51 0)
     (in_bom yes) (on_board yes)
-    (property "Reference" "#PWR0976" (id 0) (at 100.33 149.86 0)
+    (property "Reference" "#PWR0975" (id 0) (at 100.33 149.86 0)
       (effects (font (size 1.27 1.27)) hide)
     )
@@
   (symbol (lib_id "power:GND") (at 109.22 177.8 0)
     (in_bom yes) (on_board yes)
-    (property "Reference" "#PWR0980" (id 0) (at 109.22 184.15 0)
+    (property "Reference" "#PWR0979" (id 0) (at 109.22 184.15 0)
       (effects (font (size 1.27 1.27)) hide)
     )
@@
   (symbol (lib_id "power:GND") (at 125.73 143.51 0)
     (in_bom yes) (on_board yes)
-    (property "Reference" "#PWR0977" (id 0) (at 125.73 149.86 0)
+    (property "Reference" "#PWR0976" (id 0) (at 125.73 149.86 0)
       (effects (font (size 1.27 1.27)) hide)
     )
@@
   (symbol (lib_id "power:GND") (at 149.86 93.98 0)
     (in_bom yes) (on_board yes)
-    (property "Reference" "#PWR0973" (id 0) (at 149.86 100.33 0)
+    (property "Reference" "#PWR0972" (id 0) (at 149.86 100.33 0)
       (effects (font (size 1.27 1.27)) hide)
     )
@@
   (symbol (lib_id "Device:R") (at 85.09 160.02 0)
     (in_bom yes) (on_board yes)
-    (property "Reference" "R482" (id 0) (at 86.868 158.8516 0)
+    (property "Reference" "R481" (id 0) (at 86.868 158.8516 0)
       (effects (font (size 1.27 1.27)) (justify left))
     )
@@
   (symbol (lib_id "Device:R") (at 109.22 160.02 0)
     (in_bom yes) (on_board yes)
-    (property "Reference" "R483" (id 0) (at 110.998 158.8516 0)
+    (property "Reference" "R482" (id 0) (at 110.998 158.8516 0)
       (effects (font (size 1.27 1.27)) (justify left))
     )

Commit message: Some fixes.
Parts:
- renumbered Q1093 to Q1089, Q1094 to Q1090, Q1095 to Q1091, Q1096 to Q1092, Q1097 to Q1093, Q1098 to Q1094, Q1099 to Q1095, Q1100 to Q1096, Q1101 to Q1097, Q1102 to Q1098, Q1103 to Q1099, R481 to R485, R482 to R486
Changed lines of the file:
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@@
   (symbol (lib_id "power:VCC") (at 85.09 156.21 0)
     (in_bom yes) (on_board yes)
-    (property "Reference" "#PWR0977" (id 0) (at 85.09 160.02 0)
+    (property "Reference" "#PWR0987" (id 0) (at 85.09 160.02 0)
       (effects (font (size 1.27 1.27)) hide)
     )
@@
   (symbol (lib_id "power:VCC") (at 109.22 156.21 0)
     (in_bom yes) (on_board yes)
-    (property "Reference" "#PWR0978" (id 0) (at 109.22 160.02 0)
+    (property "Reference" "#PWR0988" (id 0) (at 109.22 160.02 0)
       (effects (font (size 1.27 1.27)) hide)
     )
@@
   (symbol (lib_id "power:GND") (at 49.53 143.51 0)
     (in_bom yes) (on_board yes)
-    (property "Reference" "#PWR0973" (id 0) (at 49.53 149.86 0)
+    (property "Reference" "#PWR0983" (id 0) (at 49.53 149.86 0)
       (effects (font (size 1.27 1.27)) hide)
     )
@@
   (symbol (lib_id "power:GND") (at 73.66 143.51 0)
     (in_bom yes) (on_board yes)
-    (property "Reference" "#PWR0974" (id 0) (at 73.66 149.86 0)
+    (property "Reference" "#PWR0984" (id 0) (at 73.66 149.86 0)
       (effects (font (size 1.27 1.27)) hide)
     )
@@
   (symbol (lib_id "power:GND") (at 100.33 143.51 0)
     (in_bom yes) (on_board yes)
-    (property "Reference" "#PWR0975" (id 0) (at 100.33 149.86 0)
+    (property "Reference" "#PWR0985" (id 0) (at 100.33 149.86 0)
       (effects (font (size 1.27 1.27)) hide)
     )
@@
   (symbol (lib_id "power:GND") (at 109.22 177.8 0)
     (in_bom yes) (on_board yes)
-    (property "Reference" "#PWR0979" (id 0) (at 109.22 184.15 0)
+    (property "Reference" "#PWR0989" (id 0) (at 109.22 184.15 0)
       (effects (font (size 1.27 1.27)) hide)
     )
@@
   (symbol (lib_id "power:GND") (at 125.73 143.51 0)
     (in_bom yes) (on_board yes)
-    (property "Reference" "#PWR0976" (id 0) (at 125.73 149.86 0)
+    (property "Reference" "#PWR0986" (id 0) (at 125.73 149.86 0)
       (effects (font (size 1.27 1.27)) hide)
     )
@@
   (symbol (lib_id "power:GND") (at 149.86 93.98 0)
     (in_bom yes) (on_board yes)
-    (property "Reference" "#PWR0972" (id 0) (at 149.86 100.33 0)
+    (property "Reference" "#PWR0982" (id 0) (at 149.86 100.33 0)
       (effects (font (size 1.27 1.27)) hide)
     )
@@
   (symbol (lib_id "Device:R") (at 85.09 160.02 0)
     (in_bom yes) (on_board yes)
-    (property "Reference" "R481" (id 0) (at 86.868 158.8516 0)
+    (property "Reference" "R485" (id 0) (at 86.868 158.8516 0)
       (effects (font (size 1.27 1.27)) (justify left))
     )
@@
   (symbol (lib_id "Device:R") (at 109.22 160.02 0)
     (in_bom yes) (on_board yes)
-    (property "Reference" "R482" (id 0) (at 110.998 158.8516 0)
+    (property "Reference" "R486" (id 0) (at 110.998 158.8516 0)
       (effects (font (size 1.27 1.27)) (justify left))
     )
@@
   (symbol (lib_id "Transistor_FET:2N7002") (at 46.99 123.19 0)
     (in_bom yes) (on_board yes)
-    (property "Reference" "Q1095" (id 0) (at 52.2224 122.0216 0)
+    (property "Reference" "Q1091" (id 0) (at 52.2224 122.0216 0)
       (effects (font (size 1.27 1.27)) (justify left))
     )
@@
   (symbol (lib_id "Transistor_FET:2N7002") (at 46.99 138.43 0)
     (in_bom yes) (on_board yes)
-    (property "Reference" "Q1099" (id 0) (at 52.2224 137.2616 0)
+    (property "Reference" "Q1095" (id 0) (at 52.2224 137.2616 0)
       (effects (font (size 1.27 1.27)) (justify left))
     )
@@
   (symbol (lib_id "Transistor_FET:2N7002") (at 71.12 123.19 0)
     (in_bom yes) (on_board yes)
-    (property "Reference" "Q1096" (id 0) (at 76.3524 122.0216 0)
+    (property "Reference" "Q1092" (id 0) (at 76.3524 122.0216 0)
       (effects (font (size 1.27 1.27)) (justify left))
     )
@@
   (symbol (lib_id "Transistor_FET:2N7002") (at 71.12 138.43 0)
     (in_bom yes) (on_board yes)
-    (property "Reference" "Q1100" (id 0) (at 76.3524 137.2616 0)
+    (property "Reference" "Q1096" (id 0) (at 76.3524 137.2616 0)
       (effects (font (size 1.27 1.27)) (justify left))
     )
@@
   (symbol (lib_id "Transistor_FET:2N7002") (at 97.79 123.19 0)
     (in_bom yes) (on_board yes)
-    (property "Reference" "Q1097" (id 0) (at 103.0224 122.0216 0)
+    (property "Reference" "Q1093" (id 0) (at 103.0224 122.0216 0)
       (effects (font (size 1.27 1.27)) (justify left))
     )
@@
   (symbol (lib_id "Transistor_FET:2N7002") (at 97.79 138.43 0)
     (in_bom yes) (on_board yes)
-    (property "Reference" "Q1101" (id 0) (at 103.0224 137.2616 0)
+    (property "Reference" "Q1097" (id 0) (at 103.0224 137.2616 0)
       (effects (font (size 1.27 1.27)) (justify left))
     )
@@
   (symbol (lib_id "Transistor_FET:2N7002") (at 106.68 172.72 0)
     (in_bom yes) (on_board yes)
-    (property "Reference" "Q1103" (id 0) (at 111.9124 171.5516 0)
+    (property "Reference" "Q1099" (id 0) (at 111.9124 171.5516 0)
       (effects (font (size 1.27 1.27)) (justify left))
     )
@@
   (symbol (lib_id "Transistor_FET:2N7002") (at 123.19 123.19 0)
     (in_bom yes) (on_board yes)
-    (property "Reference" "Q1098" (id 0) (at 128.4224 122.0216 0)
+    (property "Reference" "Q1094" (id 0) (at 128.4224 122.0216 0)
       (effects (font (size 1.27 1.27)) (justify left))
     )
@@
   (symbol (lib_id "Transistor_FET:2N7002") (at 123.19 138.43 0)
     (in_bom yes) (on_board yes)
-    (property "Reference" "Q1102" (id 0) (at 128.4224 137.2616 0)
+    (property "Reference" "Q1098" (id 0) (at 128.4224 137.2616 0)
       (effects (font (size 1.27 1.27)) (justify left))
     )
@@
   (symbol (lib_id "Transistor_FET:2N7002") (at 147.32 78.74 0)
     (in_bom yes) (on_board yes)
-    (property "Reference" "Q1093" (id 0) (at 152.5524 77.5716 0)
+    (property "Reference" "Q1089" (id 0) (at 152.5524 77.5716 0)
       (effects (font (size 1.27 1.27)) (justify left))
     )
@@
   (symbol (lib_id "Transistor_FET:2N7002") (at 147.32 88.9 0)
     (in_bom yes) (on_board yes)
-    (property "Reference" "Q1094" (id 0) (at 152.5524 87.7316 0)
-      (effects (font (size 1.27 1.27)) (justify left))
-    )
+    (property "Reference" "Q1090" (id 0) (at 152.5524 87.7316 0)
+      (effects (font (size 1.27 1.27)) (justify left))
+    )
