File: pcb/preg.kicad_sch (KiCad schematic)
At the start: 13 parts, among them Q1089 2N7002a, Q1090 2N7002a, Q1091 2N7002a, Q1092 2N7002a, Q1093 2N7002a, Q1094 2N7002a, Q1095 2N7002b, Q1096 2N7002b, Q1097 2N7002b, Q1098 2N7002a, Q1099 2N7002b

Commit message: Faster.
Parts:
- renumbered Q1089 to Q1087, Q1090 to Q1088, Q1091 to Q1089, Q1092 to Q1090, Q1093 to Q1091, Q1094 to Q1092, Q1095 to Q1093, Q1096 to Q1094, Q1097 to Q1095, Q1098 to Q1096, Q1099 to Q1097, R485 to R483, R486 to R484
Changed lines of the file:
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@@
   (symbol (lib_id "power:VCC") (at 85.09 156.21 0)
     (in_bom yes) (on_board yes)
-    (property "Reference" "#PWR0987" (id 0) (at 85.09 160.02 0)
+    (property "Reference" "#PWR0984" (id 0) (at 85.09 160.02 0)
       (effects (font (size 1.27 1.27)) hide)
     )
@@
   (symbol (lib_id "power:VCC") (at 109.22 156.21 0)
     (in_bom yes) (on_board yes)
-    (property "Reference" "#PWR0988" (id 0) (at 109.22 160.02 0)
+    (property "Reference" "#PWR0985" (id 0) (at 109.22 160.02 0)
       (effects (font (size 1.27 1.27)) hide)
     )
@@
   (symbol (lib_id "power:GND") (at 49.53 143.51 0)
     (in_bom yes) (on_board yes)
-    (property "Reference" "#PWR0983" (id 0) (at 49.53 149.86 0)
+    (property "Reference" "#PWR0980" (id 0) (at 49.53 149.86 0)
       (effects (font (size 1.27 1.27)) hide)
     )
@@
   (symbol (lib_id "power:GND") (at 73.66 143.51 0)
     (in_bom yes) (on_board yes)
-    (property "Reference" "#PWR0984" (id 0) (at 73.66 149.86 0)
+    (property "Reference" "#PWR0981" (id 0) (at 73.66 149.86 0)
       (effects (font (size 1.27 1.27)) hide)
     )
@@
   (symbol (lib_id "power:GND") (at 100.33 143.51 0)
     (in_bom yes) (on_board yes)
-    (property "Reference" "#PWR0985" (id 0) (at 100.33 149.86 0)
+    (property "Reference" "#PWR0982" (id 0) (at 100.33 149.86 0)
       (effects (font (size 1.27 1.27)) hide)
     )
@@
   (symbol (lib_id "power:GND") (at 109.22 177.8 0)
     (in_bom yes) (on_board yes)
-    (property "Reference" "#PWR0989" (id 0) (at 109.22 184.15 0)
+    (property "Reference" "#PWR0986" (id 0) (at 109.22 184.15 0)
       (effects (font (size 1.27 1.27)) hide)
     )
@@
   (symbol (lib_id "power:GND") (at 125.73 143.51 0)
     (in_bom yes) (on_board yes)
-    (property "Reference" "#PWR0986" (id 0) (at 125.73 149.86 0)
+    (property "Reference" "#PWR0983" (id 0) (at 125.73 149.86 0)
       (effects (font (size 1.27 1.27)) hide)
     )
@@
   (symbol (lib_id "power:GND") (at 149.86 93.98 0)
     (in_bom yes) (on_board yes)
-    (property "Reference" "#PWR0982" (id 0) (at 149.86 100.33 0)
+    (property "Reference" "#PWR0979" (id 0) (at 149.86 100.33 0)
       (effects (font (size 1.27 1.27)) hide)
     )
@@
   (symbol (lib_id "Device:R") (at 85.09 160.02 0)
     (in_bom yes) (on_board yes)
-    (property "Reference" "R485" (id 0) (at 86.868 158.8516 0)
+    (property "Reference" "R483" (id 0) (at 86.868 158.8516 0)
       (effects (font (size 1.27 1.27)) (justify left))
     )
@@
   (symbol (lib_id "Device:R") (at 109.22 160.02 0)
     (in_bom yes) (on_board yes)
-    (property "Reference" "R486" (id 0) (at 110.998 158.8516 0)
+    (property "Reference" "R484" (id 0) (at 110.998 158.8516 0)
       (effects (font (size 1.27 1.27)) (justify left))
     )
@@
   (symbol (lib_id "Transistor_FET:2N7002") (at 46.99 123.19 0)
     (in_bom yes) (on_board yes)
-    (property "Reference" "Q1091" (id 0) (at 52.2224 122.0216 0)
+    (property "Reference" "Q1089" (id 0) (at 52.2224 122.0216 0)
       (effects (font (size 1.27 1.27)) (justify left))
     )
@@
   (symbol (lib_id "Transistor_FET:2N7002") (at 46.99 138.43 0)
     (in_bom yes) (on_board yes)
-    (property "Reference" "Q1095" (id 0) (at 52.2224 137.2616 0)
+    (property "Reference" "Q1093" (id 0) (at 52.2224 137.2616 0)
       (effects (font (size 1.27 1.27)) (justify left))
     )
@@
   (symbol (lib_id "Transistor_FET:2N7002") (at 71.12 123.19 0)
     (in_bom yes) (on_board yes)
-    (property "Reference" "Q1092" (id 0) (at 76.3524 122.0216 0)
+    (property "Reference" "Q1090" (id 0) (at 76.3524 122.0216 0)
       (effects (font (size 1.27 1.27)) (justify left))
     )
@@
   (symbol (lib_id "Transistor_FET:2N7002") (at 71.12 138.43 0)
     (in_bom yes) (on_board yes)
-    (property "Reference" "Q1096" (id 0) (at 76.3524 137.2616 0)
+    (property "Reference" "Q1094" (id 0) (at 76.3524 137.2616 0)
       (effects (font (size 1.27 1.27)) (justify left))
     )
@@
   (symbol (lib_id "Transistor_FET:2N7002") (at 97.79 123.19 0)
     (in_bom yes) (on_board yes)
-    (property "Reference" "Q1093" (id 0) (at 103.0224 122.0216 0)
+    (property "Reference" "Q1091" (id 0) (at 103.0224 122.0216 0)
       (effects (font (size 1.27 1.27)) (justify left))
     )
@@
   (symbol (lib_id "Transistor_FET:2N7002") (at 97.79 138.43 0)
     (in_bom yes) (on_board yes)
-    (property "Reference" "Q1097" (id 0) (at 103.0224 137.2616 0)
+    (property "Reference" "Q1095" (id 0) (at 103.0224 137.2616 0)
       (effects (font (size 1.27 1.27)) (justify left))
     )
@@
   (symbol (lib_id "Transistor_FET:2N7002") (at 106.68 172.72 0)
     (in_bom yes) (on_board yes)
-    (property "Reference" "Q1099" (id 0) (at 111.9124 171.5516 0)
+    (property "Reference" "Q1097" (id 0) (at 111.9124 171.5516 0)
       (effects (font (size 1.27 1.27)) (justify left))
     )
@@
   (symbol (lib_id "Transistor_FET:2N7002") (at 123.19 123.19 0)
     (in_bom yes) (on_board yes)
-    (property "Reference" "Q1094" (id 0) (at 128.4224 122.0216 0)
+    (property "Reference" "Q1092" (id 0) (at 128.4224 122.0216 0)
       (effects (font (size 1.27 1.27)) (justify left))
     )
@@
   (symbol (lib_id "Transistor_FET:2N7002") (at 123.19 138.43 0)
     (in_bom yes) (on_board yes)
-    (property "Reference" "Q1098" (id 0) (at 128.4224 137.2616 0)
+    (property "Reference" "Q1096" (id 0) (at 128.4224 137.2616 0)
       (effects (font (size 1.27 1.27)) (justify left))
     )
@@
   (symbol (lib_id "Transistor_FET:2N7002") (at 147.32 78.74 0)
     (in_bom yes) (on_board yes)
-    (property "Reference" "Q1089" (id 0) (at 152.5524 77.5716 0)
+    (property "Reference" "Q1087" (id 0) (at 152.5524 77.5716 0)
       (effects (font (size 1.27 1.27)) (justify left))
     )
@@
   (symbol (lib_id "Transistor_FET:2N7002") (at 147.32 88.9 0)
     (in_bom yes) (on_board yes)
-    (property "Reference" "Q1090" (id 0) (at 152.5524 87.7316 0)
-      (effects (font (size 1.27 1.27)) (justify left))
-    )
+    (property "Reference" "Q1088" (id 0) (at 152.5524 87.7316 0)
+      (effects (font (size 1.27 1.27)) (justify left))
+    )

Commit message: Updates
Parts:
- Q1087, Q1088, Q1089, Q1090, Q1091, Q1092, Q1096: value 2N7002a -> 2N7002; LCSC C8545 -> C181083
- Q1093, Q1094, Q1095, Q1097: value 2N7002b -> 2N7002K; LCSC C8545 -> C181083
- renumbered R483 to R484, R484 to R485

Commit message: Update resistors.
Parts:
- R482: renamed from R484; value 10k -> 100k; LCSC C17414 -> C17407
- renumbered Q1087 to Q1085, Q1088 to Q1086, Q1089 to Q1087, Q1090 to Q1088, Q1091 to Q1089, Q1092 to Q1090, Q1093 to Q1091, Q1094 to Q1092, Q1095 to Q1093, Q1096 to Q1094, Q1097 to Q1095, R485 to R483
Changed lines of the file:
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@@
   (symbol (lib_id "power:VCC") (at 85.09 156.21 0)
     (in_bom yes) (on_board yes)
-    (property "Reference" "#PWR0985" (id 0) (at 85.09 160.02 0)
+    (property "Reference" "#PWR0980" (id 0) (at 85.09 160.02 0)
       (effects (font (size 1.27 1.27)) hide)
     )
@@
   (symbol (lib_id "power:VCC") (at 109.22 156.21 0)
     (in_bom yes) (on_board yes)
-    (property "Reference" "#PWR0986" (id 0) (at 109.22 160.02 0)
+    (property "Reference" "#PWR0981" (id 0) (at 109.22 160.02 0)
       (effects (font (size 1.27 1.27)) hide)
     )
@@
   (symbol (lib_id "power:GND") (at 49.53 143.51 0)
     (in_bom yes) (on_board yes)
-    (property "Reference" "#PWR0981" (id 0) (at 49.53 149.86 0)
+    (property "Reference" "#PWR0976" (id 0) (at 49.53 149.86 0)
       (effects (font (size 1.27 1.27)) hide)
     )
@@
   (symbol (lib_id "power:GND") (at 73.66 143.51 0)
     (in_bom yes) (on_board yes)
-    (property "Reference" "#PWR0982" (id 0) (at 73.66 149.86 0)
+    (property "Reference" "#PWR0977" (id 0) (at 73.66 149.86 0)
       (effects (font (size 1.27 1.27)) hide)
     )
@@
   (symbol (lib_id "power:GND") (at 100.33 143.51 0)
     (in_bom yes) (on_board yes)
-    (property "Reference" "#PWR0983" (id 0) (at 100.33 149.86 0)
+    (property "Reference" "#PWR0978" (id 0) (at 100.33 149.86 0)
       (effects (font (size 1.27 1.27)) hide)
     )
@@
   (symbol (lib_id "power:GND") (at 109.22 182.88 0)
     (in_bom yes) (on_board yes)
-    (property "Reference" "#PWR0987" (id 0) (at 109.22 189.23 0)
+    (property "Reference" "#PWR0982" (id 0) (at 109.22 189.23 0)
       (effects (font (size 1.27 1.27)) hide)
     )
@@
   (symbol (lib_id "power:GND") (at 125.73 143.51 0)
     (in_bom yes) (on_board yes)
-    (property "Reference" "#PWR0984" (id 0) (at 125.73 149.86 0)
+    (property "Reference" "#PWR0979" (id 0) (at 125.73 149.86 0)
       (effects (font (size 1.27 1.27)) hide)
     )
@@
   (symbol (lib_id "power:GND") (at 149.86 93.98 0)
     (in_bom yes) (on_board yes)
-    (property "Reference" "#PWR0980" (id 0) (at 149.86 100.33 0)
+    (property "Reference" "#PWR0975" (id 0) (at 149.86 100.33 0)
       (effects (font (size 1.27 1.27)) hide)
     )
@@
   (symbol (lib_id "Device:R") (at 85.09 160.02 0)
     (in_bom yes) (on_board yes)
-    (property "Reference" "R484" (id 0) (at 86.868 158.8516 0)
-      (effects (font (size 1.27 1.27)) (justify left))
-    )
-    (property "Value" "10k" (id 1) (at 86.868 161.163 0)
+    (property "Reference" "R482" (id 0) (at 86.868 158.8516 0)
+      (effects (font (size 1.27 1.27)) (justify left))
+    )
+    (property "Value" "100k" (id 1) (at 86.868 161.163 0)
       (effects (font (size 1.27 1.27)) (justify left))
     )
@@
       (effects (font (size 1.27 1.27)) hide)
     )
-    (property "LCSC" "C17414" (id 4) (at 85.09 160.02 0)
+    (property "LCSC" "C17407" (id 4) (at 85.09 160.02 0)
       (effects (font (size 1.27 1.27)) hide)
     )
@@
   (symbol (lib_id "Device:R") (at 109.22 160.02 0)
     (in_bom yes) (on_board yes)
-    (property "Reference" "R485" (id 0) (at 110.998 158.8516 0)
+    (property "Reference" "R483" (id 0) (at 110.998 158.8516 0)
       (effects (font (size 1.27 1.27)) (justify left))
     )
@@
   (symbol (lib_id "Transistor_FET:2N7002") (at 46.99 123.19 0)
     (in_bom yes) (on_board yes)
-    (property "Reference" "Q1089" (id 0) (at 52.2224 122.0216 0)
+    (property "Reference" "Q1087" (id 0) (at 52.2224 122.0216 0)
       (effects (font (size 1.27 1.27)) (justify left))
     )
@@
   (symbol (lib_id "Transistor_FET:2N7002") (at 46.99 138.43 0)
     (in_bom yes) (on_board yes)
-    (property "Reference" "Q1093" (id 0) (at 52.2224 137.2616 0)
+    (property "Reference" "Q1091" (id 0) (at 52.2224 137.2616 0)
       (effects (font (size 1.27 1.27)) (justify left))
     )
@@
   (symbol (lib_id "Transistor_FET:2N7002") (at 71.12 123.19 0)
     (in_bom yes) (on_board yes)
-    (property "Reference" "Q1090" (id 0) (at 76.3524 122.0216 0)
+    (property "Reference" "Q1088" (id 0) (at 76.3524 122.0216 0)
       (effects (font (size 1.27 1.27)) (justify left))
     )
@@
   (symbol (lib_id "Transistor_FET:2N7002") (at 71.12 138.43 0)
     (in_bom yes) (on_board yes)
-    (property "Reference" "Q1094" (id 0) (at 76.3524 137.2616 0)
+    (property "Reference" "Q1092" (id 0) (at 76.3524 137.2616 0)
       (effects (font (size 1.27 1.27)) (justify left))
     )
@@
   (symbol (lib_id "Transistor_FET:2N7002") (at 97.79 123.19 0)
     (in_bom yes) (on_board yes)
-    (property "Reference" "Q1091" (id 0) (at 103.0224 122.0216 0)
+    (property "Reference" "Q1089" (id 0) (at 103.0224 122.0216 0)
       (effects (font (size 1.27 1.27)) (justify left))
     )
@@
   (symbol (lib_id "Transistor_FET:2N7002") (at 97.79 138.43 0)
     (in_bom yes) (on_board yes)
-    (property "Reference" "Q1095" (id 0) (at 103.0224 137.2616 0)
+    (property "Reference" "Q1093" (id 0) (at 103.0224 137.2616 0)
       (effects (font (size 1.27 1.27)) (justify left))
     )
@@
   (symbol (lib_id "Transistor_FET:2N7002") (at 106.68 172.72 0)
     (in_bom yes) (on_board yes)
-    (property "Reference" "Q1097" (id 0) (at 111.9124 171.5516 0)
+    (property "Reference" "Q1095" (id 0) (at 111.9124 171.5516 0)
       (effects (font (size 1.27 1.27)) (justify left))
     )
@@
   (symbol (lib_id "Transistor_FET:2N7002") (at 123.19 123.19 0)
     (in_bom yes) (on_board yes)
-    (property "Reference" "Q1092" (id 0) (at 128.4224 122.0216 0)
+    (property "Reference" "Q1090" (id 0) (at 128.4224 122.0216 0)
       (effects (font (size 1.27 1.27)) (justify left))
     )
@@
   (symbol (lib_id "Transistor_FET:2N7002") (at 123.19 138.43 0)
     (in_bom yes) (on_board yes)
-    (property "Reference" "Q1096" (id 0) (at 128.4224 137.2616 0)
+    (property "Reference" "Q1094" (id 0) (at 128.4224 137.2616 0)
       (effects (font (size 1.27 1.27)) (justify left))
     )
@@
   (symbol (lib_id "Transistor_FET:2N7002") (at 147.32 78.74 0)
     (in_bom yes) (on_board yes)
-    (property "Reference" "Q1087" (id 0) (at 152.5524 77.5716 0)
+    (property "Reference" "Q1085" (id 0) (at 152.5524 77.5716 0)
       (effects (font (size 1.27 1.27)) (justify left))
     )
@@
   (symbol (lib_id "Transistor_FET:2N7002") (at 147.32 88.9 0)
     (in_bom yes) (on_board yes)
-    (property "Reference" "Q1088" (id 0) (at 152.5524 87.7316 0)
-      (effects (font (size 1.27 1.27)) (justify left))
-    )
+    (property "Reference" "Q1086" (id 0) (at 152.5524 87.7316 0)
+      (effects (font (size 1.27 1.27)) (justify left))
+    )
