File: pcb/xhreg.kicad_sch (KiCad schematic)
At the start: 12 parts, among them Q741 2N7002a, Q742 2N7002a, Q743 2N7002a, Q744 2N7002a, Q745 2N7002a, Q746 2N7002a, Q747 2N7002a, Q748 2N7002a, Q749 2N7002a, Q750 2N7002a

Commit message: New reset.
Parts:
- renumbered R317 to R316, R318 to R317
Changed lines of the file:
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@@
   (symbol (lib_id "power:VCC") (at 67.31 104.14 0)
     (in_bom yes) (on_board yes)
-    (property "Reference" "#PWR0639" (id 0) (at 67.31 107.95 0)
+    (property "Reference" "#PWR0637" (id 0) (at 67.31 107.95 0)
       (effects (font (size 1.27 1.27)) hide)
     )
@@
   (symbol (lib_id "power:VCC") (at 135.89 46.99 0)
     (in_bom yes) (on_board yes)
-    (property "Reference" "#PWR0631" (id 0) (at 135.89 50.8 0)
+    (property "Reference" "#PWR0629" (id 0) (at 135.89 50.8 0)
       (effects (font (size 1.27 1.27)) hide)
     )
@@
   (symbol (lib_id "power:GND") (at 67.31 87.63 0)
     (in_bom yes) (on_board yes)
-    (property "Reference" "#PWR0634" (id 0) (at 67.31 93.98 0)
+    (property "Reference" "#PWR0632" (id 0) (at 67.31 93.98 0)
       (effects (font (size 1.27 1.27)) hide)
     )
@@
   (symbol (lib_id "power:GND") (at 67.31 130.81 0)
     (in_bom yes) (on_board yes)
-    (property "Reference" "#PWR0640" (id 0) (at 67.31 137.16 0)
+    (property "Reference" "#PWR0638" (id 0) (at 67.31 137.16 0)
       (effects (font (size 1.27 1.27)) hide)
     )
@@
   (symbol (lib_id "power:GND") (at 93.98 95.25 0)
     (in_bom yes) (on_board yes)
-    (property "Reference" "#PWR0635" (id 0) (at 93.98 101.6 0)
+    (property "Reference" "#PWR0633" (id 0) (at 93.98 101.6 0)
       (effects (font (size 1.27 1.27)) hide)
     )
@@
   (symbol (lib_id "power:GND") (at 119.38 96.52 0)
     (in_bom yes) (on_board yes)
-    (property "Reference" "#PWR0637" (id 0) (at 119.38 102.87 0)
+    (property "Reference" "#PWR0635" (id 0) (at 119.38 102.87 0)
       (effects (font (size 1.27 1.27)) hide)
     )
@@
   (symbol (lib_id "power:GND") (at 148.59 96.52 0)
     (in_bom yes) (on_board yes)
-    (property "Reference" "#PWR0638" (id 0) (at 148.59 102.87 0)
+    (property "Reference" "#PWR0636" (id 0) (at 148.59 102.87 0)
       (effects (font (size 1.27 1.27)) hide)
     )
@@
   (symbol (lib_id "power:GND") (at 205.74 63.5 90)
     (in_bom yes) (on_board yes)
-    (property "Reference" "#PWR0632" (id 0) (at 212.09 63.5 0)
+    (property "Reference" "#PWR0630" (id 0) (at 212.09 63.5 0)
       (effects (font (size 1.27 1.27)) hide)
     )
@@
   (symbol (lib_id "power:GND") (at 205.74 68.58 90)
     (in_bom yes) (on_board yes)
-    (property "Reference" "#PWR0633" (id 0) (at 212.09 68.58 0)
+    (property "Reference" "#PWR0631" (id 0) (at 212.09 68.58 0)
       (effects (font (size 1.27 1.27)) hide)
     )
@@
   (symbol (lib_id "power:GND") (at 240.03 95.25 0)
     (in_bom yes) (on_board yes)
-    (property "Reference" "#PWR0636" (id 0) (at 240.03 101.6 0)
+    (property "Reference" "#PWR0634" (id 0) (at 240.03 101.6 0)
       (effects (font (size 1.27 1.27)) hide)
     )
@@
   (symbol (lib_id "Device:R") (at 67.31 107.95 0)
     (in_bom yes) (on_board yes)
-    (property "Reference" "R318" (id 0) (at 69.088 106.7816 0)
+    (property "Reference" "R317" (id 0) (at 69.088 106.7816 0)
       (effects (font (size 1.27 1.27)) (justify left))
     )
@@
   (symbol (lib_id "Device:R") (at 135.89 50.8 0)
     (in_bom yes) (on_board yes)
-    (property "Reference" "R317" (id 0) (at 137.668 49.6316 0)
+    (property "Reference" "R316" (id 0) (at 137.668 49.6316 0)
       (effects (font (size 1.27 1.27)) (justify left))
     )

Commit message: Some fixes.
Parts:
- renumbered Q741 to Q738, Q742 to Q739, Q743 to Q740, Q744 to Q741, Q745 to Q742, Q746 to Q743, Q747 to Q744, Q748 to Q745, Q749 to Q746, Q750 to Q747, R316 to R320, R317 to R321
Changed lines of the file:
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@@
   (symbol (lib_id "power:VCC") (at 67.31 104.14 0)
     (in_bom yes) (on_board yes)
-    (property "Reference" "#PWR0637" (id 0) (at 67.31 107.95 0)
+    (property "Reference" "#PWR0649" (id 0) (at 67.31 107.95 0)
       (effects (font (size 1.27 1.27)) hide)
     )
@@
   (symbol (lib_id "power:VCC") (at 135.89 46.99 0)
     (in_bom yes) (on_board yes)
-    (property "Reference" "#PWR0629" (id 0) (at 135.89 50.8 0)
+    (property "Reference" "#PWR0641" (id 0) (at 135.89 50.8 0)
       (effects (font (size 1.27 1.27)) hide)
     )
@@
   (symbol (lib_id "power:GND") (at 67.31 87.63 0)
     (in_bom yes) (on_board yes)
-    (property "Reference" "#PWR0632" (id 0) (at 67.31 93.98 0)
+    (property "Reference" "#PWR0644" (id 0) (at 67.31 93.98 0)
       (effects (font (size 1.27 1.27)) hide)
     )
@@
   (symbol (lib_id "power:GND") (at 67.31 130.81 0)
     (in_bom yes) (on_board yes)
-    (property "Reference" "#PWR0638" (id 0) (at 67.31 137.16 0)
+    (property "Reference" "#PWR0650" (id 0) (at 67.31 137.16 0)
       (effects (font (size 1.27 1.27)) hide)
     )
@@
   (symbol (lib_id "power:GND") (at 93.98 95.25 0)
     (in_bom yes) (on_board yes)
-    (property "Reference" "#PWR0633" (id 0) (at 93.98 101.6 0)
+    (property "Reference" "#PWR0645" (id 0) (at 93.98 101.6 0)
       (effects (font (size 1.27 1.27)) hide)
     )
@@
   (symbol (lib_id "power:GND") (at 119.38 96.52 0)
     (in_bom yes) (on_board yes)
-    (property "Reference" "#PWR0635" (id 0) (at 119.38 102.87 0)
+    (property "Reference" "#PWR0647" (id 0) (at 119.38 102.87 0)
       (effects (font (size 1.27 1.27)) hide)
     )
@@
   (symbol (lib_id "power:GND") (at 148.59 96.52 0)
     (in_bom yes) (on_board yes)
-    (property "Reference" "#PWR0636" (id 0) (at 148.59 102.87 0)
+    (property "Reference" "#PWR0648" (id 0) (at 148.59 102.87 0)
       (effects (font (size 1.27 1.27)) hide)
     )
@@
   (symbol (lib_id "power:GND") (at 205.74 63.5 90)
     (in_bom yes) (on_board yes)
-    (property "Reference" "#PWR0630" (id 0) (at 212.09 63.5 0)
+    (property "Reference" "#PWR0642" (id 0) (at 212.09 63.5 0)
       (effects (font (size 1.27 1.27)) hide)
     )
@@
   (symbol (lib_id "power:GND") (at 205.74 68.58 90)
     (in_bom yes) (on_board yes)
-    (property "Reference" "#PWR0631" (id 0) (at 212.09 68.58 0)
+    (property "Reference" "#PWR0643" (id 0) (at 212.09 68.58 0)
       (effects (font (size 1.27 1.27)) hide)
     )
@@
   (symbol (lib_id "power:GND") (at 240.03 95.25 0)
     (in_bom yes) (on_board yes)
-    (property "Reference" "#PWR0634" (id 0) (at 240.03 101.6 0)
+    (property "Reference" "#PWR0646" (id 0) (at 240.03 101.6 0)
       (effects (font (size 1.27 1.27)) hide)
     )
@@
   (symbol (lib_id "Device:R") (at 67.31 107.95 0)
     (in_bom yes) (on_board yes)
-    (property "Reference" "R317" (id 0) (at 69.088 106.7816 0)
+    (property "Reference" "R321" (id 0) (at 69.088 106.7816 0)
       (effects (font (size 1.27 1.27)) (justify left))
     )
@@
   (symbol (lib_id "Device:R") (at 135.89 50.8 0)
     (in_bom yes) (on_board yes)
-    (property "Reference" "R316" (id 0) (at 137.668 49.6316 0)
+    (property "Reference" "R320" (id 0) (at 137.668 49.6316 0)
       (effects (font (size 1.27 1.27)) (justify left))
     )
@@
   (symbol (lib_id "Transistor_FET:2N7002") (at 64.77 82.55 0)
     (in_bom yes) (on_board yes)
-    (property "Reference" "Q745" (id 0) (at 70.0024 81.3816 0)
+    (property "Reference" "Q742" (id 0) (at 70.0024 81.3816 0)
       (effects (font (size 1.27 1.27)) (justify left))
     )
@@
   (symbol (lib_id "Transistor_FET:2N7002") (at 64.77 125.73 0)
     (in_bom yes) (on_board yes)
-    (property "Reference" "Q750" (id 0) (at 70.0024 124.5616 0)
+    (property "Reference" "Q747" (id 0) (at 70.0024 124.5616 0)
       (effects (font (size 1.27 1.27)) (justify left))
     )
@@
   (symbol (lib_id "Transistor_FET:2N7002") (at 91.44 80.01 0)
     (in_bom yes) (on_board yes)
-    (property "Reference" "Q741" (id 0) (at 96.6724 78.8416 0)
+    (property "Reference" "Q738" (id 0) (at 96.6724 78.8416 0)
       (effects (font (size 1.27 1.27)) (justify left))
     )
@@
   (symbol (lib_id "Transistor_FET:2N7002") (at 91.44 90.17 0)
     (in_bom yes) (on_board yes)
-    (property "Reference" "Q746" (id 0) (at 96.6724 89.0016 0)
+    (property "Reference" "Q743" (id 0) (at 96.6724 89.0016 0)
       (effects (font (size 1.27 1.27)) (justify left))
     )
@@
   (symbol (lib_id "Transistor_FET:2N7002") (at 116.84 81.28 0)
     (in_bom yes) (on_board yes)
-    (property "Reference" "Q743" (id 0) (at 122.0724 80.1116 0)
+    (property "Reference" "Q740" (id 0) (at 122.0724 80.1116 0)
       (effects (font (size 1.27 1.27)) (justify left))
     )
@@
   (symbol (lib_id "Transistor_FET:2N7002") (at 116.84 91.44 0)
     (in_bom yes) (on_board yes)
-    (property "Reference" "Q748" (id 0) (at 122.0724 90.2716 0)
+    (property "Reference" "Q745" (id 0) (at 122.0724 90.2716 0)
       (effects (font (size 1.27 1.27)) (justify left))
     )
@@
   (symbol (lib_id "Transistor_FET:2N7002") (at 146.05 81.28 0)
     (in_bom yes) (on_board yes)
-    (property "Reference" "Q744" (id 0) (at 151.2824 80.1116 0)
+    (property "Reference" "Q741" (id 0) (at 151.2824 80.1116 0)
       (effects (font (size 1.27 1.27)) (justify left))
     )
@@
   (symbol (lib_id "Transistor_FET:2N7002") (at 146.05 91.44 0)
     (in_bom yes) (on_board yes)
-    (property "Reference" "Q749" (id 0) (at 151.2824 90.2716 0)
+    (property "Reference" "Q746" (id 0) (at 151.2824 90.2716 0)
       (effects (font (size 1.27 1.27)) (justify left))
     )
@@
   (symbol (lib_id "Transistor_FET:2N7002") (at 237.49 80.01 0)
     (in_bom yes) (on_board yes)
-    (property "Reference" "Q742" (id 0) (at 242.7224 78.8416 0)
+    (property "Reference" "Q739" (id 0) (at 242.7224 78.8416 0)
       (effects (font (size 1.27 1.27)) (justify left))
     )
@@
   (symbol (lib_id "Transistor_FET:2N7002") (at 237.49 90.17 0)
     (in_bom yes) (on_board yes)
-    (property "Reference" "Q747" (id 0) (at 242.7224 89.0016 0)
-      (effects (font (size 1.27 1.27)) (justify left))
-    )
+    (property "Reference" "Q744" (id 0) (at 242.7224 89.0016 0)
+      (effects (font (size 1.27 1.27)) (justify left))
+    )

Commit message: Faster.
Parts:
- renumbered Q738 to Q736, Q739 to Q737, Q740 to Q738, Q741 to Q739, Q742 to Q740, Q743 to Q741, Q744 to Q742, Q745 to Q743, Q746 to Q744, Q747 to Q745, R320 to R318, R321 to R319
Changed lines of the file:
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@@
   (symbol (lib_id "power:VCC") (at 67.31 104.14 0)
     (in_bom yes) (on_board yes)
-    (property "Reference" "#PWR0649" (id 0) (at 67.31 107.95 0)
+    (property "Reference" "#PWR0646" (id 0) (at 67.31 107.95 0)
       (effects (font (size 1.27 1.27)) hide)
     )
@@
   (symbol (lib_id "power:VCC") (at 135.89 46.99 0)
     (in_bom yes) (on_board yes)
-    (property "Reference" "#PWR0641" (id 0) (at 135.89 50.8 0)
+    (property "Reference" "#PWR0638" (id 0) (at 135.89 50.8 0)
       (effects (font (size 1.27 1.27)) hide)
     )
@@
   (symbol (lib_id "power:GND") (at 67.31 87.63 0)
     (in_bom yes) (on_board yes)
-    (property "Reference" "#PWR0644" (id 0) (at 67.31 93.98 0)
+    (property "Reference" "#PWR0641" (id 0) (at 67.31 93.98 0)
       (effects (font (size 1.27 1.27)) hide)
     )
@@
   (symbol (lib_id "power:GND") (at 67.31 130.81 0)
     (in_bom yes) (on_board yes)
-    (property "Reference" "#PWR0650" (id 0) (at 67.31 137.16 0)
+    (property "Reference" "#PWR0647" (id 0) (at 67.31 137.16 0)
       (effects (font (size 1.27 1.27)) hide)
     )
@@
   (symbol (lib_id "power:GND") (at 93.98 95.25 0)
     (in_bom yes) (on_board yes)
-    (property "Reference" "#PWR0645" (id 0) (at 93.98 101.6 0)
+    (property "Reference" "#PWR0642" (id 0) (at 93.98 101.6 0)
       (effects (font (size 1.27 1.27)) hide)
     )
@@
   (symbol (lib_id "power:GND") (at 119.38 96.52 0)
     (in_bom yes) (on_board yes)
-    (property "Reference" "#PWR0647" (id 0) (at 119.38 102.87 0)
+    (property "Reference" "#PWR0644" (id 0) (at 119.38 102.87 0)
       (effects (font (size 1.27 1.27)) hide)
     )
@@
   (symbol (lib_id "power:GND") (at 148.59 96.52 0)
     (in_bom yes) (on_board yes)
-    (property "Reference" "#PWR0648" (id 0) (at 148.59 102.87 0)
+    (property "Reference" "#PWR0645" (id 0) (at 148.59 102.87 0)
       (effects (font (size 1.27 1.27)) hide)
     )
@@
   (symbol (lib_id "power:GND") (at 205.74 63.5 90)
     (in_bom yes) (on_board yes)
-    (property "Reference" "#PWR0642" (id 0) (at 212.09 63.5 0)
+    (property "Reference" "#PWR0639" (id 0) (at 212.09 63.5 0)
       (effects (font (size 1.27 1.27)) hide)
     )
@@
   (symbol (lib_id "power:GND") (at 205.74 68.58 90)
     (in_bom yes) (on_board yes)
-    (property "Reference" "#PWR0643" (id 0) (at 212.09 68.58 0)
+    (property "Reference" "#PWR0640" (id 0) (at 212.09 68.58 0)
       (effects (font (size 1.27 1.27)) hide)
     )
@@
   (symbol (lib_id "power:GND") (at 240.03 95.25 0)
     (in_bom yes) (on_board yes)
-    (property "Reference" "#PWR0646" (id 0) (at 240.03 101.6 0)
+    (property "Reference" "#PWR0643" (id 0) (at 240.03 101.6 0)
       (effects (font (size 1.27 1.27)) hide)
     )
@@
   (symbol (lib_id "Device:R") (at 67.31 107.95 0)
     (in_bom yes) (on_board yes)
-    (property "Reference" "R321" (id 0) (at 69.088 106.7816 0)
+    (property "Reference" "R319" (id 0) (at 69.088 106.7816 0)
       (effects (font (size 1.27 1.27)) (justify left))
     )
@@
   (symbol (lib_id "Device:R") (at 135.89 50.8 0)
     (in_bom yes) (on_board yes)
-    (property "Reference" "R320" (id 0) (at 137.668 49.6316 0)
+    (property "Reference" "R318" (id 0) (at 137.668 49.6316 0)
       (effects (font (size 1.27 1.27)) (justify left))
     )
@@
   (symbol (lib_id "Transistor_FET:2N7002") (at 64.77 82.55 0)
     (in_bom yes) (on_board yes)
-    (property "Reference" "Q742" (id 0) (at 70.0024 81.3816 0)
+    (property "Reference" "Q740" (id 0) (at 70.0024 81.3816 0)
       (effects (font (size 1.27 1.27)) (justify left))
     )
@@
   (symbol (lib_id "Transistor_FET:2N7002") (at 64.77 125.73 0)
     (in_bom yes) (on_board yes)
-    (property "Reference" "Q747" (id 0) (at 70.0024 124.5616 0)
+    (property "Reference" "Q745" (id 0) (at 70.0024 124.5616 0)
       (effects (font (size 1.27 1.27)) (justify left))
     )
@@
   (symbol (lib_id "Transistor_FET:2N7002") (at 91.44 80.01 0)
     (in_bom yes) (on_board yes)
-    (property "Reference" "Q738" (id 0) (at 96.6724 78.8416 0)
+    (property "Reference" "Q736" (id 0) (at 96.6724 78.8416 0)
       (effects (font (size 1.27 1.27)) (justify left))
     )
@@
   (symbol (lib_id "Transistor_FET:2N7002") (at 91.44 90.17 0)
     (in_bom yes) (on_board yes)
-    (property "Reference" "Q743" (id 0) (at 96.6724 89.0016 0)
+    (property "Reference" "Q741" (id 0) (at 96.6724 89.0016 0)
       (effects (font (size 1.27 1.27)) (justify left))
     )
@@
   (symbol (lib_id "Transistor_FET:2N7002") (at 116.84 81.28 0)
     (in_bom yes) (on_board yes)
-    (property "Reference" "Q740" (id 0) (at 122.0724 80.1116 0)
+    (property "Reference" "Q738" (id 0) (at 122.0724 80.1116 0)
       (effects (font (size 1.27 1.27)) (justify left))
     )
@@
   (symbol (lib_id "Transistor_FET:2N7002") (at 116.84 91.44 0)
     (in_bom yes) (on_board yes)
-    (property "Reference" "Q745" (id 0) (at 122.0724 90.2716 0)
+    (property "Reference" "Q743" (id 0) (at 122.0724 90.2716 0)
       (effects (font (size 1.27 1.27)) (justify left))
     )
@@
   (symbol (lib_id "Transistor_FET:2N7002") (at 146.05 81.28 0)
     (in_bom yes) (on_board yes)
-    (property "Reference" "Q741" (id 0) (at 151.2824 80.1116 0)
+    (property "Reference" "Q739" (id 0) (at 151.2824 80.1116 0)
       (effects (font (size 1.27 1.27)) (justify left))
     )
@@
   (symbol (lib_id "Transistor_FET:2N7002") (at 146.05 91.44 0)
     (in_bom yes) (on_board yes)
-    (property "Reference" "Q746" (id 0) (at 151.2824 90.2716 0)
+    (property "Reference" "Q744" (id 0) (at 151.2824 90.2716 0)
       (effects (font (size 1.27 1.27)) (justify left))
     )
@@
   (symbol (lib_id "Transistor_FET:2N7002") (at 237.49 80.01 0)
     (in_bom yes) (on_board yes)
-    (property "Reference" "Q739" (id 0) (at 242.7224 78.8416 0)
+    (property "Reference" "Q737" (id 0) (at 242.7224 78.8416 0)
       (effects (font (size 1.27 1.27)) (justify left))
     )
@@
   (symbol (lib_id "Transistor_FET:2N7002") (at 237.49 90.17 0)
     (in_bom yes) (on_board yes)
-    (property "Reference" "Q744" (id 0) (at 242.7224 89.0016 0)
-      (effects (font (size 1.27 1.27)) (justify left))
-    )
+    (property "Reference" "Q742" (id 0) (at 242.7224 89.0016 0)
+      (effects (font (size 1.27 1.27)) (justify left))
+    )
