File: pcb/xhreg.kicad_sch (KiCad schematic)
At the start: 12 parts, among them Q736 2N7002a, Q737 2N7002a, Q738 2N7002a, Q739 2N7002a, Q740 2N7002a, Q741 2N7002a, Q742 2N7002a, Q743 2N7002a, Q744 2N7002a, Q745 2N7002a

Commit message: Updates
Parts:
- Q736, Q737, Q738, Q739, Q740, Q741, Q742, Q743, Q744, Q745: value 2N7002a -> 2N7002; LCSC C8545 -> C181083
Changed lines of the file:
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@@
       (effects (font (size 1.27 1.27)) (justify left))
     )
-    (property "Value" "2N7002a" (id 1) (at 70.0024 83.693 0)
+    (property "Value" "2N7002" (id 1) (at 70.0024 83.693 0)
       (effects (font (size 1.27 1.27)) (justify left))
     )
@@
       (effects (font (size 1.27 1.27) italic) (justify left) hide)
     )
-    (property "Datasheet" "https://www.fairchildsemi.com/datasheets/2N/2N7002.pdf" (id 3) (at 64.77 82.55 0)
-      (effects (font (size 1.27 1.27)) (justify left) hide)
-    )
-    (property "LCSC" "C8545" (id 4) (at 64.77 82.55 0)
+    (property "Datasheet" "https://datasheet.lcsc.com/szlcsc/Guangdong-Hottech-2N7002K_C181083.pdf" (id 3) (at 64.77 82.55 0)
+      (effects (font (size 1.27 1.27)) (justify left) hide)
+    )
+    (property "LCSC" "C181083" (id 4) (at 64.77 82.55 0)
       (effects (font (size 1.27 1.27)) hide)
     )
@@
       (effects (font (size 1.27 1.27)) (justify left))
     )
-    (property "Value" "2N7002a" (id 1) (at 70.0024 126.873 0)
+    (property "Value" "2N7002" (id 1) (at 70.0024 126.873 0)
       (effects (font (size 1.27 1.27)) (justify left))
     )
@@
       (effects (font (size 1.27 1.27) italic) (justify left) hide)
     )
-    (property "Datasheet" "https://www.fairchildsemi.com/datasheets/2N/2N7002.pdf" (id 3) (at 64.77 125.73 0)
-      (effects (font (size 1.27 1.27)) (justify left) hide)
-    )
-    (property "LCSC" "C8545" (id 4) (at 64.77 125.73 0)
+    (property "Datasheet" "https://datasheet.lcsc.com/szlcsc/Guangdong-Hottech-2N7002K_C181083.pdf" (id 3) (at 64.77 125.73 0)
+      (effects (font (size 1.27 1.27)) (justify left) hide)
+    )
+    (property "LCSC" "C181083" (id 4) (at 64.77 125.73 0)
       (effects (font (size 1.27 1.27)) hide)
     )
@@
       (effects (font (size 1.27 1.27)) (justify left))
     )
-    (property "Value" "2N7002a" (id 1) (at 96.6724 81.153 0)
+    (property "Value" "2N7002" (id 1) (at 96.6724 81.153 0)
       (effects (font (size 1.27 1.27)) (justify left))
     )
@@
       (effects (font (size 1.27 1.27) italic) (justify left) hide)
     )
-    (property "Datasheet" "https://www.fairchildsemi.com/datasheets/2N/2N7002.pdf" (id 3) (at 91.44 80.01 0)
-      (effects (font (size 1.27 1.27)) (justify left) hide)
-    )
-    (property "LCSC" "C8545" (id 4) (at 91.44 80.01 0)
+    (property "Datasheet" "https://datasheet.lcsc.com/szlcsc/Guangdong-Hottech-2N7002K_C181083.pdf" (id 3) (at 91.44 80.01 0)
+      (effects (font (size 1.27 1.27)) (justify left) hide)
+    )
+    (property "LCSC" "C181083" (id 4) (at 91.44 80.01 0)
       (effects (font (size 1.27 1.27)) hide)
     )
@@
       (effects (font (size 1.27 1.27)) (justify left))
     )
-    (property "Value" "2N7002a" (id 1) (at 96.6724 91.313 0)
+    (property "Value" "2N7002" (id 1) (at 96.6724 91.313 0)
       (effects (font (size 1.27 1.27)) (justify left))
     )
@@
       (effects (font (size 1.27 1.27) italic) (justify left) hide)
     )
-    (property "Datasheet" "https://www.fairchildsemi.com/datasheets/2N/2N7002.pdf" (id 3) (at 91.44 90.17 0)
-      (effects (font (size 1.27 1.27)) (justify left) hide)
-    )
-    (property "LCSC" "C8545" (id 4) (at 91.44 90.17 0)
+    (property "Datasheet" "https://datasheet.lcsc.com/szlcsc/Guangdong-Hottech-2N7002K_C181083.pdf" (id 3) (at 91.44 90.17 0)
+      (effects (font (size 1.27 1.27)) (justify left) hide)
+    )
+    (property "LCSC" "C181083" (id 4) (at 91.44 90.17 0)
       (effects (font (size 1.27 1.27)) hide)
     )
@@
       (effects (font (size 1.27 1.27)) (justify left))
     )
-    (property "Value" "2N7002a" (id 1) (at 122.0724 82.423 0)
+    (property "Value" "2N7002" (id 1) (at 122.0724 82.423 0)
       (effects (font (size 1.27 1.27)) (justify left))
     )
@@
       (effects (font (size 1.27 1.27) italic) (justify left) hide)
     )
-    (property "Datasheet" "https://www.fairchildsemi.com/datasheets/2N/2N7002.pdf" (id 3) (at 116.84 81.28 0)
-      (effects (font (size 1.27 1.27)) (justify left) hide)
-    )
-    (property "LCSC" "C8545" (id 4) (at 116.84 81.28 0)
+    (property "Datasheet" "https://datasheet.lcsc.com/szlcsc/Guangdong-Hottech-2N7002K_C181083.pdf" (id 3) (at 116.84 81.28 0)
+      (effects (font (size 1.27 1.27)) (justify left) hide)
+    )
+    (property "LCSC" "C181083" (id 4) (at 116.84 81.28 0)
       (effects (font (size 1.27 1.27)) hide)
     )
@@
       (effects (font (size 1.27 1.27)) (justify left))
     )
-    (property "Value" "2N7002a" (id 1) (at 122.0724 92.583 0)
+    (property "Value" "2N7002" (id 1) (at 122.0724 92.583 0)
       (effects (font (size 1.27 1.27)) (justify left))
     )
@@
       (effects (font (size 1.27 1.27) italic) (justify left) hide)
     )
-    (property "Datasheet" "https://www.fairchildsemi.com/datasheets/2N/2N7002.pdf" (id 3) (at 116.84 91.44 0)
-      (effects (font (size 1.27 1.27)) (justify left) hide)
-    )
-    (property "LCSC" "C8545" (id 4) (at 116.84 91.44 0)
+    (property "Datasheet" "https://datasheet.lcsc.com/szlcsc/Guangdong-Hottech-2N7002K_C181083.pdf" (id 3) (at 116.84 91.44 0)
+      (effects (font (size 1.27 1.27)) (justify left) hide)
+    )
+    (property "LCSC" "C181083" (id 4) (at 116.84 91.44 0)
       (effects (font (size 1.27 1.27)) hide)
     )
@@
       (effects (font (size 1.27 1.27)) (justify left))
     )
-    (property "Value" "2N7002a" (id 1) (at 151.2824 82.423 0)
+    (property "Value" "2N7002" (id 1) (at 151.2824 82.423 0)
       (effects (font (size 1.27 1.27)) (justify left))
     )
@@
       (effects (font (size 1.27 1.27) italic) (justify left) hide)
     )
-    (property "Datasheet" "https://www.fairchildsemi.com/datasheets/2N/2N7002.pdf" (id 3) (at 146.05 81.28 0)
-      (effects (font (size 1.27 1.27)) (justify left) hide)
-    )
-    (property "LCSC" "C8545" (id 4) (at 146.05 81.28 0)
+    (property "Datasheet" "https://datasheet.lcsc.com/szlcsc/Guangdong-Hottech-2N7002K_C181083.pdf" (id 3) (at 146.05 81.28 0)
+      (effects (font (size 1.27 1.27)) (justify left) hide)
+    )
+    (property "LCSC" "C181083" (id 4) (at 146.05 81.28 0)
       (effects (font (size 1.27 1.27)) hide)
     )
@@
       (effects (font (size 1.27 1.27)) (justify left))
     )
-    (property "Value" "2N7002a" (id 1) (at 151.2824 92.583 0)
+    (property "Value" "2N7002" (id 1) (at 151.2824 92.583 0)
       (effects (font (size 1.27 1.27)) (justify left))
     )
@@
       (effects (font (size 1.27 1.27) italic) (justify left) hide)
     )
-    (property "Datasheet" "https://www.fairchildsemi.com/datasheets/2N/2N7002.pdf" (id 3) (at 146.05 91.44 0)
-      (effects (font (size 1.27 1.27)) (justify left) hide)
-    )
-    (property "LCSC" "C8545" (id 4) (at 146.05 91.44 0)
+    (property "Datasheet" "https://datasheet.lcsc.com/szlcsc/Guangdong-Hottech-2N7002K_C181083.pdf" (id 3) (at 146.05 91.44 0)
+      (effects (font (size 1.27 1.27)) (justify left) hide)
+    )
+    (property "LCSC" "C181083" (id 4) (at 146.05 91.44 0)
       (effects (font (size 1.27 1.27)) hide)
     )
@@
       (effects (font (size 1.27 1.27)) (justify left))
     )
-    (property "Value" "2N7002a" (id 1) (at 242.7224 81.153 0)
+    (property "Value" "2N7002" (id 1) (at 242.7224 81.153 0)
       (effects (font (size 1.27 1.27)) (justify left))
     )
@@
       (effects (font (size 1.27 1.27) italic) (justify left) hide)
     )
-    (property "Datasheet" "https://www.fairchildsemi.com/datasheets/2N/2N7002.pdf" (id 3) (at 237.49 80.01 0)
-      (effects (font (size 1.27 1.27)) (justify left) hide)
-    )
-    (property "LCSC" "C8545" (id 4) (at 237.49 80.01 0)
+    (property "Datasheet" "https://datasheet.lcsc.com/szlcsc/Guangdong-Hottech-2N7002K_C181083.pdf" (id 3) (at 237.49 80.01 0)
+      (effects (font (size 1.27 1.27)) (justify left) hide)
+    )
+    (property "LCSC" "C181083" (id 4) (at 237.49 80.01 0)
       (effects (font (size 1.27 1.27)) hide)
     )
@@
       (effects (font (size 1.27 1.27)) (justify left))
     )
-    (property "Value" "2N7002a" (id 1) (at 242.7224 91.313 0)
+    (property "Value" "2N7002" (id 1) (at 242.7224 91.313 0)
       (effects (font (size 1.27 1.27)) (justify left))
     )
@@
       (effects (font (size 1.27 1.27) italic) (justify left) hide)
     )
-    (property "Datasheet" "https://www.fairchildsemi.com/datasheets/2N/2N7002.pdf" (id 3) (at 237.49 90.17 0)
-      (effects (font (size 1.27 1.27)) (justify left) hide)
-    )
-    (property "LCSC" "C8545" (id 4) (at 237.49 90.17 0)
-      (effects (font (size 1.27 1.27)) hide)
-    )
+    (property "Datasheet" "https://datasheet.lcsc.com/szlcsc/Guangdong-Hottech-2N7002K_C181083.pdf" (id 3) (at 237.49 90.17 0)
+      (effects (font (size 1.27 1.27)) (justify left) hide)
+    )
+    (property "LCSC" "C181083" (id 4) (at 237.49 90.17 0)
+      (effects (font (size 1.27 1.27)) hide)
+    )

Commit message: Update resistors.
Parts:
- renumbered Q736 to Q734, Q737 to Q735, Q738 to Q736, Q739 to Q737, Q740 to Q738, Q741 to Q739, Q742 to Q740, Q743 to Q741, Q744 to Q742, Q745 to Q743, R318 to R316, R319 to R317
Changed lines of the file:
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@@
   (symbol (lib_id "power:VCC") (at 67.31 104.14 0)
     (in_bom yes) (on_board yes)
-    (property "Reference" "#PWR0646" (id 0) (at 67.31 107.95 0)
+    (property "Reference" "#PWR0642" (id 0) (at 67.31 107.95 0)
       (effects (font (size 1.27 1.27)) hide)
     )
@@
   (symbol (lib_id "power:VCC") (at 135.89 46.99 0)
     (in_bom yes) (on_board yes)
-    (property "Reference" "#PWR0638" (id 0) (at 135.89 50.8 0)
+    (property "Reference" "#PWR0634" (id 0) (at 135.89 50.8 0)
       (effects (font (size 1.27 1.27)) hide)
     )
@@
   (symbol (lib_id "power:GND") (at 67.31 87.63 0)
     (in_bom yes) (on_board yes)
-    (property "Reference" "#PWR0641" (id 0) (at 67.31 93.98 0)
+    (property "Reference" "#PWR0637" (id 0) (at 67.31 93.98 0)
       (effects (font (size 1.27 1.27)) hide)
     )
@@
   (symbol (lib_id "power:GND") (at 67.31 130.81 0)
     (in_bom yes) (on_board yes)
-    (property "Reference" "#PWR0647" (id 0) (at 67.31 137.16 0)
+    (property "Reference" "#PWR0643" (id 0) (at 67.31 137.16 0)
       (effects (font (size 1.27 1.27)) hide)
     )
@@
   (symbol (lib_id "power:GND") (at 93.98 95.25 0)
     (in_bom yes) (on_board yes)
-    (property "Reference" "#PWR0642" (id 0) (at 93.98 101.6 0)
+    (property "Reference" "#PWR0638" (id 0) (at 93.98 101.6 0)
       (effects (font (size 1.27 1.27)) hide)
     )
@@
   (symbol (lib_id "power:GND") (at 119.38 96.52 0)
     (in_bom yes) (on_board yes)
-    (property "Reference" "#PWR0644" (id 0) (at 119.38 102.87 0)
+    (property "Reference" "#PWR0640" (id 0) (at 119.38 102.87 0)
       (effects (font (size 1.27 1.27)) hide)
     )
@@
   (symbol (lib_id "power:GND") (at 148.59 96.52 0)
     (in_bom yes) (on_board yes)
-    (property "Reference" "#PWR0645" (id 0) (at 148.59 102.87 0)
+    (property "Reference" "#PWR0641" (id 0) (at 148.59 102.87 0)
       (effects (font (size 1.27 1.27)) hide)
     )
@@
   (symbol (lib_id "power:GND") (at 205.74 63.5 90)
     (in_bom yes) (on_board yes)
-    (property "Reference" "#PWR0639" (id 0) (at 212.09 63.5 0)
+    (property "Reference" "#PWR0635" (id 0) (at 212.09 63.5 0)
       (effects (font (size 1.27 1.27)) hide)
     )
@@
   (symbol (lib_id "power:GND") (at 205.74 68.58 90)
     (in_bom yes) (on_board yes)
-    (property "Reference" "#PWR0640" (id 0) (at 212.09 68.58 0)
+    (property "Reference" "#PWR0636" (id 0) (at 212.09 68.58 0)
       (effects (font (size 1.27 1.27)) hide)
     )
@@
   (symbol (lib_id "power:GND") (at 240.03 95.25 0)
     (in_bom yes) (on_board yes)
-    (property "Reference" "#PWR0643" (id 0) (at 240.03 101.6 0)
+    (property "Reference" "#PWR0639" (id 0) (at 240.03 101.6 0)
       (effects (font (size 1.27 1.27)) hide)
     )
@@
   (symbol (lib_id "Device:R") (at 67.31 107.95 0)
     (in_bom yes) (on_board yes)
-    (property "Reference" "R319" (id 0) (at 69.088 106.7816 0)
+    (property "Reference" "R317" (id 0) (at 69.088 106.7816 0)
       (effects (font (size 1.27 1.27)) (justify left))
     )
@@
   (symbol (lib_id "Device:R") (at 135.89 50.8 0)
     (in_bom yes) (on_board yes)
-    (property "Reference" "R318" (id 0) (at 137.668 49.6316 0)
+    (property "Reference" "R316" (id 0) (at 137.668 49.6316 0)
       (effects (font (size 1.27 1.27)) (justify left))
     )
@@
   (symbol (lib_id "Transistor_FET:2N7002") (at 64.77 82.55 0)
     (in_bom yes) (on_board yes)
-    (property "Reference" "Q740" (id 0) (at 70.0024 81.3816 0)
+    (property "Reference" "Q738" (id 0) (at 70.0024 81.3816 0)
       (effects (font (size 1.27 1.27)) (justify left))
     )
@@
   (symbol (lib_id "Transistor_FET:2N7002") (at 64.77 125.73 0)
     (in_bom yes) (on_board yes)
-    (property "Reference" "Q745" (id 0) (at 70.0024 124.5616 0)
+    (property "Reference" "Q743" (id 0) (at 70.0024 124.5616 0)
       (effects (font (size 1.27 1.27)) (justify left))
     )
@@
   (symbol (lib_id "Transistor_FET:2N7002") (at 91.44 80.01 0)
     (in_bom yes) (on_board yes)
-    (property "Reference" "Q736" (id 0) (at 96.6724 78.8416 0)
+    (property "Reference" "Q734" (id 0) (at 96.6724 78.8416 0)
       (effects (font (size 1.27 1.27)) (justify left))
     )
@@
   (symbol (lib_id "Transistor_FET:2N7002") (at 91.44 90.17 0)
     (in_bom yes) (on_board yes)
-    (property "Reference" "Q741" (id 0) (at 96.6724 89.0016 0)
+    (property "Reference" "Q739" (id 0) (at 96.6724 89.0016 0)
       (effects (font (size 1.27 1.27)) (justify left))
     )
@@
   (symbol (lib_id "Transistor_FET:2N7002") (at 116.84 81.28 0)
     (in_bom yes) (on_board yes)
-    (property "Reference" "Q738" (id 0) (at 122.0724 80.1116 0)
+    (property "Reference" "Q736" (id 0) (at 122.0724 80.1116 0)
       (effects (font (size 1.27 1.27)) (justify left))
     )
@@
   (symbol (lib_id "Transistor_FET:2N7002") (at 116.84 91.44 0)
     (in_bom yes) (on_board yes)
-    (property "Reference" "Q743" (id 0) (at 122.0724 90.2716 0)
+    (property "Reference" "Q741" (id 0) (at 122.0724 90.2716 0)
       (effects (font (size 1.27 1.27)) (justify left))
     )
@@
   (symbol (lib_id "Transistor_FET:2N7002") (at 146.05 81.28 0)
     (in_bom yes) (on_board yes)
-    (property "Reference" "Q739" (id 0) (at 151.2824 80.1116 0)
+    (property "Reference" "Q737" (id 0) (at 151.2824 80.1116 0)
       (effects (font (size 1.27 1.27)) (justify left))
     )
@@
   (symbol (lib_id "Transistor_FET:2N7002") (at 146.05 91.44 0)
     (in_bom yes) (on_board yes)
-    (property "Reference" "Q744" (id 0) (at 151.2824 90.2716 0)
+    (property "Reference" "Q742" (id 0) (at 151.2824 90.2716 0)
       (effects (font (size 1.27 1.27)) (justify left))
     )
@@
   (symbol (lib_id "Transistor_FET:2N7002") (at 237.49 80.01 0)
     (in_bom yes) (on_board yes)
-    (property "Reference" "Q737" (id 0) (at 242.7224 78.8416 0)
+    (property "Reference" "Q735" (id 0) (at 242.7224 78.8416 0)
       (effects (font (size 1.27 1.27)) (justify left))
     )
@@
   (symbol (lib_id "Transistor_FET:2N7002") (at 237.49 90.17 0)
     (in_bom yes) (on_board yes)
-    (property "Reference" "Q742" (id 0) (at 242.7224 89.0016 0)
-      (effects (font (size 1.27 1.27)) (justify left))
-    )
+    (property "Reference" "Q740" (id 0) (at 242.7224 89.0016 0)
+      (effects (font (size 1.27 1.27)) (justify left))
+    )

Commit message: Updates
Parts:
- renumbered Q734 to Q731, Q735 to Q732, Q736 to Q733, Q737 to Q734, Q738 to Q735, Q739 to Q736, Q740 to Q737, Q741 to Q738, Q742 to Q739, Q743 to Q740
Changed lines of the file:
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@@
   (symbol (lib_id "power:VCC") (at 67.31 104.14 0)
     (in_bom yes) (on_board yes)
-    (property "Reference" "#PWR0642" (id 0) (at 67.31 107.95 0)
+    (property "Reference" "#PWR0641" (id 0) (at 67.31 107.95 0)
       (effects (font (size 1.27 1.27)) hide)
     )
@@
   (symbol (lib_id "power:VCC") (at 135.89 46.99 0)
     (in_bom yes) (on_board yes)
-    (property "Reference" "#PWR0634" (id 0) (at 135.89 50.8 0)
+    (property "Reference" "#PWR0633" (id 0) (at 135.89 50.8 0)
       (effects (font (size 1.27 1.27)) hide)
     )
@@
   (symbol (lib_id "power:GND") (at 67.31 87.63 0)
     (in_bom yes) (on_board yes)
-    (property "Reference" "#PWR0637" (id 0) (at 67.31 93.98 0)
+    (property "Reference" "#PWR0636" (id 0) (at 67.31 93.98 0)
       (effects (font (size 1.27 1.27)) hide)
     )
@@
   (symbol (lib_id "power:GND") (at 67.31 130.81 0)
     (in_bom yes) (on_board yes)
-    (property "Reference" "#PWR0643" (id 0) (at 67.31 137.16 0)
+    (property "Reference" "#PWR0642" (id 0) (at 67.31 137.16 0)
       (effects (font (size 1.27 1.27)) hide)
     )
@@
   (symbol (lib_id "power:GND") (at 93.98 95.25 0)
     (in_bom yes) (on_board yes)
-    (property "Reference" "#PWR0638" (id 0) (at 93.98 101.6 0)
+    (property "Reference" "#PWR0637" (id 0) (at 93.98 101.6 0)
       (effects (font (size 1.27 1.27)) hide)
     )
@@
   (symbol (lib_id "power:GND") (at 119.38 96.52 0)
     (in_bom yes) (on_board yes)
-    (property "Reference" "#PWR0640" (id 0) (at 119.38 102.87 0)
+    (property "Reference" "#PWR0639" (id 0) (at 119.38 102.87 0)
       (effects (font (size 1.27 1.27)) hide)
     )
@@
   (symbol (lib_id "power:GND") (at 148.59 96.52 0)
     (in_bom yes) (on_board yes)
-    (property "Reference" "#PWR0641" (id 0) (at 148.59 102.87 0)
+    (property "Reference" "#PWR0640" (id 0) (at 148.59 102.87 0)
       (effects (font (size 1.27 1.27)) hide)
     )
@@
   (symbol (lib_id "power:GND") (at 205.74 63.5 90)
     (in_bom yes) (on_board yes)
-    (property "Reference" "#PWR0635" (id 0) (at 212.09 63.5 0)
+    (property "Reference" "#PWR0634" (id 0) (at 212.09 63.5 0)
       (effects (font (size 1.27 1.27)) hide)
     )
@@
   (symbol (lib_id "power:GND") (at 205.74 68.58 90)
     (in_bom yes) (on_board yes)
-    (property "Reference" "#PWR0636" (id 0) (at 212.09 68.58 0)
+    (property "Reference" "#PWR0635" (id 0) (at 212.09 68.58 0)
       (effects (font (size 1.27 1.27)) hide)
     )
@@
   (symbol (lib_id "power:GND") (at 240.03 95.25 0)
     (in_bom yes) (on_board yes)
-    (property "Reference" "#PWR0639" (id 0) (at 240.03 101.6 0)
+    (property "Reference" "#PWR0638" (id 0) (at 240.03 101.6 0)
       (effects (font (size 1.27 1.27)) hide)
     )
@@
   (symbol (lib_id "Transistor_FET:2N7002") (at 64.77 82.55 0)
     (in_bom yes) (on_board yes)
-    (property "Reference" "Q738" (id 0) (at 70.0024 81.3816 0)
+    (property "Reference" "Q735" (id 0) (at 70.0024 81.3816 0)
       (effects (font (size 1.27 1.27)) (justify left))
     )
@@
   (symbol (lib_id "Transistor_FET:2N7002") (at 64.77 125.73 0)
     (in_bom yes) (on_board yes)
-    (property "Reference" "Q743" (id 0) (at 70.0024 124.5616 0)
+    (property "Reference" "Q740" (id 0) (at 70.0024 124.5616 0)
       (effects (font (size 1.27 1.27)) (justify left))
     )
@@
   (symbol (lib_id "Transistor_FET:2N7002") (at 91.44 80.01 0)
     (in_bom yes) (on_board yes)
-    (property "Reference" "Q734" (id 0) (at 96.6724 78.8416 0)
+    (property "Reference" "Q731" (id 0) (at 96.6724 78.8416 0)
       (effects (font (size 1.27 1.27)) (justify left))
     )
@@
   (symbol (lib_id "Transistor_FET:2N7002") (at 91.44 90.17 0)
     (in_bom yes) (on_board yes)
-    (property "Reference" "Q739" (id 0) (at 96.6724 89.0016 0)
+    (property "Reference" "Q736" (id 0) (at 96.6724 89.0016 0)
       (effects (font (size 1.27 1.27)) (justify left))
     )
@@
   (symbol (lib_id "Transistor_FET:2N7002") (at 116.84 81.28 0)
     (in_bom yes) (on_board yes)
-    (property "Reference" "Q736" (id 0) (at 122.0724 80.1116 0)
+    (property "Reference" "Q733" (id 0) (at 122.0724 80.1116 0)
       (effects (font (size 1.27 1.27)) (justify left))
     )
@@
   (symbol (lib_id "Transistor_FET:2N7002") (at 116.84 91.44 0)
     (in_bom yes) (on_board yes)
-    (property "Reference" "Q741" (id 0) (at 122.0724 90.2716 0)
+    (property "Reference" "Q738" (id 0) (at 122.0724 90.2716 0)
       (effects (font (size 1.27 1.27)) (justify left))
     )
@@
   (symbol (lib_id "Transistor_FET:2N7002") (at 146.05 81.28 0)
     (in_bom yes) (on_board yes)
-    (property "Reference" "Q737" (id 0) (at 151.2824 80.1116 0)
+    (property "Reference" "Q734" (id 0) (at 151.2824 80.1116 0)
       (effects (font (size 1.27 1.27)) (justify left))
     )
@@
   (symbol (lib_id "Transistor_FET:2N7002") (at 146.05 91.44 0)
     (in_bom yes) (on_board yes)
-    (property "Reference" "Q742" (id 0) (at 151.2824 90.2716 0)
+    (property "Reference" "Q739" (id 0) (at 151.2824 90.2716 0)
       (effects (font (size 1.27 1.27)) (justify left))
     )
@@
   (symbol (lib_id "Transistor_FET:2N7002") (at 237.49 80.01 0)
     (in_bom yes) (on_board yes)
-    (property "Reference" "Q735" (id 0) (at 242.7224 78.8416 0)
+    (property "Reference" "Q732" (id 0) (at 242.7224 78.8416 0)
       (effects (font (size 1.27 1.27)) (justify left))
     )
@@
   (symbol (lib_id "Transistor_FET:2N7002") (at 237.49 90.17 0)
     (in_bom yes) (on_board yes)
-    (property "Reference" "Q740" (id 0) (at 242.7224 89.0016 0)
-      (effects (font (size 1.27 1.27)) (justify left))
-    )
+    (property "Reference" "Q737" (id 0) (at 242.7224 89.0016 0)
+      (effects (font (size 1.27 1.27)) (justify left))
+    )
