File: pcb/decode.kicad_sch (KiCad schematic)
At the start: 21 parts, among them Q82 2N7002, Q83 2N7002, Q84 2N7002, Q85 2N7002, Q86 2N7002, Q87 2N7002, Q88 2N7002, Q89 2N7002, Q90 2N7002, Q91 2N7002, Q92 2N7002, Q93 2N7002, Q94 2N7002, Q95 2N7002, Q96 2N7002

Commit message: Revision 3.
Parts:
- added R366: 10k, Resistor_SMD:R_0805_2012Metric, symbol Device:R
Connections:
- net VCC: now also R366.1
- net ~STATE_LOAD: now also R366.2; no longer Q82.3 (D), R36.2
- new net ~STATE_DEREF: Q82.3 (D), R36.2
Changed lines of the file:
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@@
   (junction (at 86.36 71.12) (diameter 1.016) (color 0 0 0 0))
   (junction (at 86.36 86.36) (diameter 0.9144) (color 0 0 0 0))
-  (junction (at 110.49 44.45) (diameter 0.9144) (color 0 0 0 0))
+  (junction (at 110.49 43.815) (diameter 0.9144) (color 0 0 0 0))
   (junction (at 119.38 152.4) (diameter 0.9144) (color 0 0 0 0))
-  (junction (at 120.65 44.45) (diameter 0.9144) (color 0 0 0 0))
+  (junction (at 138.43 43.18) (diameter 0.9144) (color 0 0 0 0))
   (junction (at 138.43 69.85) (diameter 1.016) (color 0 0 0 0))
   (junction (at 138.43 86.36) (diameter 0.9144) (color 0 0 0 0))
@@
     (stroke (width 0) (type solid) (color 0 0 0 0))
   )
-  (wire (pts (xy 110.49 39.37) (xy 110.49 44.45))
-    (stroke (width 0) (type solid) (color 0 0 0 0))
-  )
-  (wire (pts (xy 110.49 44.45) (xy 110.49 46.99))
-    (stroke (width 0) (type solid) (color 0 0 0 0))
-  )
-  (wire (pts (xy 110.49 44.45) (xy 120.65 44.45))
+  (wire (pts (xy 110.49 39.37) (xy 110.49 43.815))
+    (stroke (width 0) (type solid) (color 0 0 0 0))
+  )
+  (wire (pts (xy 110.49 43.815) (xy 110.49 46.99))
+    (stroke (width 0) (type solid) (color 0 0 0 0))
+  )
+  (wire (pts (xy 110.49 43.815) (xy 119.38 43.815))
     (stroke (width 0) (type solid) (color 0 0 0 0))
   )
@@
     (stroke (width 0) (type solid) (color 0 0 0 0))
   )
+  (wire (pts (xy 119.38 43.815) (xy 119.38 39.37))
+    (stroke (width 0) (type solid) (color 0 0 0 0))
+  )
   (wire (pts (xy 119.38 134.62) (xy 119.38 139.7))
     (stroke (width 0) (type solid) (color 0 0 0 0))
@@
     (stroke (width 0) (type solid) (color 0 0 0 0))
   )
-  (wire (pts (xy 120.65 39.37) (xy 120.65 44.45))
-    (stroke (width 0) (type solid) (color 0 0 0 0))
-  )
-  (wire (pts (xy 120.65 44.45) (xy 138.43 44.45))
-    (stroke (width 0) (type solid) (color 0 0 0 0))
-  )
-  (wire (pts (xy 138.43 44.45) (xy 138.43 46.99))
+  (wire (pts (xy 138.43 39.37) (xy 138.43 43.18))
+    (stroke (width 0) (type solid) (color 0 0 0 0))
+  )
+  (wire (pts (xy 138.43 43.18) (xy 138.43 46.99))
+    (stroke (width 0) (type solid) (color 0 0 0 0))
+  )
+  (wire (pts (xy 138.43 43.18) (xy 146.685 43.18))
     (stroke (width 0) (type solid) (color 0 0 0 0))
   )
@@
   )
   (wire (pts (xy 146.05 134.62) (xy 146.05 146.05))
+    (stroke (width 0) (type solid) (color 0 0 0 0))
+  )
+  (wire (pts (xy 146.685 43.18) (xy 146.685 39.37))
     (stroke (width 0) (type solid) (color 0 0 0 0))
   )
@@
     (effects (font (size 1.27 1.27)) (justify left bottom))
   )
-  (text "Fanout to 2 gates (0.7us)" (at 111.125 24.13 0)
+  (text "Fanout to 2 gates (0.7us)" (at 117.475 24.13 0)
     (effects (font (size 1.27 1.27)) (justify left bottom))
   )
@@
     (effects (font (size 1.27 1.27)) (justify left))
   )
-  (hierarchical_label "~STATE_LOAD" (shape input) (at 120.65 39.37 90)
+  (hierarchical_label "~STATE_DEREF" (shape input) (at 119.38 39.37 90)
+    (effects (font (size 1.27 1.27)) (justify left))
+  )
+  (hierarchical_label "~STATE_LOAD" (shape input) (at 146.685 39.37 90)
     (effects (font (size 1.27 1.27)) (justify left))
   )
@@
     (pin "1")
   )
+  (symbol (lib_id "power:VCC") (at 138.43 31.75 0) (unit 1)
+    (in_bom yes) (on_board yes)
+    (property "Reference" "#PWR0982" (id 0) (at 138.43 35.56 0)
+      (effects (font (size 1.27 1.27)) hide)
+    )
+    (property "Value" "VCC" (id 1) (at 138.8618 27.3558 0))
+    (property "Footprint" "" (id 2) (at 138.43 31.75 0)
+      (effects (font (size 1.27 1.27)) hide)
+    )
+    (property "Datasheet" "" (id 3) (at 138.43 31.75 0)
+      (effects (font (size 1.27 1.27)) hide)
+    )
+    (pin "1")
+  )
   (symbol (lib_id "power:VCC") (at 146.05 118.11 0) (unit 1)
     (in_bom yes) (on_board yes)
@@
       (effects (font (size 1.27 1.27)) hide)
     )
+    (pin "1")
+    (pin "2")
+  )
+  (symbol (lib_id "Device:R") (at 138.43 35.56 0) (unit 1)
+    (in_bom yes) (on_board yes)
+    (property "Reference" "R366" (id 0) (at 140.208 34.3916 0)
+      (effects (font (size 1.27 1.27)) (justify left))
+    )
+    (property "Value" "10k" (id 1) (at 140.208 36.703 0)
+      (effects (font (size 1.27 1.27)) (justify left))
+    )
+    (property "Footprint" "Resistor_SMD:R_0805_2012Metric" (id 2) (at 136.652 35.56 90)
+      (effects (font (size 1.27 1.27)) hide)
+    )
+    (property "Datasheet" "~" (id 3) (at 138.43 35.56 0)
+      (effects (font (size 1.27 1.27)) hide)
+    )
+    (property "LCSC" "C17414" (id 4) (at 138.43 35.56 0)
+      (effects (font (size 1.27 1.27)) hide)
+    )
