File: pcb/xlreg.kicad_sch (KiCad schematic)
At the start: 9 parts, among them Q1058 2N7002a, Q1059 2N7002a, Q1060 2N7002a, Q1061 2N7002a, Q1062 2N7002a, Q1063 2N7002a, Q1064 2N7002a

Commit message: New reset.
Parts:
- renumbered R466 to R465, R467 to R466
Changed lines of the file:
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@@
   (symbol (lib_id "power:VCC") (at 67.31 104.14 0)
     (in_bom yes) (on_board yes)
-    (property "Reference" "#PWR0953" (id 0) (at 67.31 107.95 0)
+    (property "Reference" "#PWR0952" (id 0) (at 67.31 107.95 0)
       (effects (font (size 1.27 1.27)) hide)
     )
@@
   (symbol (lib_id "power:VCC") (at 135.89 46.99 0)
     (in_bom yes) (on_board yes)
-    (property "Reference" "#PWR0947" (id 0) (at 135.89 50.8 0)
+    (property "Reference" "#PWR0946" (id 0) (at 135.89 50.8 0)
       (effects (font (size 1.27 1.27)) hide)
     )
@@
   (symbol (lib_id "power:GND") (at 67.31 130.81 0)
     (in_bom yes) (on_board yes)
-    (property "Reference" "#PWR0954" (id 0) (at 67.31 137.16 0)
+    (property "Reference" "#PWR0953" (id 0) (at 67.31 137.16 0)
       (effects (font (size 1.27 1.27)) hide)
     )
@@
   (symbol (lib_id "power:GND") (at 93.98 95.25 0)
     (in_bom yes) (on_board yes)
-    (property "Reference" "#PWR0950" (id 0) (at 93.98 101.6 0)
+    (property "Reference" "#PWR0949" (id 0) (at 93.98 101.6 0)
       (effects (font (size 1.27 1.27)) hide)
     )
@@
   (symbol (lib_id "power:GND") (at 148.59 96.52 0)
     (in_bom yes) (on_board yes)
-    (property "Reference" "#PWR0952" (id 0) (at 148.59 102.87 0)
+    (property "Reference" "#PWR0951" (id 0) (at 148.59 102.87 0)
       (effects (font (size 1.27 1.27)) hide)
     )
@@
   (symbol (lib_id "power:GND") (at 205.74 63.5 90)
     (in_bom yes) (on_board yes)
-    (property "Reference" "#PWR0948" (id 0) (at 212.09 63.5 0)
+    (property "Reference" "#PWR0947" (id 0) (at 212.09 63.5 0)
       (effects (font (size 1.27 1.27)) hide)
     )
@@
   (symbol (lib_id "power:GND") (at 205.74 68.58 90)
     (in_bom yes) (on_board yes)
-    (property "Reference" "#PWR0949" (id 0) (at 212.09 68.58 0)
+    (property "Reference" "#PWR0948" (id 0) (at 212.09 68.58 0)
       (effects (font (size 1.27 1.27)) hide)
     )
@@
   (symbol (lib_id "power:GND") (at 240.03 95.25 0)
     (in_bom yes) (on_board yes)
-    (property "Reference" "#PWR0951" (id 0) (at 240.03 101.6 0)
+    (property "Reference" "#PWR0950" (id 0) (at 240.03 101.6 0)
       (effects (font (size 1.27 1.27)) hide)
     )
@@
   (symbol (lib_id "Device:R") (at 67.31 107.95 0)
     (in_bom yes) (on_board yes)
-    (property "Reference" "R467" (id 0) (at 69.088 106.7816 0)
+    (property "Reference" "R466" (id 0) (at 69.088 106.7816 0)
       (effects (font (size 1.27 1.27)) (justify left))
     )
@@
   (symbol (lib_id "Device:R") (at 135.89 50.8 0)
     (in_bom yes) (on_board yes)
-    (property "Reference" "R466" (id 0) (at 137.668 49.6316 0)
+    (property "Reference" "R465" (id 0) (at 137.668 49.6316 0)
       (effects (font (size 1.27 1.27)) (justify left))
     )

Commit message: Some fixes.
Parts:
- renumbered Q1058 to Q1054, Q1059 to Q1055, Q1060 to Q1056, Q1064 to Q1057, Q1061 to Q1058, Q1062 to Q1059, Q1063 to Q1060, R465 to R469, R466 to R470
Other:
- moved on the sheet: Q1057, R470

Commit message: Faster.
Parts:
- Q1047: renamed from Q1054; value 2N7002a -> 2N7002; LCSC C8545 -> C181083
- Q1048: renamed from Q1055; value 2N7002a -> 2N7002; LCSC C8545 -> C181083
- Q1049: renamed from Q1056; value 2N7002a -> 2N7002; LCSC C8545 -> C181083
- Q1050: renamed from Q1057; value 2N7002a -> 2N7002; LCSC C8545 -> C181083
- Q1051: renamed from Q1058; value 2N7002a -> 2N7002; LCSC C8545 -> C181083
- Q1052: renamed from Q1059; value 2N7002a -> 2N7002; LCSC C8545 -> C181083
- Q1053: renamed from Q1060; value 2N7002a -> 2N7002; LCSC C8545 -> C181083
- renumbered R469 to R466, R470 to R467
