File: pcb/logic.kicad_sch (KiCad schematic)
At the start: 66 parts, among them Q179 2N7002a, Q180 2N7002a, Q181 2N7002a, Q182 2N7002a, Q183 2N7002a, Q184 2N7002a, Q185 2N7002a, Q186 2N7002a, Q187 2N7002a, Q188 2N7002a, Q189 2N7002a, Q190 2N7002a, Q191 2N7002a, Q192 2N7002a, Q193 2N7002a, Q194 2N7002a, Q195 2N7002a, Q196 2N7002a, Q197 2N7002a, Q198 2N7002a, Q199 2N7002a, Q200 2N7002a, Q201 2N7002a, Q202 2N7002a, Q203 2N7002a, Q204 2N7002a, Q205 2N7002a, Q206 2N7002a, Q207 2N7002a, Q208 2N7002a, Q209 2N7002a, Q210 2N7002a, Q211 2N7002a, Q212 2N7002a, Q213 2N7002a, Q214 2N7002a, Q215 2N7002a, Q216 2N7002a, Q217 2N7002a, Q218 2N7002a, Q219 2N7002a, Q220 2N7002a, Q221 2N7002a, Q222 2N7002a, Q223 2N7002a, Q224 2N7002a, Q225 2N7002a

Commit message: Pi programmer.
Parts:
- added Q1126, Q1127: 2N7002a, Package_TO_SOT_SMD:SOT-23, symbol Transistor_FET:2N7002
- added R484: 10k, Resistor_SMD:R_0805_2012Metric, symbol Device:R
- renumbered C7 to C6, Q182 to Q100, Q183 to Q101, Q184 to Q102, Q185 to Q103, Q186 to Q104, Q187 to Q105, Q188 to Q106, Q189 to Q107, Q190 to Q108, Q191 to Q109, Q192 to Q110, Q193 to Q111, Q194 to Q112, Q195 to Q113, Q196 to Q114, Q197 to Q115, Q198 to Q116, Q199 to Q117, Q200 to Q118, Q201 to Q119, Q202 to Q120, Q203 to Q121, Q204 to Q122, Q205 to Q123, Q206 to Q124, Q207 to Q125, Q208 to Q126, Q209 to Q127, Q210 to Q128, Q211 to Q129, Q212 to Q130, Q213 to Q131, Q214 to Q132, Q215 to Q133, Q216 to Q134, Q217 to Q135, Q218 to Q136, Q219 to Q137, Q220 to Q138, Q221 to Q139, Q222 to Q140, Q223 to Q141, Q224 to Q142, Q225 to Q143, Q179 to Q97, Q180 to Q98, Q181 to Q99, R76 to R41, R77 to R42, R78 to R43, R79 to R44, R80 to R45, R81 to R46, R82 to R47, R83 to R48, R84 to R49, R85 to R50, R86 to R51, R87 to R52, R88 to R53, R89 to R54, R90 to R55, R91 to R56, R92 to R57, R93 to R58
Connections:
- net GND: now also Q1126.2 (S), Q1127.2 (S); no longer Q99.2 (S)
- net RDP_ABUS: now also Q1127.1 (G)
- net VCC: now also R484.1
- net ~STATE_ALU: now also Q1126.1 (G)
- new net: Q1126.3 (D), Q99.2 (S)
- new net RDX_ABUS: Q1127.3 (D), R484.2
Other:
- note added: "Fanout to 13 gates."
- note added: "Set ABUS to P for FETCH and ALU (ignored)."
- note added: "Set ABUS to X for LOAD and DEREF."
- note removed: "Fanout to 12 gates."
- note removed: "Set ABUS to P to fetch the instruction."
- moved on the sheet: C6, Q112, Q113, Q117, Q118, Q121, R50, R53, R54

Commit message: Buttons.
Parts:
- removed Q1126, Q1127: 2N7002a, Package_TO_SOT_SMD:SOT-23, symbol Transistor_FET:2N7002
- removed R484: 10k, Resistor_SMD:R_0805_2012Metric, symbol Device:R
- renumbered Q119 to Q118, Q120 to Q119, Q118 to Q120
Connections:
- net GND: now also Q99.2 (S)
Other:
- note added: "Fanout to 12 gates."
- note added: "Set ABUS to P for FETCH."
- note removed: "Fanout to 13 gates."
- note removed: "Set ABUS to P for FETCH and ALU (ignored)."
- note removed: "Set ABUS to X for LOAD and DEREF."
- moved on the sheet: C6, Q112, Q113, Q117, Q120, Q121, R50, R53, R54

Commit message: Some fixes.
Parts:
- removed Q107: 2N7002a, Package_TO_SOT_SMD:SOT-23, symbol Transistor_FET:2N7002
- removed R41, R45, R47, R55, R58: 10k, Resistor_SMD:R_0805_2012Metric, symbol Device:R
- added R39, R56: 1k, Resistor_SMD:R_0805_2012Metric, symbol Device:R
- added R48, R59: 10k, Resistor_SMD:R_0805_2012Metric, symbol Device:R
- R46: value 4.7k -> 10k; LCSC C17673 -> C17414
- renumbered C6 to C7, Q103 to Q100, Q99 to Q101, Q100 to Q102, Q101 to Q103, Q110 to Q107, Q111 to Q108, Q112 to Q109, Q113 to Q110, Q116 to Q111, Q108 to Q112, Q109 to Q113, Q117 to Q116, Q120 to Q117, Q121 to Q118, Q118 to Q119, Q119 to Q120, Q124 to Q121, Q126 to Q123, Q127 to Q124, Q128 to Q125, Q129 to Q126, Q130 to Q127, Q123 to Q128, Q125 to Q129, Q131 to Q130, Q132 to Q131, Q133 to Q132, Q134 to Q133, Q138 to Q134, Q139 to Q138, Q140 to Q139, Q141 to Q140, Q142 to Q141, Q143 to Q142, Q98 to Q97, Q97 to Q98, Q102 to Q99, R42 to R44, R44 to R45, R48 to R51, R51 to R52, R52 to R55, R56 to R57, R57 to R58
Connections:
- net ~DBUS7 is gone; now on net XHIN_P: Q100.1 (G)
- net RDA_DBUS: now also R56.2
- net RDP_ABUS: now also R46.2
- net VCC: now also R39.1, R48.1, R56.1, R59.1
- net WRM: now also R59.2
- net WRO: now also R39.2; no longer R46.2
- net XIN_SHIFT: now also R48.2
Other:
- note added: "Capacitive load on DBUS is limited to 5 gates. At 50pF per gate, this gives 1.7us delay from DBUS valid to write. SRAM is 70ns from ABUS valid to DBUS valid (we round to 0.1us)."
- note added: "Clock fanout to 12 DFFs (24 gates) SC to WRA: 5+0.8=5.8us."
- note added: "Clock fanout to 12 DFFs (24 gates) SC to WRX: 5+0.8=5.8us"
- note added: "Clock fanout to 8 gates. SC to WRO: 5+0.3=5.3us."
- note added: "Fanout to 12 gates. SC to RDP: 5+4.2=9.2us. ABUS valid to DBUS valid is 0.1us, so a total of 9.3us."
- note added: "Fanout to 12 gates. SC to XIN_SHIFT: 5+4.2=9.2us."
- note added: "Fanout to 2 gates. SC to INCP_CLK: 5+0.7=5.7us. P is 12 levels, 2 gates per level, so the delay from INCP_CLK to P is: 8.4us."
- note added: "Fanout to 2 gates. SC to WRF: 5+0.7=5.7us."
- note added: "Fanout to 2 gates. SC to WRM: 5+0.7=5.7us."
- note added: "Fanout to 5 gates. SC to XHIN_DBUS: 5+1.7=6.7us."
- note added: "Fanout to 6 gates. WS to ~WS~ is 0.2us."
- note added: "Relative (Z=0). Fanout to 5 gates. SC to XHIN_P: 5+1.7=6.7us."
- note added: "Set DBUS = A. Fanout to 12 gates. SC to RDA: 5+0.4=5.4us. SC to DBUS: 5.4+1.7=7.1us."
- note added: "Set P = X Fanout to 24 gates. SC to ~WRP~: 5.4+0.8=6.2us."
- note added: "The max delay from SC through the control lines is based on the max delay through the state decoder (5us) plus the time through the control logic. Max delay is under 10us. Assuming 10us, we should be able to run the clock at 100 kHz."
- note added: "When not running, ~WS~ will be high, allowing the INCP switch to let INCP_CLK float high when pressed."
- note added: "Write operand Saves the top 4 bits of DBUS to the top 4 bits of the state register. This happens in the same state as P is incremented, so it must be fast."
- note added: "Zero-Page (Z=1). Fanout to 5 gates. SC to XHIN_ZERO: 6.7+1.7=8.4us."
- note removed: "Clock fanout to 12 DFFs (24 gates)"
- note removed: "Fanout to 12 gates."
- note removed: "Fanout to 2 gates"
- note removed: "Fanout to 6 gates"
- note removed: "Fanout to 8 gates"
- note removed: "Relative (Z=0)"
- note removed: "Set DBUS = A"
- note removed: "Set P = X Fanout to 24 gates"
- note removed: "Write operand Saves the top 4 bits of DBUS to the top 4 bits of the state register."
- note removed: "Zero-Page (Z=1)"
- moved on the sheet: C7, Q100, Q101, Q102, Q103, Q106, Q107, Q108, Q109, Q110, Q111, Q114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

Commit message: Faster.
Parts:
- removed Q106, Q128: 2N7002a, Package_TO_SOT_SMD:SOT-23, symbol Transistor_FET:2N7002
- removed R48: 10k, Resistor_SMD:R_0805_2012Metric, symbol Device:R
- added R44: 1k, Resistor_SMD:R_0805_2012Metric, symbol Device:R
- Q100, Q101, Q102, Q103, Q104, Q105, Q97, Q98, Q99: value 2N7002a -> 2N7002; LCSC C8545 -> C181083
- Q106: renamed from Q107; value 2N7002a -> 2N7002; LCSC C8545 -> C181083
- Q107: renamed from Q108; value 2N7002a -> 2N7002; LCSC C8545 -> C181083
- Q108: renamed from Q109; value 2N7002a -> 2N7002; LCSC C8545 -> C181083
- Q109: renamed from Q110; value 2N7002a -> 2N7002; LCSC C8545 -> C181083
- Q110: renamed from Q111; value 2N7002a -> 2N7002; LCSC C8545 -> C181083
- Q111: renamed from Q112; value 2N7002a -> 2N7002; LCSC C8545 -> C181083
- Q112: renamed from Q113; value 2N7002a -> 2N7002; LCSC C8545 -> C181083
- Q113: renamed from Q114; value 2N7002a -> 2N7002; LCSC C8545 -> C181083
- Q114: renamed from Q115; value 2N7002a -> 2N7002; LCSC C8545 -> C181083
- Q115: renamed from Q116; value 2N7002a -> 2N7002; LCSC C8545 -> C181083
- Q116: renamed from Q117; value 2N7002a -> 2N7002; LCSC C8545 -> C181083
- Q117: renamed from Q118; value 2N7002a -> 2N7002; LCSC C8545 -> C181083
- Q118: renamed from Q119; value 2N7002a -> 2N7002; LCSC C8545 -> C181083
- Q119: renamed from Q120; value 2N7002a -> 2N7002; LCSC C8545 -> C181083
- Q120: renamed from Q121; value 2N7002a -> 2N7002; LCSC C8545 -> C181083
- Q121: renamed from Q122; value 2N7002a -> 2N7002; LCSC C8545 -> C181083
- Q122: renamed from Q123; value 2N7002a -> 2N7002; LCSC C8545 -> C181083
- Q123: renamed from Q124; value 2N7002a -> 2N7002; LCSC C8545 -> C181083
- Q124: renamed from Q125; value 2N7002a -> 2N7002; LCSC C8545 -> C181083
- Q125: renamed from Q126; value 2N7002a -> 2N7002; LCSC C8545 -> C181083
- Q126: renamed from Q127; value 2N7002a -> 2N7002; LCSC C8545 -> C181083
- Q127: renamed from Q129; value 2N7002a -> 2N7002; LCSC C8545 -> C181083
- Q128: renamed from Q130; value 2N7002a -> 2N7002; LCSC C8545 -> C181083
- Q129: renamed from Q131; value 2N7002a -> 2N7002; LCSC C8545 -> C181083
- Q130: renamed from Q132; value 2N7002a -> 2N7002; LCSC C8545 -> C181083
- Q131: renamed from Q133; value 2N7002a -> 2N7002; LCSC C8545 -> C181083
- Q132: renamed from Q134; value 2N7002a -> 2N7002; LCSC C8545 -> C181083
- Q133: renamed from Q135; value 2N7002a -> 2N7002; LCSC C8545 -> C181083
- Q134: renamed from Q136; value 2N7002a -> 2N7002; LCSC C8545 -> C181083
- Q135: renamed from Q137; value 2N7002a -> 2N7002; LCSC C8545 -> C181083
- Q136: renamed from Q138; value 2N7002a -> 2N7002; LCSC C8545 -> C181083
- Q137: renamed from Q139; value 2N7002a -> 2N7002; LCSC C8545 -> C181083
- Q138: renamed from Q140; value 2N7002a -> 2N7002; LCSC C8545 -> C181083
- Q139: renamed from Q141; value 2N7002a -> 2N7002; LCSC C8545 -> C181083
- Q140: renamed from Q142; value 2N7002a -> 2N7002; LCSC C8545 -> C181083
- R46: value 10k -> 1k; LCSC C17414 -> C17513
- renumbered C7 to C8, R43 to R41, R44 to R42, R45 to R43, R39 to R45, R49 to R47, R50 to R48, R51 to R49, R52 to R50, R53 to R51, R54 to R52, R55 to R53, R56 to R54, R57 to R55, R58 to R56, R59 to R57
Connections:
- net GND: now also Q97.2 (S)
- net RDP_ABUS: now also R44.2; no longer R46.2
- net VCC: now also R44.1
- net XIN_SHIFT: now also R46.2
- net at Q127.3 (D): now also Q121.2 (S)
Other:
- note added: "Clock fanout to 12 DFFs (24 gates, 0.8us)"
- note added: "Fanout to 12 gates (0.4us)"
- note added: "Fanout to 2 gates (0.7 us)."
- note added: "Fanout to 2 gates (0.7us)"
- note added: "Fanout to 2 gates (0.7us). P is 12 levels, 2 gates per level each with a fanout of 3, so the delay from INCP_CLK to P is 25us, but the result is not needed until the next FETCH."
- note added: "Fanout to 5 gates (1.7us)"
- note added: "Fanout to 8 gates (0.3us)"
- note added: "Relative (Z=0) Fanout to 5 gates (1.7us)"
- note added: "Set DBUS = A. Fanout to 13 gates (0.5us)"
- note added: "Set P = X Fanout to 24 gates (0.5+0.8=1.3us)."
- note added: "The max delay from SC through the control lines is based on the max delay through the state decoder plus the delay through the control logic. This gives us 10.1+1.7=11.7us. Assuming 12us, we should be able to run the clock at 80 kHz safely."
- note added: "Zero-Page (Z=1). Fanout to 5 gates (1.7us)"
- note removed: "Clock fanout to 12 DFFs (24 gates) SC to WRA: 5+0.8=5.8us."
- note removed: "Clock fanout to 12 DFFs (24 gates) SC to WRX: 5+0.8=5.8us"
- note removed: "Clock fanout to 8 gates. SC to WRO: 5+0.3=5.3us."
- note removed: "Fanout to 12 gates. SC to RDP: 5+4.2=9.2us. ABUS valid to DBUS valid is 0.1us, so a total of 9.3us."
- note removed: "Fanout to 12 gates. SC to XIN_SHIFT: 5+4.2=9.2us."
- note removed: "Fanout to 2 gates. SC to INCP_CLK: 5+0.7=5.7us. P is 12 levels, 2 gates per level, so the delay from INCP_CLK to P is: 8.4us."
- note removed: "Fanout to 2 gates. SC to WRF: 5+0.7=5.7us."
- note removed: "Fanout to 2 gates. SC to WRM: 5+0.7=5.7us."
- note removed: "Fanout to 5 gates. SC to XHIN_DBUS: 5+1.7=6.7us."
- note removed: "Relative (Z=0). Fanout to 5 gates. SC to XHIN_P: 5+1.7=6.7us."
- note removed: "Set DBUS = A. Fanout to 12 gates. SC to RDA: 5+0.4=5.4us. SC to DBUS: 5.4+1.7=7.1us."
- note removed: "Set P = X Fanout to 24 gates. SC to ~WRP~: 5.4+0.8=6.2us."
- note removed: "The max delay from SC through the control lines is based on the max delay through the state decoder (5us) plus the time through the control logic. Max delay is under 10us. Assuming 10us, we should be able to run the clock at 100 kHz."
- note removed: "Zero-Page (Z=1). Fanout to 5 gates. SC to XHIN_ZERO: 6.7+1.7=8.4us."
- moved on the sheet: Q127
