File: pcb/q2/address.kicad_sch (KiCad schematic)
At the start: 27 parts

Commit message: PCB fixes/updates.
Parts:
- Q637, Q638, Q639, Q640, Q641, Q642, Q643, Q644, Q645, Q646, Q647, Q648, Q649, Q650, Q651, Q652, Q653: renamed from Q?; value (none) -> 2N7002; footprint (none) -> Package_TO_SOT_SMD:SOT-23
- R287, R288, R289, R290, R291, R292, R293, R294, R295, R296: renamed from R?; value (none) -> 10k; footprint (none) -> Resistor_SMD:R_0603_1608Metric
