File: pcb/q2/areg.kicad_sch (KiCad schematic)
At the start: 2 parts

Commit message: PCB fixes/updates.
Parts:
- Q3, Q4: renamed from Q?; value (none) -> 2N7002; footprint (none) -> Package_TO_SOT_SMD:SOT-23
Connections:
- net RDA renamed STATE_EXEC
Changed lines of the file:
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@@
     (stroke (width 0) (type default) (color 0 0 0 0))
   )
-  (global_label "RDA" (shape input) (at 156.21 93.98 180) (fields_autoplaced)
+  (global_label "STATE_EXEC" (shape input) (at 156.21 93.98 180) (fields_autoplaced)
     (effects (font (size 1.27 1.27)) (justify right))
-    (property "Intersheet References" "${INTERSHEET_REFS}" (id 0) (at 0 0 0)
-      (effects (font (size 1.27 1.27)) hide)
+    (property "Intersheet References" "${INTERSHEET_REFS}" (id 0) (at 142.7582 93.9006 0)
+      (effects (font (size 1.27 1.27)) (justify right) hide)
     )
   )
@@
   (symbol (lib_id "Transistor_FET:2N7002") (at 161.29 83.82 0) (unit 1)
     (in_bom yes) (on_board yes)
-    (property "Reference" "Q?" (id 0) (at 166.4716 82.6516 0)
+    (property "Reference" "Q3" (id 0) (at 166.4716 82.6516 0)
       (effects (font (size 1.27 1.27)) (justify left))
     )
-    (property "Value" "" (id 1) (at 166.4716 84.963 0)
+    (property "Value" "2N7002" (id 1) (at 166.4716 84.963 0)
       (effects (font (size 1.27 1.27)) (justify left))
     )
-    (property "Footprint" "" (id 2) (at 166.37 85.725 0)
+    (property "Footprint" "Package_TO_SOT_SMD:SOT-23" (id 2) (at 166.37 85.725 0)
       (effects (font (size 1.27 1.27) italic) (justify left) hide)
     )
@@
   (symbol (lib_id "Transistor_FET:2N7002") (at 161.29 93.98 0) (unit 1)
     (in_bom yes) (on_board yes)
-    (property "Reference" "Q?" (id 0) (at 166.4716 92.8116 0)
+    (property "Reference" "Q4" (id 0) (at 166.4716 92.8116 0)
       (effects (font (size 1.27 1.27)) (justify left))
     )
-    (property "Value" "" (id 1) (at 166.4716 95.123 0)
+    (property "Value" "2N7002" (id 1) (at 166.4716 95.123 0)
       (effects (font (size 1.27 1.27)) (justify left))
     )
-    (property "Footprint" "" (id 2) (at 166.37 95.885 0)
+    (property "Footprint" "Package_TO_SOT_SMD:SOT-23" (id 2) (at 166.37 95.885 0)
       (effects (font (size 1.27 1.27) italic) (justify left) hide)
     )
@@
   (symbol (lib_id "power:GND") (at 163.83 99.06 0) (unit 1)
     (in_bom yes) (on_board yes)
-    (property "Reference" "#PWR?" (id 0) (at 163.83 105.41 0)
+    (property "Reference" "#PWR012" (id 0) (at 163.83 105.41 0)
       (effects (font (size 1.27 1.27)) hide)
     )
-    (property "Value" "" (id 1) (at 163.957 103.4542 0))
+    (property "Value" "GND" (id 1) (at 163.957 103.4542 0))
     (property "Footprint" "" (id 2) (at 163.83 99.06 0)
       (effects (font (size 1.27 1.27)) hide)
@@
   (symbol (lib_id "power:GND") (at 116.84 86.36 270) (unit 1)
     (in_bom yes) (on_board yes)
-    (property "Reference" "#PWR?" (id 0) (at 110.49 86.36 0)
+    (property "Reference" "#PWR010" (id 0) (at 110.49 86.36 0)
       (effects (font (size 1.27 1.27)) hide)
     )
-    (property "Value" "" (id 1) (at 112.4458 86.487 0))
+    (property "Value" "GND" (id 1) (at 112.4458 86.487 0))
     (property "Footprint" "" (id 2) (at 116.84 86.36 0)
       (effects (font (size 1.27 1.27)) hide)
@@
   (symbol (lib_id "power:GND") (at 116.84 90.17 270) (unit 1)
     (in_bom yes) (on_board yes)
-    (property "Reference" "#PWR?" (id 0) (at 110.49 90.17 0)
+    (property "Reference" "#PWR011" (id 0) (at 110.49 90.17 0)
       (effects (font (size 1.27 1.27)) hide)
     )
-    (property "Value" "" (id 1) (at 112.4458 90.297 0))
+    (property "Value" "GND" (id 1) (at 112.4458 90.297 0))
     (property "Footprint" "" (id 2) (at 116.84 90.17 0)
       (effects (font (size 1.27 1.27)) hide)
@@
       (effects (font (size 1.27 1.27)) (justify left))
     )
-    (pin "Q" input (at 142.24 74.93 0)
+    (pin "Q" output (at 142.24 74.93 0)
       (effects (font (size 1.27 1.27)) (justify right))
     )
-    (pin "~{Q}" input (at 142.24 83.82 0)
+    (pin "~{Q}" output (at 142.24 83.82 0)
       (effects (font (size 1.27 1.27)) (justify right))
     )
