File: pcb/q2/i2c.kicad_sch (KiCad schematic)
At the start: 9 parts

Commit message: PCB fixes/updates.
Parts:
- D59, D60: renamed from D?; value (none) -> BAT43W; footprint (none) -> Diode_SMD:D_SOD-123
- J3: value (none) -> I2C; footprint (none) -> Connector_PinHeader_2.54mm:PinHeader_1x05_P2.54mm_Horizontal
- Q830, Q832: renamed from Q?; value (none) -> 2N7002; footprint (none) -> Package_TO_SOT_SMD:SOT-23
- Q831, Q833: renamed from Q?; value (none) -> 2N7002K; footprint (none) -> Package_TO_SOT_SMD:SOT-23
- R367, R368: renamed from R?; value (none) -> 10k; footprint (none) -> Resistor_SMD:R_0603_1608Metric
