File: pcb/q2/preg.kicad_sch (KiCad schematic)
At the start: 12 parts

Commit message: PCB fixes/updates.
Parts:
- Q38, Q39, Q40, Q41, Q42, Q43, Q45: renamed from Q?; value (none) -> 2N7002; footprint (none) -> Package_TO_SOT_SMD:SOT-23
- Q44, Q46, Q47, Q48: renamed from Q?; value (none) -> 2N7002K; footprint (none) -> Package_TO_SOT_SMD:SOT-23
- R18: renamed from R?; value (none) -> 100k; footprint (none) -> Resistor_SMD:R_0603_1608Metric
Connections:
- net RDP renamed STATE_FETCH
- no-connect marks 0 -> 1
