File: pcb/q2/slice-low.kicad_sch (KiCad schematic)
At the start: 8 parts

Commit message: PCB fixes/updates.
Parts:
- C22, C40: renamed from C?; value (none) -> 0.1u; footprint (none) -> Capacitor_SMD:C_0805_2012Metric
- Q834: renamed from Q?; value (none) -> 2N7002; footprint (none) -> Package_TO_SOT_SMD:SOT-23
- Q835, Q836: renamed from Q?; value (none) -> 2N7002K; footprint (none) -> Package_TO_SOT_SMD:SOT-23
- R369, R370: renamed from R?; value (none) -> 10k; footprint (none) -> Resistor_SMD:R_0603_1608Metric
- R371: renamed from R?; value (none) -> 100k; footprint (none) -> Resistor_SMD:R_0603_1608Metric
Other:
- sheet XL Register ports: added none; removed XIN_DBUS, XIN_SHIFT
