File: pcb/q2/ui.kicad_sch (KiCad schematic)
At the start: 16 parts

Commit message: PCB fixes/updates.
Parts:
- C28: renamed from C?; value (none) -> 0.1u; footprint (none) -> Capacitor_SMD:C_0805_2012Metric
- DS1: value (none) -> WC1602A; footprint (none) -> Display:WC1602A
- Q824, Q825, Q826, Q827, Q828, Q829: renamed from Q?; value (none) -> 2N7002; footprint (none) -> Package_TO_SOT_SMD:SOT-23
- R274: renamed from R?; value (none) -> 100; footprint (none) -> Resistor_SMD:R_1206_3216Metric
- R366: renamed from R?; value (none) -> 10k; footprint (none) -> Resistor_SMD:R_0603_1608Metric
- RV3: renamed from RV?; value (none) -> 10k; footprint (none) -> Potentiometer_THT:Potentiometer_Bourns_3386P_Vertical
- SW2, SW3, SW4, SW5, SW6: value (none) -> Button; footprint (none) -> Button_Switch_SMD:SW_SPST_PTS645
