File: pcb/q2/xhreg.kicad_sch (KiCad schematic)
At the start: 13 parts

Commit message: PCB fixes/updates.
Parts:
- Q16, Q17, Q18, Q19, Q20, Q21, Q22, Q23, Q24, Q25, Q26: renamed from Q?; value (none) -> 2N7002; footprint (none) -> Package_TO_SOT_SMD:SOT-23
- R10, R11: renamed from R?; value (none) -> 10k; footprint (none) -> Resistor_SMD:R_0603_1608Metric
Connections:
- net RDX renamed ~{STATE_FETCH}
- net XIN_SHIFT renamed STATE_ALU
