File: hardware/q2a/pcb/q2a/fp.kicad_sch (KiCad schematic)
At the start: 8 parts, among them J3 High, J4 Low, U20 245, U21 245, U22 245

Commit message: Board updates.
Parts:
- removed J3: High, Connector_IDC:IDC-Header_2x20_P2.54mm_Vertical, symbol Connector_Generic:Conn_02x20_Odd_Even
- removed J4: Low, Connector_IDC:IDC-Header_2x20_P2.54mm_Vertical, symbol Connector_Generic:Conn_02x20_Odd_Even
- added D1, D10, D11, D12, D13, D14, D15, D16, D17, D18, D19, D2, D20, D21, D22, D23, D24, D25, D26, D27, D28, D29, D3, D4, D5, D6, D7, D8, D9: LED, LED_SMD:LED_0805_2012Metric, symbol Device:LED
- added R19, R20, R21, R22, R23, R24, R25, R26, R27, R28, R29, R30, R31, R32, R33, R34, R35, R36, R37, R38, R39, R40, R41, R42, R43, R44, R45, R46, R47: 10k, Resistor_THT:R_Axial_DIN0207_L6.3mm_D2.5mm_P10.16mm_Horizontal, symbol Device:R
- added SW1: FIELD2, Button_Switch_THT:SW_MINI_TOGGLE, symbol Switch:SW_SPST
- added SW10: 6, Button_Switch_THT:SW_MINI_TOGGLE, symbol Switch:SW_SPST
- added SW11: START, Button_Switch_THT:SW_MINI_TOGGLE, symbol Switch:SW_SPST
- added SW12: 5, Button_Switch_THT:SW_MINI_TOGGLE, symbol Switch:SW_SPST
- added SW13: STOP, Button_Switch_THT:SW_MINI_TOGGLE, symbol Switch:SW_SPST
- added SW14: 4, Button_Switch_THT:SW_MINI_TOGGLE, symbol Switch:SW_SPST
- added SW15: 3, Button_Switch_THT:SW_MINI_TOGGLE, symbol Switch:SW_SPST
- added SW16: SET, Button_Switch_THT:SW_MINI_TOGGLE, symbol Switch:SW_SPST
- added SW17: 2, Button_Switch_THT:SW_MINI_TOGGLE, symbol Switch:SW_SPST
- added SW18: INC, Button_Switch_THT:SW_MINI_TOGGLE, symbol Switch:SW_SPST
- added SW19: 1, Button_Switch_THT:SW_MINI_TOGGLE, symbol Switch:SW_SPST
- added SW2: FIELD1, Button_Switch_THT:SW_MINI_TOGGLE, symbol Switch:SW_SPST
- added SW20: DEP, Button_Switch_THT:SW_MINI_TOGGLE, symbol Switch:SW_SPST
- added SW21: 0, Button_Switch_THT:SW_MINI_TOGGLE, symbol Switch:SW_SPST
- added SW3: FIELD0, Button_Switch_THT:SW_MINI_TOGGLE, symbol Switch:SW_SPST
- added SW4: POWER, Button_Switch_THT:SW_MINI_TOGGLE, symbol Switch:SW_SPST
- added SW5: 11, Button_Switch_THT:SW_MINI_TOGGLE, symbol Switch:SW_SPST
- added SW6: 10, Button_Switch_THT:SW_MINI_TOGGLE, symbol Switch:SW_SPST
- added SW7: 9, Button_Switch_THT:SW_MINI_TOGGLE, symbol Switch:SW_SPST
- added SW8: 8, Button_Switch_THT:SW_MINI_TOGGLE, symbol Switch:SW_SPST
- added SW9: 7, Button_Switch_THT:SW_MINI_TOGGLE, symbol Switch:SW_SPST
- renumbered U20 to U19, U21 to U20, U22 to U21
Connections:
- net FIELD0: now also R22.1
- net FIELD1: now also R20.1
- net GND: now also D1.1 (K), D10.1 (K), D11.1 (K), D12.1 (K), D13.1 (K), D14.1 (K), D15.1 (K), D16.1 (K), D17.1 (K), D18.1 (K), D19.1 (K), D2.1 (K), D20.1 (K), D21.1 (K), D22.1 (K), D23.1 (K), D24.1 (K), D25.1 (K), D26.1 (K), D27.1 (K), D28.1 (K), D29.1 (K), D3.1 (K), D4.1 (K), D5.1 (K), D6.1 (K), D7.1 (K), D8.1 (K), D9.1 (K), SW1.1 (A), SW10.1 (A), SW11.1 (A), SW12.1 (A), SW13.1 (A), SW14.1 (A), SW15.1 (A), SW16.1 (A), SW17.1 (A), SW18.1 (A), SW19.1 (A), SW2.1 (A), SW20.1 (A), SW21.1 (A), SW3.1 (A), SW5.1 (A), SW6.1 (A), SW7.1 (A), SW8.1 (A), SW9.1 (A)
- net PWR: now also SW4.1 (A)
- net RUN: now also R33.1
- net VCC: now also R21.1, SW4.2 (B)
- net ~{DEPSW}: now also SW20.2 (B)
- net ~{INCPSW}: now also SW18.2 (B)
- net ~{RSTSW}: now also SW16.2 (B)
- net ~{STARTSW}: now also SW11.2 (B)
- net ~{STOPSW}: now also SW13.2 (B)
- net ~{SW0}: now also SW21.2 (B)
- net ~{SW10}: now also SW6.2 (B)
- net ~{SW11}: now also SW5.2 (B)
- net ~{SW1}: now also SW19.2 (B)
- net ~{SW2}: now also SW17.2 (B)
- net ~{SW3}: now also SW15.2 (B)
- net ~{SW4}: now also SW14.2 (B)
- net ~{SW5}: now also SW12.2 (B)
- net ~{SW6}: now also SW10.2 (B)
- net ~{SW7}: now also SW9.2 (B)
- net ~{SW8}: now also SW8.2 (B)
- net ~{SW9}: now also SW7.2 (B)
- net at U20.2 (A0): now also R31.1
- net at U20.3 (A1): now also R32.1
- net at U20.4 (A2): now also R34.1
- net at U20.5 (A3): now also R35.1
- net at U20.6 (A4): now also R36.1
- net at U20.7 (A5): now also R37.1
- net at U20.8 (A6): now also R38.1
- net at U20.9 (A7): now also R39.1
- net at U19.9 (A7): now also R30.1
- net at U19.8 (A6): now also R29.1
- net at U19.7 (A5): now also R28.1
- net at U19.6 (A4): now also R27.1
- net at U19.5 (A3): now also R26.1
- net at U19.4 (A2): now also R25.1
- net at U19.3 (A1): now also R24.1
- net at U19.2 (A0): now also R23.1
- net at U21.9 (A7): now also R47.1
- net at U21.4 (A2): now also R42.1
- net at U21.3 (A1): now also R41.1
- net at U21.2 (A0): now also R40.1
- net at U21.8 (A6): now also R46.1
- net at U21.7 (A5): now also R45.1
- net at U21.6 (A4): now also R44.1
- net at U21.5 (A3): now also R43.1
- new net: D22.2 (A), R40.2
- new net: D20.2 (A), R38.2
- new net: D15.2 (A), R33.2
- new net: D1.2 (A), R19.2
- new net: D18.2 (A), R36.2
- new net: D6.2 (A), R24.2
- new net: D2.2 (A), R20.2
- new net: D25.2 (A), R43.2
- new net: D10.2 (A), R28.2
- new net: D21.2 (A), R39.2
- new net: D16.2 (A), R34.2
- new net: D7.2 (A), R25.2
- new net: D24.2 (A), R42.2
- new net: D17.2 (A), R35.2
- new net: D9.2 (A), R27.2
- new net: D19.2 (A), R37.2
- new net: D4.2 (A), R22.2
- new net: D5.2 (A), R23.2
- new net: D13.2 (A), R31.2
- new net: D26.2 (A), R44.2
- new net: D29.2 (A), R47.2
- new net: D14.2 (A), R32.2
- new net: D12.2 (A), R30.2
- new net: D8.2 (A), R26.2
- new net: D28.2 (A), R46.2
- new net: D3.2 (A), R21.2
- new net: D27.2 (A), R45.2
- new net: D23.2 (A), R41.2
- new net: D11.2 (A), R29.2
- new net FIELD2: R19.1
- new net ~{FIELD0SW}: SW3.2 (B)
- new net ~{FIELD1SW}: SW2.2 (B)
- new net ~{FIELD2SW}: SW1.2 (B)
Other:
- moved on the sheet: C6, U19, U20, U21
