File: hardware/q2a/pcb/q2a/io.kicad_sch (KiCad schematic)
At the start: 3 parts, among them J1 IO, U7 245

Commit message: Board updates.
Parts:
- renumbered U7 to U?
Changed lines of the file:
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@@
         )
         (path "/a14fee10-9a48-449e-80d1-f8dffaea277c"
-          (reference "#PWR0160") (unit 1)
+          (reference "#PWR?") (unit 1)
         )
         (path "/a14fee10-9a48-449e-80d1-f8dffaea277c/00000000-0000-0000-0000-000060b90c82"
@@
         )
         (path "/a14fee10-9a48-449e-80d1-f8dffaea277c/2d699bb0-6bf7-4e34-bbb8-42651e38942b"
-          (reference "#PWR0133") (unit 1)
+          (reference "#PWR0123") (unit 1)
         )
       )
@@
       (project "q2a"
         (path "/a14fee10-9a48-449e-80d1-f8dffaea277c"
-          (reference "#PWR0103") (unit 1)
-        )
-        (path "/a14fee10-9a48-449e-80d1-f8dffaea277c/2d699bb0-6bf7-4e34-bbb8-42651e38942b"
-          (reference "#PWR0137") (unit 1)
+          (reference "#PWR?") (unit 1)
+        )
+        (path "/a14fee10-9a48-449e-80d1-f8dffaea277c/2d699bb0-6bf7-4e34-bbb8-42651e38942b"
+          (reference "#PWR0127") (unit 1)
         )
       )
@@
   (symbol (lib_id "power:VCC") (at 95.25 64.77 0) (unit 1)
     (in_bom yes) (on_board yes) (dnp no)
-    (property "Reference" "#PWR094" (at 95.25 68.58 0)
+    (property "Reference" "#PWR?" (at 95.25 68.58 0)
       (effects (font (size 1.27 1.27)) hide)
     )
@@
       (project "q2a"
         (path "/a14fee10-9a48-449e-80d1-f8dffaea277c"
-          (reference "#PWR094") (unit 1)
-        )
-        (path "/a14fee10-9a48-449e-80d1-f8dffaea277c/2d699bb0-6bf7-4e34-bbb8-42651e38942b"
-          (reference "#PWR0134") (unit 1)
+          (reference "#PWR?") (unit 1)
+        )
+        (path "/a14fee10-9a48-449e-80d1-f8dffaea277c/2d699bb0-6bf7-4e34-bbb8-42651e38942b"
+          (reference "#PWR0124") (unit 1)
         )
       )
@@
       (project "q2a"
         (path "/a14fee10-9a48-449e-80d1-f8dffaea277c"
-          (reference "J1") (unit 1)
+          (reference "J?") (unit 1)
         )
         (path "/a14fee10-9a48-449e-80d1-f8dffaea277c/2d699bb0-6bf7-4e34-bbb8-42651e38942b"
@@
         )
         (path "/a14fee10-9a48-449e-80d1-f8dffaea277c"
-          (reference "#PWR0159") (unit 1)
+          (reference "#PWR?") (unit 1)
         )
         (path "/a14fee10-9a48-449e-80d1-f8dffaea277c/00000000-0000-0000-0000-000060b90c82"
@@
         )
         (path "/a14fee10-9a48-449e-80d1-f8dffaea277c/2d699bb0-6bf7-4e34-bbb8-42651e38942b"
-          (reference "#PWR0132") (unit 1)
+          (reference "#PWR0122") (unit 1)
         )
       )
@@
   (symbol (lib_id "power:GND") (at 95.25 105.41 0) (unit 1)
     (in_bom yes) (on_board yes) (dnp no)
-    (property "Reference" "#PWR096" (at 95.25 111.76 0)
+    (property "Reference" "#PWR?" (at 95.25 111.76 0)
       (effects (font (size 1.27 1.27)) hide)
     )
@@
       (project "q2a"
         (path "/a14fee10-9a48-449e-80d1-f8dffaea277c"
-          (reference "#PWR096") (unit 1)
-        )
-        (path "/a14fee10-9a48-449e-80d1-f8dffaea277c/2d699bb0-6bf7-4e34-bbb8-42651e38942b"
-          (reference "#PWR0135") (unit 1)
+          (reference "#PWR?") (unit 1)
+        )
+        (path "/a14fee10-9a48-449e-80d1-f8dffaea277c/2d699bb0-6bf7-4e34-bbb8-42651e38942b"
+          (reference "#PWR0125") (unit 1)
         )
       )
@@
         )
         (path "/a14fee10-9a48-449e-80d1-f8dffaea277c"
-          (reference "#PWR095") (unit 1)
+          (reference "#PWR?") (unit 1)
         )
         (path "/a14fee10-9a48-449e-80d1-f8dffaea277c/00000000-0000-0000-0000-000060b9649c"
@@
         )
         (path "/a14fee10-9a48-449e-80d1-f8dffaea277c/2d699bb0-6bf7-4e34-bbb8-42651e38942b"
-          (reference "#PWR0136") (unit 1)
+          (reference "#PWR0126") (unit 1)
         )
       )
@@
   (symbol (lib_id "74xx:74LS245") (at 95.25 85.09 0) (unit 1)
     (in_bom yes) (on_board yes) (dnp no) (fields_autoplaced)
-    (property "Reference" "U7" (at 97.4441 64.77 0)
+    (property "Reference" "U?" (at 97.4441 64.77 0)
       (effects (font (size 1.27 1.27)) (justify left))
     )
@@
       (project "q2a"
         (path "/a14fee10-9a48-449e-80d1-f8dffaea277c"
-          (reference "U7") (unit 1)
-        )
-        (path "/a14fee10-9a48-449e-80d1-f8dffaea277c/2d699bb0-6bf7-4e34-bbb8-42651e38942b"
-          (reference "U19") (unit 1)
+          (reference "U?") (unit 1)
+        )
+        (path "/a14fee10-9a48-449e-80d1-f8dffaea277c/2d699bb0-6bf7-4e34-bbb8-42651e38942b"
+          (reference "U18") (unit 1)
         )
       )
@@
         )
         (path "/a14fee10-9a48-449e-80d1-f8dffaea277c"
-          (reference "C23") (unit 1)
-        )
-        (path "/a14fee10-9a48-449e-80d1-f8dffaea277c/2d699bb0-6bf7-4e34-bbb8-42651e38942b"
-          (reference "C25") (unit 1)
-        )
-      )
+          (reference "C?") (unit 1)
+        )
+        (path "/a14fee10-9a48-449e-80d1-f8dffaea277c/2d699bb0-6bf7-4e34-bbb8-42651e38942b"
+          (reference "C26") (unit 1)
+        )
+      )
