File: hardware/q2a/pcb/q2a/memory.kicad_sch (KiCad schematic)
At the start: 18 parts, among them U10 2864, U7 6264, U8 2864, U9 6264

Commit message: Board updates.
Parts:
- removed R10, R13, R14, R7, R8, R9: 100k, Resistor_THT:R_Axial_DIN0207_L6.3mm_D2.5mm_P10.16mm_Horizontal, symbol Device:R
- removed U10, U8: 2864, Package_DIP:DIP-28_W15.24mm_Socket, symbol Memory_RAM:KM62256CLP
- added U7: MCP101-450D, symbol Power_Supervisor:MCP101-450D
- U8: renamed from U7; value 6264 -> 62256
- renumbered R16 to R10, R11 to R7, R12 to R8, R15 to R9
Connections:
- net ABUS11: now also U8.23 (A11), U9.23 (A11); no longer U8.20 (~{CS}), U9.20 (~{CS})
- net FIELD0: now also U8.2 (A12), U9.2 (A12)
- net FIELD1: now also U8.26 (A13), U9.26 (A13)
- net GND: now also U7.3 (VSS); no longer U8.1 (A14), U8.2 (A12), U8.23 (A11), U9.1 (A14), U9.2 (A12), U9.23 (A11)
- net VCC: now also U7.2 (VDD); no longer U8.26 (A13), U9.26 (A13)
- new net: U7.1 (RST), U8.20 (~{CS}), U9.20 (~{CS})
- new net FIELD2: U8.1 (A14), U9.1 (A14)
- no-connect marks 4 -> 0
