File: hardware/q2a/pcb/q2a/q2a.kicad_sch (KiCad schematic)
At the start: 28 parts, among them J1 Barrel_Jack_MountingPin, U1 Clock, U2 State, U3 IO, U4 Opcode, U5 14, X1 CXO

Commit message: Board updates.
Parts:
- renumbered C32 to C9
Connections:
- net ABUS11: no longer U5.1
- net GND: now also U5.1
- net WRF: now reaches U3.19 (IO1)
- net ~{ROMCE}: no longer names the net of U5.2
Other:
- added sheet Field (field.kicad_sch)
- added sheet Programmer (programmer.kicad_sch)
- moved on the sheet: C?, R1, U5A, U5B, U5C, U5D, U5E, U5F
